File: RPiPCB/LaserDriver/LaserDriver.kicad_sch (KiCad schematic)
At the start: 0 parts

Commit message: Merge RPi HAT schematic into LaserDriver project; add PCB template
- Replace empty placeholder with 4-sheet hierarchical schematic
  (root + laser driver, MSPM0 controller, USB-C UART sub-sheets)
- Update LaserDriver.kicad_pro with Laser_Power net class and BOM settings
- LaserDriver.kicad_pcb: HAT board outline (65×56.5 mm, 3.5 mm corner radii),
  four M2.5 NPTH mounting holes, and J1 GPIO 2×20 connector at Pi-spec position
  (pin 1 at 8.37, 2.23 mm from top-left / GPIO edge); ready for manual layout

Co-Authored-By: Claude Sonnet 4.6 <noreply@anthropic.com>
Parts:
- added J1: RaspberryPi_2x20_HAT, Connector_PinHeader_2.54mm:PinHeader_2x20_P2.54mm_Vertical, symbol Connector_Generic:Conn_02x20_Odd_Even
- added J_BNC: BNC_Trigger, Connector_Coaxial:BNC_Amphenol_B6252HB-NPP3G-50_EdgeMount, symbol Connector:BNC
- added J_SWD: SWD_5pin_0.1in, Connector_PinHeader_2.54mm:PinHeader_1x05_P2.54mm_Vertical, symbol Connector_Generic:Conn_01x05
- added Q_PWR: DMG2305UX, Package_TO_SOT_SMD:SOT-23, symbol Transistor_FET:DMG2305UX
- added R_GATE: 1k, Resistor_SMD:R_0402_1005Metric, symbol Device:R
- added R_I2C_SCL, R_I2C_SDA: 4.7k, Resistor_SMD:R_0402_1005Metric, symbol Device:R
- added R_PD: 10k, Resistor_SMD:R_0402_1005Metric, symbol Device:R
- added R_TERM: 50R DNP, Resistor_SMD:R_0402_1005Metric, symbol Device:R
- added U_EEPROM: AT24C256, Package_SO:SOIC-8_3.9x4.9mm_P1.27mm, symbol Memory_EEPROM:AT24C256
Other:
- added sheet Laser Driver Circuit (laser_driver_circuit.kicad_sch)
- added sheet MSPM0 Controller (mspm0_controller.kicad_sch)
- added sheet USB-C UART Interface (usb_uart.kicad_sch)
- note added: "BNC Trigger Interface J_BNC center → TRIGGER net MSPM0 PB21 internal pull-up enabled Active-low, 10 ms debounce in firmware R_TERM (50Ω): DNP by default Pi GPIO18 connected in parallel"
- note added: "HAT EEPROM (AT24C256) Required by Pi HAT spec. I2C address: A0=A1=A2=GND → 0x50 Interface: ID_SD/ID_SC (Pi GPIO0/GPIO1) 4.7kΩ pull-ups to +3.3V on SDA and SCL WP=GND (write enabled during programming)"
- note added: "MSPM0 Power Switch Q_PWR (DMG2305UX, P-MOSFET) +3.3V (Pi) → Source Drain → VCC_3V3_MCU Gate: R_GATE (1kΩ) from GPIO17 R_PD (10kΩ) to GND Default: gate LOW → MOSFET ON GPIO17 HIGH → power cycle MSPM0"
- note added: "Raspberry Pi 40-pin HAT Connector Pin Assignments Pins 1,17: +3.3V Pins 2,4: +5V Pins 6,9,14,20,25,30,34,39: GND Pin 8 (GPIO14/TXD): Pi UART TX → MSPM0 PA11 (RX) Pin 10 (GPIO15/RXD): Pi UART RX ← MSPM0 PA10 (TX) Pin 11 (GPIO17): PWR_EN → Q_PWR gate (P-MOSFET) Pin 12 (GPIO18): TRIGGER → MSPM0 PB21 ‖ BNC Pin 16 (GPIO23): SWCLK → MSPM0 PA19 ‖ J_SWD pin 2 Pin 18 (GPIO24): SWDIO → MSPM0 PA20 ‖ J_SWD p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"
- note added: "SWD Debug Header J_SWD (5-pin, 0.1" pitch) Pin 1: NRST Pin 2: SWCLK (MSPM0 PA19) Pin 3: SWDIO (MSPM0 PA20) Pin 4: +3.3V (target power reference) Pin 5: GND Also connected to Pi GPIO23/24/25 for OpenOCD bit-bang (bcm2835gpio). When using external debugger, set Pi GPIOs to input (high-impedance)."
- company: (none) -> Rice University
- title: (none) -> Laser Diode Driver — Raspberry Pi HAT
