File: LaserHAT/LaserDriver.kicad_sch (KiCad schematic)
At the start: 9 parts

Commit message: Implement schematic design rules; add CLAUDE.md
- Rule 1: hide pin names/numbers on passive parts (R, C, L)
- Rule 2: add ≥5mm wire stub before every net label
- Rule 3: preserve hand-edited laser_driver.kicad_sch by loading from PCB/ original
- Rule 4: generous component spacing across multiple sheets
- Add CLAUDE.md documenting all rules, setup, signal naming, and kiutils conventions

Co-Authored-By: Claude Sonnet 4.6 <noreply@anthropic.com>
Parts:
- removed Q_PWR: DMG2305UX, Package_TO_SOT_SMD:SOT-323_SC-70, symbol Transistor_FET:DMG2305UX
- added Q_PWR: DMG2305UX, Package_TO_SOT_SMD:SOT-323_SC-70, symbol Transistor_FET:DMG2302U

Commit message: Fix three schematic generation bugs
- Symbol unit names: set entryName on manually-created Symbol units so
  they serialize as "+LASER_V_0_1" not "None_0_1" (KiCad load error)
- Passive pin hiding: set pinNames=True alongside pinNamesHide=True so
  the (pin_names hide) token is actually emitted for Device:C and Device:L
- Property visibility: hide Footprint/Datasheet/Description on all
  schematic symbol instances; only Reference and Value remain shown

Co-Authored-By: Claude Sonnet 4.6 <noreply@anthropic.com>
Changed lines of the file:
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@@
     )
     (property "Footprint" "Package_TO_SOT_SMD:SOT-323_SC-70" (at 60 40 0)
-      (effects (font (size 1.27 1.27)))
+      (effects (font (size 1.27 1.27)) hide)
     )
     (property "Datasheet" "~" (at 60 40 0)
-      (effects (font (size 1.27 1.27)))
+      (effects (font (size 1.27 1.27)) hide)
     )
     (pin "1")
@@
     )
     (property "Footprint" "" (at 0.0 0.0 0)
-      (effects (font (size 1.27 1.27)))
-    )
-    (property "Datasheet" "~" (at 0.0 0.0 0)
-      (effects (font (size 1.27 1.27)))
+      (effects (font (size 1.27 1.27)) hide)
+    )
+    (property "Datasheet" "~" (at 0.0 0.0 0)
+      (effects (font (size 1.27 1.27)) hide)
     )
     (pin "1")
@@
     )
     (property "Footprint" "Resistor_SMD:R_0402_1005Metric" (at 40 40 0)
-      (effects (font (size 1.27 1.27)))
+      (effects (font (size 1.27 1.27)) hide)
     )
     (property "Datasheet" "~" (at 40 40 0)
-      (effects (font (size 1.27 1.27)))
+      (effects (font (size 1.27 1.27)) hide)
     )
     (pin "1")
@@
     )
     (property "Footprint" "Resistor_SMD:R_0402_1005Metric" (at 50 40 0)
-      (effects (font (size 1.27 1.27)))
+      (effects (font (size 1.27 1.27)) hide)
     )
     (property "Datasheet" "~" (at 50 40 0)
-      (effects (font (size 1.27 1.27)))
+      (effects (font (size 1.27 1.27)) hide)
     )
     (pin "1")
@@
     )
     (property "Footprint" "Connector_Coaxial:BNC_Amphenol_031-221-RFX_Horizontal" (at 90 40 0)
-      (effects (font (size 1.27 1.27)))
+      (effects (font (size 1.27 1.27)) hide)
     )
     (property "Datasheet" "~" (at 90 40 0)
-      (effects (font (size 1.27 1.27)))
+      (effects (font (size 1.27 1.27)) hide)
     )
     (pin "1")
@@
     )
     (property "Footprint" "Resistor_SMD:R_0402_1005Metric" (at 105 40 0)
-      (effects (font (size 1.27 1.27)))
+      (effects (font (size 1.27 1.27)) hide)
     )
     (property "Datasheet" "~" (at 105 40 0)
-      (effects (font (size 1.27 1.27)))
+      (effects (font (size 1.27 1.27)) hide)
     )
     (pin "1")
@@
     )
     (property "Footprint" "Connector_PinHeader_2.54mm:PinHeader_1x05_P2.54mm_Vertical" (at 130 30 0)
-      (effects (font (size 1.27 1.27)))
+      (effects (font (size 1.27 1.27)) hide)
     )
     (property "Datasheet" "~" (at 130 30 0)
-      (effects (font (size 1.27 1.27)))
+      (effects (font (size 1.27 1.27)) hide)
     )
     (pin "1")
@@
     )
     (property "Footprint" "" (at 0.0 0.0 0)
-      (effects (font (size 1.27 1.27)))
-    )
-    (property "Datasheet" "~" (at 0.0 0.0 0)
-      (effects (font (size 1.27 1.27)))
+      (effects (font (size 1.27 1.27)) hide)
+    )
+    (property "Datasheet" "~" (at 0.0 0.0 0)
+      (effects (font (size 1.27 1.27)) hide)
     )
     (pin "1")
@@
     )
     (property "Footprint" "" (at 0.0 0.0 0)
-      (effects (font (size 1.27 1.27)))
-    )
-    (property "Datasheet" "~" (at 0.0 0.0 0)
-      (effects (font (size 1.27 1.27)))
+      (effects (font (size 1.27 1.27)) hide)
+    )
+    (property "Datasheet" "~" (at 0.0 0.0 0)
+      (effects (font (size 1.27 1.27)) hide)
     )
     (pin "1")
@@
     )
     (property "Footprint" "Package_SO:SOIC-8_3.9x4.9mm_P1.27mm" (at 160 35 0)
-      (effects (font (size 1.27 1.27)))
+      (effects (font (size 1.27 1.27)) hide)
     )
     (property "Datasheet" "~" (at 160 35 0)
-      (effects (font (size 1.27 1.27)))
+      (effects (font (size 1.27 1.27)) hide)
     )
     (pin "1")
@@
     )
     (property "Footprint" "" (at 0.0 0.0 0)
-      (effects (font (size 1.27 1.27)))
-    )
-    (property "Datasheet" "~" (at 0.0 0.0 0)
-      (effects (font (size 1.27 1.27)))
+      (effects (font (size 1.27 1.27)) hide)
+    )
+    (property "Datasheet" "~" (at 0.0 0.0 0)
+      (effects (font (size 1.27 1.27)) hide)
     )
     (pin "1")
@@
     )
     (property "Footprint" "" (at 0.0 0.0 0)
-      (effects (font (size 1.27 1.27)))
-    )
-    (property "Datasheet" "~" (at 0.0 0.0 0)
-      (effects (font (size 1.27 1.27)))
+      (effects (font (size 1.27 1.27)) hide)
+    )
+    (property "Datasheet" "~" (at 0.0 0.0 0)
+      (effects (font (size 1.27 1.27)) hide)
     )
     (pin "1")
@@
     )
     (property "Footprint" "" (at 0.0 0.0 0)
-      (effects (font (size 1.27 1.27)))
-    )
-    (property "Datasheet" "~" (at 0.0 0.0 0)
-      (effects (font (size 1.27 1.27)))
+      (effects (font (size 1.27 1.27)) hide)
+    )
+    (property "Datasheet" "~" (at 0.0 0.0 0)
+      (effects (font (size 1.27 1.27)) hide)
     )
     (pin "1")
@@
     )
     (property "Footprint" "" (at 0.0 0.0 0)
-      (effects (font (size 1.27 1.27)))
-    )
-    (property "Datasheet" "~" (at 0.0 0.0 0)
-      (effects (font (size 1.27 1.27)))
+      (effects (font (size 1.27 1.27)) hide)
+    )
+    (property "Datasheet" "~" (at 0.0 0.0 0)
+      (effects (font (size 1.27 1.27)) hide)
     )
     (pin "1")
@@
     )
     (property "Footprint" "" (at 0.0 0.0 0)
-      (effects (font (size 1.27 1.27)))
-    )
-    (property "Datasheet" "~" (at 0.0 0.0 0)
-      (effects (font (size 1.27 1.27)))
+      (effects (font (size 1.27 1.27)) hide)
+    )
+    (property "Datasheet" "~" (at 0.0 0.0 0)
+      (effects (font (size 1.27 1.27)) hide)
     )
     (pin "1")
@@
     )
     (property "Footprint" "" (at 0.0 0.0 0)
-      (effects (font (size 1.27 1.27)))
-    )
-    (property "Datasheet" "~" (at 0.0 0.0 0)
-      (effects (font (size 1.27 1.27)))
+      (effects (font (size 1.27 1.27)) hide)
+    )
+    (property "Datasheet" "~" (at 0.0 0.0 0)
+      (effects (font (size 1.27 1.27)) hide)
     )
     (pin "1")
@@
     )
     (property "Footprint" "Resistor_SMD:R_0402_1005Metric" (at 175 25 0)
-      (effects (font (size 1.27 1.27)))
+      (effects (font (size 1.27 1.27)) hide)
     )
     (property "Datasheet" "~" (at 175 25 0)
-      (effects (font (size 1.27 1.27)))
+      (effects (font (size 1.27 1.27)) hide)
     )
     (pin "1")
@@
     )
     (property "Footprint" "Resistor_SMD:R_0402_1005Metric" (at 188 25 0)
-      (effects (font (size 1.27 1.27)))
+      (effects (font (size 1.27 1.27)) hide)
     )
     (property "Datasheet" "~" (at 188 25 0)
-      (effects (font (size 1.27 1.27)))
+      (effects (font (size 1.27 1.27)) hide)
     )
     (pin "1")
@@
   )
   (symbol_instances
-    (path "/212bfd25-f831-4b85-926b-437df65a6b12/2273e221-0dec-4925-a92b-55abdd2272a4"
+    (path "/212bfd25-f831-4b85-926b-437df65a6b12/e70f625d-7d06-442e-9b18-c1751305972d"
       (reference "Q_PWR") (unit 1) (value "DMG2305UX") (footprint "Package_TO_SOT_SMD:SOT-323_SC-70")
     )
-    (path "/212bfd25-f831-4b85-926b-437df65a6b12/e01ad76c-6498-4dd8-a2bf-954fa6cc9c12"
+    (path "/212bfd25-f831-4b85-926b-437df65a6b12/0fde6227-3832-425f-b386-a30eed4b015b"
       (reference "R_GATE") (unit 1) (value "1k") (footprint "Resistor_SMD:R_0402_1005Metric")
     )
-    (path "/212bfd25-f831-4b85-926b-437df65a6b12/edae41b1-7739-43ab-a5d7-a4fb30d89e5c"
+    (path "/212bfd25-f831-4b85-926b-437df65a6b12/6ef04b3d-1484-4460-994a-39a9d54ef708"
       (reference "R_PD") (unit 1) (value "10k") (footprint "Resistor_SMD:R_0402_1005Metric")
     )
-    (path "/212bfd25-f831-4b85-926b-437df65a6b12/bd32e647-b638-4309-941c-c35694abb9cf"
+    (path "/212bfd25-f831-4b85-926b-437df65a6b12/aac20f33-436c-4050-9bf9-b50d0c643378"
       (reference "J_BNC") (unit 1) (value "BNC_Trigger") (footprint "Connector_Coaxial:BNC_Amphenol_031-221-RFX_Horizontal")
     )
-    (path "/212bfd25-f831-4b85-926b-437df65a6b12/508b592e-9bdd-4f92-848d-3c6cdacbbbcb"
+    (path "/212bfd25-f831-4b85-926b-437df65a6b12/f2abfaaa-4d54-43e4-8061-4bd458261007"
       (reference "R_TERM") (unit 1) (value "50R DNP") (footprint "Resistor_SMD:R_0402_1005Metric")
     )
-    (path "/212bfd25-f831-4b85-926b-437df65a6b12/99da9392-c63d-48a3-9b82-a683e475dca8"
+    (path "/212bfd25-f831-4b85-926b-437df65a6b12/bd01444e-fae3-4f21-a236-da7c5715de8b"
       (reference "J_SWD") (unit 1) (value "SWD 5-pin 0.1\"") (footprint "Connector_PinHeader_2.54mm:PinHeader_1x05_P2.54mm_Vertical")
     )
-    (path "/212bfd25-f831-4b85-926b-437df65a6b12/f3bca928-9fcf-49cc-be1d-67576cd9f3f8"
+    (path "/212bfd25-f831-4b85-926b-437df65a6b12/30b6c333-dc4b-4fc1-9c78-ffc1e01f4d78"
       (reference "U_EEPROM") (unit 1) (value "AT24C256C") (footprint "Package_SO:SOIC-8_3.9x4.9mm_P1.27mm")
     )
-    (path "/212bfd25-f831-4b85-926b-437df65a6b12/1efdddc3-7059-450d-8e0f-1c2e3f0f2de3"
+    (path "/212bfd25-f831-4b85-926b-437df65a6b12/1e9bf496-5246-47c5-a27e-dad4bd12fe13"
       (reference "R_I2C_SDA") (unit 1) (value "4k7") (footprint "Resistor_SMD:R_0402_1005Metric")
     )
-    (path "/212bfd25-f831-4b85-926b-437df65a6b12/105773d2-d31a-429c-ac6b-55f92f87073e"
+    (path "/212bfd25-f831-4b85-926b-437df65a6b12/aa131af2-e2f0-4146-9762-65fcedcfdbea"
       (reference "R_I2C_SCL") (unit 1) (value "4k7") (footprint "Resistor_SMD:R_0402_1005Metric")
     )

Commit message: Add RPi 40-pin GPIO header to root schematic with full pin connections
- place_pi_header() places Conn_02x20_Odd_Even at (40, 230) with:
  - Pins 1,17: +3V3 power symbols
  - Pins 2,4: VCC_5V_IN net labels (boost converter input)
  - Pins 6,9,14,20,25,30,34,39: GND power symbols
  - Pin 8/10: UART_TX/UART_RX (GPIO14/15)
  - Pin 11: Pi_GPIO17 (MCU power enable → R_GATE)
  - Pins 27/28: ID_SDA/ID_SCL (HAT EEPROM, per HAT spec)
  - Pin 37: TRIGGER (GPIO26 → BNC/MSPM0)
  - All other pins: no-connect markers
- Fix TRIGGER_SIG → TRIGGER to match MSPM0 sub-sheet port name
- Fix power:3V3 → power:+3V3 bug (lstrip("+") was wrong)

Co-Authored-By: Claude Sonnet 4.6 <noreply@anthropic.com>
Parts:
- added J_PI: RPi_GPIO_40, Connector_PinHeader_2.54mm:PinHeader_2x20_P2.54mm_Vertical, symbol Connector_Generic:Conn_02x20_Odd_Even
Connections:
- net TRIGGER_SIG is gone; now on net TRIGGER: R_TERM.2
- net +3V3: now also J_PI.1 (Pin_1)
- net VCC_5V_IN: now also J_PI.2 (Pin_2)
- no-connect marks 0 -> 22

Commit message: Preserve GPIO header UUID by loading from original schematic
The PCB footprint for J1 (40-pin GPIO header) has
  (path "/212bfd25-0010-0000-0000-000000000001")
which must match the schematic symbol UUID. Regenerating the symbol
with a random UUID silently orphans the footprint.

Fix: build_root() now loads PCB/laserhat_root_orig.kicad_sch (extracted
from the initial commit) and borrows the pristine Conn_02x20_Odd_Even
lib symbol + J1 instance verbatim. Only net labels/power symbols/
no-connects are added; the symbol itself (UUID, pin UUIDs, position,
lib symbol definition) is untouched.

Also add hide_extra_properties() call at end of build_root() and
document the UUID invariant in CLAUDE.md.

Co-Authored-By: Claude Sonnet 4.6 <noreply@anthropic.com>
Parts:
- removed J_PI: RPi_GPIO_40, Connector_PinHeader_2.54mm:PinHeader_2x20_P2.54mm_Vertical, symbol Connector_Generic:Conn_02x20_Odd_Even
- added J1: RaspberryPi_2x20_HAT, Connector_PinHeader_2.54mm:PinHeader_2x20_P2.54mm_Vertical, symbol Connector_Generic:Conn_02x20_Odd_Even
Connections:
- net +3V3: now also J1.1 (Pin_1)
- net VCC_5V_IN: now also J1.2 (Pin_2)

Commit message: Rebase schematic and PCB from PiHatTemplate
Schematic (LaserDriver.kicad_sch): template taken as base verbatim,
preserving all GPIO connector symbols, pin labels, decoupling caps,
ID EEPROM notes, and solder jumpers exactly as drawn. Paper changed
A4→A3; title block updated. Three sub-sheet boxes (Laser Driver,
MSPM0, USB-C UART) appended at x=230 to avoid overlap with the
template's GPIO content.

PCB (LaserDriver.kicad_pcb): replaced with PiHatTemplate PCB, which
uses the correct PinSocket_2x20 on B.Cu (female, mates with Pi header)
and includes proper board-outline notches, stackup, and mounting holes.
Updated sheetfile reference to LaserDriver.kicad_sch; J1 UUID link
(00000000-0000-0000-0000-000059ad464a) is consistent with schematic.

Added merge_template.py script that performs the merge reproducibly.

Co-Authored-By: Claude Sonnet 4.6 <noreply@anthropic.com>
Parts:
- removed J_BNC: BNC_Trigger, Connector_Coaxial:BNC_Amphenol_031-221-RFX_Horizontal, symbol Connector_Coaxial:BNC
- removed J_SWD: SWD 5-pin 0.1", Connector_PinHeader_2.54mm:PinHeader_1x05_P2.54mm_Vertical, symbol Connector_Generic:Conn_01x05
- removed Q_PWR: DMG2305UX, Package_TO_SOT_SMD:SOT-323_SC-70, symbol Transistor_FET:DMG2302U
- removed R_GATE: 1k, Resistor_SMD:R_0402_1005Metric, symbol Device:R
- removed R_I2C_SCL, R_I2C_SDA: 4k7, Resistor_SMD:R_0402_1005Metric, symbol Device:R
- removed R_PD: 10k, Resistor_SMD:R_0402_1005Metric, symbol Device:R
- removed R_TERM: 50R DNP, Resistor_SMD:R_0402_1005Metric, symbol Device:R
- removed U_EEPROM: AT24C256C, Package_SO:SOIC-8_3.9x4.9mm_P1.27mm, symbol Memory_EEPROM:AT24C256C
- added C1: 100n, symbol Device:C_Small
- added JP1: ID_WP, symbol Jumper:SolderJumper_2_Open
- added R1, R2: 3.9k, symbol Device:R_Small
- added U1: CAT24C256, symbol Memory_EEPROM:CAT24C256
- J1: value RaspberryPi_2x20_HAT -> GPIO; footprint Connector_PinHeader_2.54mm:PinHeader_2x20_P2.54mm_Vertical -> Connector_PinSocket_2.54mm:PinSocket_2x20_P2.54mm_Vertical
Connections:
- net VCC_5V_IN is gone; now on net +5V: J1.2 (Pin_2)
- net +3V3: now also J1.17 (Pin_17), C1.1, JP1.2 (B), R1.1, R2.1, U1.8 (VCC)
- net GND: now also J1.14 (Pin_14), J1.20 (Pin_20), J1.25 (Pin_25), J1.30 (Pin_30), J1.34 (Pin_34), J1.39 (Pin_39), J1.6 (Pin_6), J1.9 (Pin_9), C1.2, U1.4 (GND)
- net ID_SCL: now also J1.28 (Pin_28), R2.2, U1.6 (SCL)
- net ID_SDA: now also J1.27 (Pin_27), R1.2, U1.5 (SDA)
- net GPIO15/RXD0: now reaches J1.10 (Pin_10)
- net GPIO17: now reaches J1.11 (Pin_11)
- net GPIO18/PCM.CLK: now reaches J1.12 (Pin_12)
- net GPIO27: now reaches J1.13 (Pin_13)
- net GPIO22: now reaches J1.15 (Pin_15)
- net GPIO23: now reaches J1.16 (Pin_16)
- net GPIO24: now reaches J1.18 (Pin_18)
- net GPIO10/SPI0.MOSI: now reaches J1.19 (Pin_19)
- net GPIO9/SPI0.MISO: now reaches J1.21 (Pin_21)
- net GPIO25: now reaches J1.22 (Pin_22)
- net GPIO11/SPI0.SCLK: now reaches J1.23 (Pin_23)
- net GPIO8/SPI0.CE0: now reaches J1.24 (Pin_24)
- net GPIO7/SPI0.CE1: now reaches J1.26 (Pin_26)
- net GPIO5: now reaches J1.29 (Pin_29)
- net GPIO2/SDA1: now reaches J1.3 (Pin_3)
- net GPIO6: now reaches J1.31 (Pin_31)
- net GPIO12/PWM0: now reaches J1.32 (Pin_32)
- net GPIO13/PWM1: now reaches J1.33 (Pin_33)
- net GPIO19/PCM.FS: now reaches J1.35 (Pin_35)
- net GPIO16: now reaches J1.36 (Pin_36)
- net GPIO26: now reaches J1.37 (Pin_37)
- net GPIO20/PCM.DIN: now reaches J1.38 (Pin_38)
- net +5V: now reaches J1.4 (Pin_4)
- net GPIO21/PCM.DOUT: now reaches J1.40 (Pin_40)
- net GPIO3/SCL1: now reaches J1.5 (Pin_5)
- net GPIO4/GPCLK0: now reaches J1.7 (Pin_7)
- net GPIO14/TXD0: now reaches J1.8 (Pin_8)
- new net: JP1.1 (A), U1.7 (WP)
- no-connect marks 22 -> 3
Other:
- note added: "Additional pin functions: https://pinout.xyz/"
- note added: "ID_SD and ID_SC PINS: These pins are reserved for HAT ID EEPROM. At boot time this I2C interface will be interrogated to look for an EEPROM that identifes the attached board and allows automagic setup of the GPIOs (and optionally, Linux drivers). Bridging JP1 enables write protection. DO NOT USE these pins for anything other than attaching an I2C ID EEPROM. Leave unconnected if ID EEPROM not requ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"
