File: LaserHAT/LaserDriver.kicad_sch (KiCad schematic)
At the start: 6 parts, among them J1 GPIO, U1 CAT24C256

Commit message: Updates with lots of manual work
Parts:
- added C12: 100nF Ceramic, Capacitor_SMD:C_0402_1005Metric, symbol Device:C_Small
- added C13: 1uF Ceramic, Capacitor_SMD:C_0603_1608Metric, symbol Device:C_Small
- added C14: 10nF, Capacitor_SMD:C_0402_1005Metric, symbol Device:C_Small
- added D5: 5V, Diode_SMD:D_0603_1608Metric, symbol Device:LED
- added D6: 3v3, Diode_SMD:D_0603_1608Metric, symbol Device:LED
- added D7: MSPM0, Diode_SMD:D_0603_1608Metric, symbol Device:LED
- added D8: LASER_V, Diode_SMD:D_0603_1608Metric, symbol Device:LED
- added D9: STIM, Diode_SMD:D_0603_1608Metric, symbol Device:LED
- added J6, J7: Conn_Coaxial, Connector_Coaxial:BNC_Amphenol_031-5539_Vertical, symbol Connector:Conn_Coaxial
- added JP4: ID_WP, Jumper:SolderJumper-2_P1.3mm_Open_TrianglePad1.0x1.5mm, symbol Jumper:SolderJumper_2_Open
- added R13, R15, R18: 1k, Resistor_SMD:R_0402_1005Metric, symbol Device:R
- added R14, R16: 500, Resistor_SMD:R_0402_1005Metric, symbol Device:R
- added R17: 10k, Resistor_SMD:R_0402_1005Metric, symbol Device:R
- added U4: MCP1700x-330xxMB, Package_TO_SOT_SMD:SOT-89-3, symbol Regulator_Linear:MCP1700x-330xxMB
- JP1: footprint (none) -> Jumper:SolderJumper-2_P1.3mm_Open_TrianglePad1.0x1.5mm
Connections:
- net +5V: now also C12.1, D5.2 (A), U4.2 (VI)
- net GND: now also C12.2, C13.2, C14.2, J6.2 (Ext), J7.2 (Ext), R13.2, R14.2, R15.2, R16.2, R18.2, U4.1 (GND)
- net +3V3 renamed RPi +3V3
- net GPIO10/SPI0.MOSI renamed EINK_COPI
- net GPIO11/SPI0.SCLK renamed EINK_SCK
- net GPIO14/TXD0 renamed MCU_UART_TX
- net GPIO15/RXD0 renamed MCU_UART_RX
- net GPIO17 renamed EINK_BUSY
- net GPIO18/PCM.CLK renamed MSPM0_NRST
- net MSPM0_NRST: now also JP4.1 (A)
- net GPIO22 renamed EINK_DC
- net GPIO23 renamed MCU_POWER_EN
- net MCU_POWER_EN: now also C14.1, R17.2
- net GPIO24 renamed MSPM0_SWDIO
- net GPIO25 renamed MSPM0_SWCLK
- net GPIO27 renamed EINK_RESET
- net GPIO8/SPI0.CE0 renamed EINK_CS
- net GPIO9/SPI0.MISO renamed EINK_CIPO
- new net: D9.1 (K), R16.1
- new net: D5.1 (K), R13.1
- new net: D6.1 (K), R14.1
- new net: D8.1 (K), R18.1
- new net: D7.1 (K), R15.1
- new net +3.3V: C13.1, D6.2 (A), R17.1, U4.3 (VO)
- new net LASER_BOOST: D8.2 (A)
- new net MSPM0_3v3: D7.2 (A)
- new net STIM_MIRROR: D9.2 (A), J7.1 (In)
- new net STIM_TRIGGER: J6.1 (In)
- new net USB-C UART/CH340_RTS: JP4.2 (B)
Other:
- added sheet EInk Display (eink.kicad_sch)
- sheet Laser Driver Circuit ports: added BOOST_EN, DIODE_ADC, LASER_V, LASER_VREF, V_LASER_BOOST_IN; removed GND, VCC_3V3, VCC_5V_IN, VREF
- sheet MSPM0 Controller ports: added LASER_BOOST_EN, MCU_POWER_EN, MCU_UART_RX, MCU_UART_TX, MSPM0_3v3, MSPM0_ADC, MSPM0_DAC, MSPM0_NRST, MSPM0_SWCLK, MSPM0_SWDIO, STIM_MIRROR, STIM_TRIGGER; removed GND, NRST, SWCLK, SWDIO, TRIGGER, UART_RX, UART_TX, VCC_3V3_MCU, VREF
- sheet USB-C UART ports: added 3v3_REG, CH340_RTS, CH340_RX, CH340_TX; removed GND, UART_RX, UART_TX, VBUS_5V
- note added: "TODO - Add in Rev 2. For now, can use an Adafruit Bonnet"

Commit message: Updates to design, finalized PCB layout
Parts:
- removed C14: 10nF, Capacitor_SMD:C_0402_1005Metric, symbol Device:C_Small
- removed D8: LASER_V, Diode_SMD:D_0603_1608Metric, symbol Device:LED
- added D10: D_Zener 6.2V, Diode_SMD:D_SOD-523, symbol Device:D_Zener
- added D8: LED_Dual_AKAK, LED_SMD:LED_LiteOn_LTST-C295K_1.6x0.8mm, symbol Device:LED_Dual_AKAK
- added R17: 500, Resistor_SMD:R_0402_1005Metric, symbol Device:R
- C15: renamed from C1; footprint (none) -> Capacitor_SMD:C_0402_1005Metric
- J1: footprint Connector_PinSocket_2.54mm:PinSocket_2x20_P2.54mm_Vertical -> Connector_Samtec_HLE_SMD:Samtec_HLE-120-02-xxx-DV-BE-LC_2x20_P2.54mm_Horizontal; LCSC Part # (none) -> C42411761
- JP1: footprint Jumper:SolderJumper-2_P1.3mm_Open_TrianglePad1.0x1.5mm -> Jumper:SolderJumper-2_P1.3mm_Open_RoundedPad1.0x1.5mm
- R1, R2: footprint (none) -> Resistor_SMD:R_0402_1005Metric
- R16: renamed from R18; value 1k -> 500
- U1: value CAT24C256 -> CAT24C32; footprint (none) -> Package_SO:TSSOP-8_4.4x3mm_P0.65mm; LCSC Part # (none) -> C94264
- renumbered R16 to R18, R17 to R7
Connections:
- net GND: now also R17.2
- net at R16.1: now also D8.4 (K2)
- net +3.3V renamed +3V3
- net MSPM0_3v3 renamed MSPM0_3V3
- new net: D10.2 (A), D8.2 (K1)
- new net: D10.1 (K), R17.1
- new net LASER_V: D8.1 (A1), D8.3 (A2)
Other:
- sheet Laser Driver Circuit ports: added none; removed BOOST_EN, LASER_V
- sheet MSPM0 Controller ports: added none; removed LASER_BOOST_EN, MSPM0_3v3
- moved on the sheet: D9, R16, R18
