File: LaserHAT/LaserDriver.kicad_sch (KiCad schematic)
At the start: 25 parts, among them J1 GPIO, J6 Conn_Coaxial, J7 Conn_Coaxial, U1 CAT24C32, U4 MCP1700x-330xxMB

Commit message: Updated project for manufacturing. Should merge branch if/when we get back a working product
Parts:
- removed D8: LED_Dual_AKAK, LED_SMD:LED_LiteOn_LTST-C295K_1.6x0.8mm, symbol Device:LED_Dual_AKAK
- added D11: LED_ABGR, LED_SMD:LED_RGB_1210, symbol Device:LED_ABGR
- C12: value 100nF Ceramic -> 100nF; LCSC Part # (none) -> C307331
- C13: footprint Capacitor_SMD:C_0603_1608Metric -> Capacitor_SMD:C_0402_1005Metric; LCSC Part # (none) -> C52923
- C15: value 100n -> 100nF; LCSC Part # (none) -> C307331
- D10: LCSC Part # (none) -> C2886074; LCSC Part# C2886074 -> (none)
- D5, D6, D7, D9: LCSC Part # (none) -> C5336487
- J6, J7: now not fitted
- R1, R2: LCSC Part # (none) -> C51721
- R13: value 1k -> 1k 1%; LCSC Part # (none) -> C131360
- R14: value 500 -> 200; LCSC Part # (none) -> C25087
- R15: value 1k -> 200; LCSC Part # (none) -> C25087
- R16, R18: value 500 -> 470; LCSC Part # (none) -> C25117
- R17: value 500 -> 1k 1%; LCSC Part # (none) -> C131360
- R7: LCSC Part # (none) -> C25744
- U4: LCSC Part # (none) -> C632000; LCSC Part# C632000 -> (none)
Connections:
- net LASER_V: now also D11.1 (A)
- net at D10.2 (A): now also D11.4 (RK)
- net at R16.1: now also D11.2 (BK)
Other:
- moved on the sheet: D10, R16, R17
