File: LaserHAT/LaserDriver.kicad_sch (KiCad schematic)
At the start: 19 parts, among them J1 GPIO, U1 CAT24C32, U4 MCP1700x-330xxMB

Commit message: Small shifts on PCB and updated version of schematic
Parts:
- J1: now not fitted
