File: LaserHAT/LaserDriver.kicad_sch (KiCad schematic)
At the start: 19 parts, among them J1 GPIO, U1 CAT24C32, U4 MCP1700x-330xxMB

Commit message: LaserHAT: owl logo's laser eyes and beams are pads on GND
- Footprints.pretty/OwlLogo_Laser_14mm: the two eye polygons and two beam lines on F.Cu/F.Mask
  become four custom pads numbered 1 (solid zone connection), so the exposed copper is on a net
- LaserHAT.kicad_sym + root sheet lib copy: OwlLogo gets pin 1 "GND" (passive, below the body);
  G1 moved onto the 1.27 mm grid and a GND power symbol placed on its pin
- LaserDriver.kicad_pcb: G1 swapped for the new footprint (same position/path), pads on GND,
  zones refilled; DRC unchanged, 0 unconnected; backup stash/LaserDriver_user_2026-09-30_pre-owlgnd
- tools/jlc_fab.py: footprints excluded from both BOM and position files count as non-parts
  (the logo was being listed as hand-fit); HAT fab outputs regenerated

Co-Authored-By: Claude Fable 5.1 <noreply@anthropic.com>
Claude-Session: https://claude.ai/code/session_018vgLizGzYPynnY93ajvoVA
Connections:
- net GND: now also G1.1 (GND)
Changed lines of the file:
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@@
 	(symbol
 		(lib_id "LaserHAT:OwlLogo")
-		(at 25.4 275 0)
+		(at 25.4 274.32 0)
 		(unit 1)
 		(exclude_from_sim yes)
@@
 		(dnp no)
 		(property "Reference" "G1"
-			(at 25.4 267.15 0)
+			(at 25.4 266.47 0)
 			(effects
 				(font
@@
 		)
 		(property "Value" "OwlLogo"
-			(at 25.4 282.85 0)
+			(at 25.4 282.17 0)
 			(effects
 				(font
@@
 		)
 		(property "Footprint" "Footprints:OwlLogo_Laser_14mm"
-			(at 25.4 275 0)
+			(at 25.4 274.32 0)
 			(effects
 				(font
@@
 		)
 		(property "Datasheet" ""
-			(at 25.4 275 0)
+			(at 25.4 274.32 0)
 			(effects
 				(font
@@
 			)
 		)
-		(property "Description" "Owl logo with laser eyes (graphic only, no pins); keeps the board logo through F8"
-			(at 25.4 275 0)
+		(property "Description" "Owl logo with laser eyes; pin 1 = exposed-copper eyes and beams, tied to GND; keeps the board logo through F8"
+			(at 25.4 274.32 0)
 			(effects
 				(font
@@
 			)
 		)
+		(pin "1"
+		)
 		(instances
 			(project "LaserDriver"
@@
 					(unit 1)
 				)
+			)
+		)
+	)
+	(symbol
+		(lib_id "power:GND")
+		(at 25.4 284.48 0)
+		(unit 1)
+		(exclude_from_sim no)
+		(in_bom yes)
+		(on_board yes)
+		(dnp no)
+		(property "Reference" "#PWR0924"
+			(at 25.4 290.83 0)
+			(effects
+				(font
+					(size 1.27 1.27)
+				)
+				(hide yes)
+			)
+		)
+		(property "Value" "GND"
+			(at 25.5143 288.8044 0)
+			(effects
+				(font
+					(size 1.27 1.27)
+				)
+			)
+		)
+		(property "Footprint" ""
+			(at 25.4 284.48 0)
+			(effects
+				(font
+					(size 1.27 1.27)
+				)
+			)
+		)
+		(property "Datasheet" ""
+			(at 25.4 284.48 0)
+			(effects
+				(font
+					(size 1.27 1.27)
+				)
+			)
+		)
+		(property "Description" "Power symbol creates a global label with name \"GND\" , ground"
+			(at 25.4 284.48 0)
+			(effects
+				(font
+					(size 1.27 1.27)
+				)
+				(hide yes)
+			)
+		)
+		(pin "1"
+		)
+		(instances
+			(project "LaserDriver"
+				(path "/e63e39d7-6ac0-4ffd-8aa3-1841a4541b55"
+					(reference "#PWR0924")
+					(unit 1)
+				)

Commit message: LaserHAT + LaserDaughter: one verified "LCSC Part #" field per part for the Fabrication Toolkit
The schematics carried Rev 1 fields under four spellings ("LCSC Part #", "LCSC Part#",
"LCSC Parth#", "LCSC Part") with stale codes (every 0402 resistor = 47k, TLV2371 = AP2171,
74LVC2G17 = SI3134, zeners = SS14, DMMT5401 = MT3608 ...), which is what the toolkit's BOM showed.

- tools/lcsc_parts.py: every code re-verified against LCSC/JLC (MPN, package, value); LEDs to JLC
  basic KT-0603 (D5 white C2290, D7/D9 red C2286; was extended C5336487), R13 3k -> 2k basic,
  U1 CAT24C32 (out of stock) -> M24C32-WDW6TP C283445 (TSSOP-8, pin-compatible), U5 AP2171
  -> the WG-7 SOT-25 variant C110466 (32k in stock vs 250); VALUES table for the changed parts
- tools/stamp_lcsc.py: writes the table into one "LCSC Part #" field per symbol (text patch of
  the KiCad 9 sheets) and footprint (pcbnew), removes the misspelt variants, sets the Values;
  make_laser_daughter.py stamps its output so the laser sheet stays correct on regeneration
- jlc_fab.py warns when a board field disagrees with the table
- both schematics + boards stamped; ERC/DRC unchanged, path_check 0 mismatches; fab outputs
  regenerated; HAT board backup in stash/LaserDriver_user_2026-09-30_pre-lcsc.kicad_pcb

Co-Authored-By: Claude Fable 5.1 <noreply@anthropic.com>
Claude-Session: https://claude.ai/code/session_018vgLizGzYPynnY93ajvoVA
Parts:
- D5: LCSC Part # C5336487 -> C2290
- D7: LCSC Part # C5336487 -> C2286
- R13: value 3k -> 2k; LCSC Part # C131360 -> C4109
- R15: LCSC Part # C25087 -> C4109
- R19, R20: LCSC Part # (none) -> C25900
- U1: value CAT24C32 -> M24C32-WDW6TP; LCSC Part # C94264 -> C283445
Changed lines of the file:
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@@
 			)
 		)
-		(property "LCSC Part #" "C5336487"
+		(property "LCSC Part #" "C2290"
 			(at 275.59 127 90)
 			(effects
@@
 			)
 		)
+		(property "LCSC Part #" "C25900"
+			(at 271.78 185.42 0)
+			(effects
+				(font
+					(size 1.27 1.27)
+				)
+				(hide yes)
+			)
+		)
 		(pin "1"
 		)
@@
 			)
 		)
-		(property "Value" "CAT24C32"
+		(property "Value" "M24C32-WDW6TP"
 			(at 87.63 184.5245 0)
 			(effects
@@
 			)
 		)
-		(property "LCSC Part #" "C94264"
+		(property "LCSC Part #" "C283445"
 			(at 81.28 177.8 0)
 			(effects
@@
 			)
 		)
-		(property "LCSC Part #" "C25087"
+		(property "LCSC Part #" "C4109"
 			(at 300.99 140.97 0)
 			(effects
@@
 			)
 		)
+		(property "LCSC Part #" "C25900"
+			(at 256.54 185.42 0)
+			(effects
+				(font
+					(size 1.27 1.27)
+				)
+				(hide yes)
+			)
+		)
 		(pin "1"
 		)
@@
 			)
 		)
-		(property "Value" "3k"
+		(property "Value" "2k"
 			(at 278.13 142.2399 0)
 			(effects
@@
 			)
 		)
-		(property "LCSC Part #" "C131360"
+		(property "LCSC Part #" "C4109"
 			(at 275.59 140.97 0)
 			(effects
@@
 			)
 		)
-		(property "LCSC Part #" "C5336487"
+		(property "LCSC Part #" "C2286"
 			(at 300.99 127 90)
 			(effects

Commit message: Fab flags: DNP = not populated, hand-fitted = no part number + exclude from position files
The schematic DNP attribute had been doing double duty ("JLC doesn't place it" for the Pi header,
BNCs and the laser-diode socket, and "not fitted"). KiCad has a flag for each:
- lcsc_parts.NOT_FITTED -> symbol DNP (schematic, carried to the board): HAT R1/R2, the ID_SD/ID_SC
  pull-ups the Pi already provides
- lcsc_parts.HAND_FIT -> DNP cleared, no "LCSC Part #", footprint attribute "exclude from position
  files" (board-only): HAT J1/J6/J7/J8/J9/SW8, laser J1/J2/J3/J5, e-stim J1/J8/J9. They stay in the
  Fabrication Toolkit BOM with an empty number, which JLC's upload shows as "do not place".
stamp_lcsc.py applies both (e-stim board: flags only, its own "LCSC" fields untouched);
jlc_fab.py lists "Hand-fitted" and "Not fitted (DNP)" separately and accepts the toolkit's field
names. HAT now 42 placements / 28 unique. ERC/DRC/path_check unchanged; fab outputs regenerated.

Co-Authored-By: Claude Fable 5.1 <noreply@anthropic.com>
Claude-Session: https://claude.ai/code/session_018vgLizGzYPynnY93ajvoVA
Parts:
- J1: LCSC Part # C42411761 -> (none); now fitted
- R1, R2: now not fitted
Changed lines of the file:
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@@
 		(in_bom yes)
 		(on_board yes)
-		(dnp yes)
+		(dnp no)
 		(property "Reference" "J1"
 			(at 67.31 22.4598 0)
@@
 		)
 		(property "Description" "Generic connector, double row, 02x20, odd/even pin numbering scheme (row 1 odd numbers, row 2 even numbers), script generated (kicad-library-utils/schlib/autogen/connector/)"
-			(at 66.04 50.8 0)
-			(effects
-				(font
-					(size 1.27 1.27)
-				)
-				(hide yes)
-			)
-		)
-		(property "LCSC Part #" "C42411761"
 			(at 66.04 50.8 0)
 			(effects
@@
 		(in_bom yes)
 		(on_board yes)
-		(dnp no)
+		(dnp yes)
 		(property "Reference" "R1"
 			(at 95.4786 169.037 0)
@@
 		(in_bom yes)
 		(on_board yes)
-		(dnp no)
+		(dnp yes)
 		(property "Reference" "R2"
 			(at 103.0986 169.037 0)

Commit message: BOM clean-up: one line per part, non-parts excluded, SW10 shield pads unnumbered
- Values unified where the same LCSC part had two spellings (HAT R3 "47k 1%" -> "47k";
  laser R1-R5 drop the " 1%"), so the Fabrication Toolkit merges them into one BOM line
- lcsc_parts.NON_PARTS (solder jumpers, mounting holes, logo, laser J4/TP1): symbol
  "exclude from BOM" + footprint exclude-from-BOM/-position-files, so they no longer show up
  as BOM lines without a part number
- SW10 (MSK12C02) footprint: the four "SH" shield pads are unnumbered now (library + board),
  which removes the F8 warning "no pin SH in symbol"
- verified by running the Fabrication Toolkit's ProcessManager headlessly on both boards:
  HAT 36 BOM lines / 42 CPL rows, laser 24 / 23; ERC, DRC and path_check unchanged

Co-Authored-By: Claude Fable 5.1 <noreply@anthropic.com>
Claude-Session: https://claude.ai/code/session_018vgLizGzYPynnY93ajvoVA
Parts:
- JP1, JP4, JP5: now left out of the parts list
Changed lines of the file:
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@@
 		(unit 1)
 		(exclude_from_sim no)
-		(in_bom yes)
+		(in_bom no)
 		(on_board yes)
 		(dnp no)
@@
 		(unit 1)
 		(exclude_from_sim no)
-		(in_bom yes)
+		(in_bom no)
 		(on_board yes)
 		(dnp no)
@@
 		(unit 1)
 		(exclude_from_sim no)
-		(in_bom yes)
-		(on_board yes)
-		(dnp no)
+		(in_bom no)
+		(on_board yes)
+		(dnp no)
