File: LaserHAT/mspm0_controller.kicad_sch (KiCad schematic)
At the start: 6 parts

Commit message: Updates with lots of manual work
Parts:
- removed C_MCU1, C_MCU2, C_VDDA: 100nF, Capacitor_SMD:C_0402_1005Metric, symbol Device:C
- removed C_MCU3: 10µF, Capacitor_SMD:C_0805_2012Metric, symbol Device:C
- removed C_VDDA2: 1µF, Capacitor_SMD:C_0402_1005Metric, symbol Device:C
- removed U_MCU: MSPM0G3507RGZR, Package_DFN_QFN:QFN-64-1EP_9x9mm_P0.5mm_EP6.45x6.45mm, symbol MCU_TI_MSPM0:MSPM0G3507RGZR
- added C1: 100nF, Capacitor_SMD:C_0402_1005Metric, symbol Device:C_Small
- added C2: 10uF, Capacitor_SMD:C_0805_2012Metric, symbol Device:C_Small
- added C3: 10nF, Capacitor_SMD:C_0402_1005Metric, symbol Device:C_Small
- added C4: 0.47uF, Capacitor_SMD:C_0603_1608Metric, symbol Device:C_Small
- added IC1: MSPM0G3507SPTR, QFP50P900X900X160-48N, symbol ELEC327-Kicad:MSPM0G3507SPTR
- added R3: 47K, symbol Device:R
- added R4: 100K 0.1%, symbol Device:R
- added SW1, SW2, SW3, SW4, SW5: B, Button_Switch_SMD:SW_SPST_TS-1088-xR020, symbol Switch:SW_Push
- added SW6: BSL, Button_Switch_SMD:SW_SPST_TS-1088-xR020, symbol Switch:SW_Push
- added U5: AP2171W, Package_TO_SOT_SMD:SOT-23-5, symbol Power_Management:AP2171W
Connections:
- net PWM_DUMMY: now also IC1.40 (PA22_/_CLK_OUT_/_A0_7)
- net PWM_LASER: now also IC1.16 (PA8)
- new net +3.3V: U5.5 (IN)
- new net BUTTON1: IC1.9 (PA3_/_COMP1_OUT_/_LFXIN), SW1.1
- new net BUTTON2: IC1.10 (PA4_/_LFCLK_IN_/_LFXOUT), SW2.1
- new net BUTTON3: IC1.11 (PA5_/_HFXIN_/_FCC_IN), SW3.1
- new net BUTTON4: IC1.12 (PA6_/_HFCLK_IN_/_HFXOUT), SW4.1
- new net BUTTON5: IC1.13 (PA7_/_CLK_OUT), SW5.1
- new net GND: C1.2, C2.2, C3.2, C4.2, IC1.7 (VSS), R4.2, U5.2 (GND)
- new net LASER_BOOST_EN: IC1.29 (PA14_/_CLK_OUT_/A0_12)
- new net MCU_POWER_EN: U5.4 (EN)
- new net MCU_UART_RX: IC1.19 (PA11)
- new net MCU_UART_TX: IC1.18 (PA10_/_CLK_OUT)
- new net MSPM0_3v3: C1.1, C2.1, IC1.6 (VDD), R3.1, SW1.2, SW2.2, SW3.2, SW4.2, SW5.2, SW6.2, U5.1 (OUT)
- new net MSPM0_ADC: IC1.47 (PA27_/_RTC_OUT_/_A0_0)
- new net MSPM0_BSL_INVOKE: IC1.33 (PA18_/_A1_3), SW6.1
- new net MSPM0_DAC: IC1.30 (PA15_/_A1_0/DAC_OUT)
- new net MSPM0_NRST: C3.1, IC1.4 (NRST), R3.2
- new net MSPM0_SWCLK: IC1.35 (PA20_/_SWCLK)
- new net MSPM0_SWDIO: IC1.34 (PA19_/_SWDIO)
- new net ROSC: IC1.8 (PA2_/_ROSC), R4.1
- new net STIM_MIRROR: IC1.31 (PA16_/_A1_1_/FCC_IN)
- new net STIM_TRIGGER: IC1.32 (PA17_/_A1_2)
- new net VCORE: C4.1, IC1.48 (VCORE)

Commit message: Updates to design, finalized PCB layout
Parts:
- removed SW5: B, Button_Switch_SMD:SW_SPST_TS-1088-xR020, symbol Switch:SW_Push
- added U7: MSPM0G3507SRHBR, VQFN32_RHB_TEX, symbol ELEC327-Kicad:MSPM0G3507SRHBR
- R3, R4: footprint (none) -> Resistor_SMD:R_0402_1005Metric
Connections:
- net BUTTON1: now also U7.7 (PA3/COMP1_OUT/LFXIN)
- net BUTTON2: now also U7.8 (PA4/LFCLK_IN/LFXOUT)
- net BUTTON3: now also U7.9 (PA5/HFXIN/FCC_IN)
- net BUTTON4: now also U7.10 (PA6/HFCLK_IN/HFXOUT)
- net GND: now also U7.5 (VSS)
- net MCU_UART_RX: now also U7.15 (PA11)
- net MCU_UART_TX: now also U7.14 (PA10/CLK_OUT)
- net MSPM0_ADC: now also U7.21 (PA17/A1_2)
- net MSPM0_BSL_INVOKE: now also U7.22 (PA18/A1_3)
- net MSPM0_DAC: now also U7.19 (PA15/A1_0/DAC_OUT)
- net MSPM0_NRST: now also U7.3 (NRST)
- net MSPM0_SWCLK: now also U7.24 (PA20/SWCLK)
- net MSPM0_SWDIO: now also U7.23 (PA19/SWDIO)
- net PWM_DUMMY: now also U7.26 (PA22/CLK_OUT/A0_7)
- net PWM_LASER: now also U7.25 (PA21/A1_7/VREF-)
- net ROSC: now also U7.6 (PA2/ROSC)
- net STIM_MIRROR: now also U7.17 (PA13)
- net STIM_TRIGGER: now also U7.18 (PA14/CLK_OUT/A0_12)
- net VCORE: now also U7.32 (VCORE)
- net +3.3V renamed +3V3
- net BUTTON5: no longer names the net of IC1.13 (PA7_/_CLK_OUT)
- net LASER_BOOST_EN: no longer names the net of IC1.29 (PA14_/_CLK_OUT_/A0_12)
- net MSPM0_3v3 renamed MSPM0_3V3
- net MSPM0_3V3: now also U7.4 (VDD)
