File: LaserHAT/mspm0_controller.kicad_sch (KiCad schematic)
At the start: 14 parts, among them IC1 MSPM0G3507SPTR, SW1 B, SW2 B, SW3 B, SW4 B, SW6 BSL, U5 AP2171W, U7 MSPM0G3507SRHBR

Commit message: Updated project for manufacturing. Should merge branch if/when we get back a working product
Parts:
- C1: LCSC Part # (none) -> C307331
- C2: LCSC Part # (none) -> C95841
- C3: LCSC Part # (none) -> C15195
- C4: footprint Capacitor_SMD:C_0603_1608Metric -> Capacitor_SMD:C_0402_1005Metric; LCSC Part # (none) -> C47339
- R3: value 47K -> 47k 1%; LCSC Part # (none) -> C25792
- R4: value 100K 0.1% -> 100k 0.1%; LCSC Part # (none) -> C844674
- SW1, SW2, SW3, SW4, SW6: LCSC Part # (none) -> C720477; LCSC Part# C720477 -> (none)
- U5: LCSC Part # (none) -> C2680322; LCSC Parth# C2680322 -> (none)
- U7: LCSC Part # (none) -> C20618748; LCSC Part# C20618748 -> (none)
Changed lines of the file:
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@@
 			)
 		)
-		(property "Description" "Unpolarized capacitor, small symbol"
+		(property "Description" "100nF ±10% 50V Ceramic Capacitor X7R 0402"
 			(at 74.93 121.92 0)
 			(effects
@@
 			)
 		)
-		(property "LCSC Part #" ""
+		(property "LCSC Part #" "C307331"
 			(at 74.93 121.92 0)
 			(effects
@@
 			)
 		)
-		(property "Description" "Unpolarized capacitor, small symbol"
+		(property "Description" "10uF ±10% 16V Ceramic Capacitor X7R 0805"
 			(at 85.09 121.92 0)
 			(effects
@@
 			)
 		)
-		(property "LCSC Part #" ""
+		(property "LCSC Part #" "C95841"
 			(at 85.09 121.92 0)
 			(effects
@@
 			)
 		)
-		(property "LCSC Part#" "C720477"
+		(property "LCSC Part #" "C720477"
 			(at 96.52 208.28 0)
 			(effects
@@
 			)
 		)
-		(property "LCSC Part#" "C20618748"
+		(property "LCSC Part #" "C20618748"
 			(at 152.4 236.22 0)
 			(effects
@@
 			)
 		)
-		(property "Description" "Unpolarized capacitor, small symbol"
+		(property "Description" "10nF ±10% 50V Ceramic Capacitor X7R 0402"
 			(at 118.11 134.62 0)
 			(effects
@@
 			)
 		)
-		(property "LCSC Part #" ""
+		(property "LCSC Part #" "C15195"
 			(at 118.11 134.62 0)
 			(effects
@@
 			)
 		)
-		(property "LCSC Part#" "C720477"
+		(property "LCSC Part #" "C720477"
 			(at 96.52 193.04 0)
 			(effects
@@
 			)
 		)
-		(property "LCSC Part#" "C720477"
+		(property "LCSC Part #" "C720477"
 			(at 96.52 185.42 0)
 			(effects
@@
 			)
 		)
-		(property "LCSC Part #" ""
-			(at 234.95 90.17 0)
-			(effects
-				(font
-					(size 1.27 1.27)
-				)
-				(hide yes)
-			)
-		)
 		(pin "27"
 		)
@@
 			)
 		)
-		(property "Value" "100K 0.1%"
+		(property "Value" "100k 0.1%"
 			(at 142.24 124.4599 0)
 			(effects
@@
 			)
 		)
-		(property "Description" "Resistor"
+		(property "Description" "100mW 100kΩ Thin Film Resistor ±25ppm/℃ ±0.1% 0402 Chip Resistor - Surface Mount RoHS"
 			(at 139.7 123.19 0)
 			(effects
@@
 			)
 		)
-		(property "LCSC Part #" ""
+		(property "LCSC Part #" "C844674"
 			(at 139.7 123.19 0)
 			(effects
@@
 			)
 		)
-		(property "LCSC Parth#" "C2680322"
+		(property "LCSC Part #" "C2680322"
 			(at 95.25 82.55 0)
 			(effects
@@
 			)
 		)
-		(property "Value" "47K"
+		(property "Value" "47k 1%"
 			(at 120.65 121.9199 0)
 			(effects
@@
 			)
 		)
-		(property "Description" "Resistor"
+		(property "Description" "47kΩ ±1% 100mW 0402 Thick Film Resistor AEC-Q200"
 			(at 118.11 120.65 0)
 			(effects
@@
 			)
 		)
-		(property "LCSC Part #" ""
+		(property "LCSC Part #" "C25792"
 			(at 118.11 120.65 0)
 			(effects
@@
 			)
 		)
-		(property "LCSC Part#" "C720477"
+		(property "LCSC Part #" "C720477"
 			(at 368.3 97.79 0)
 			(effects
@@
 			)
 		)
-		(property "Footprint" "Capacitor_SMD:C_0603_1608Metric"
+		(property "Footprint" "Capacitor_SMD:C_0402_1005Metric"
 			(at 163.83 121.92 0)
 			(effects
@@
 			)
 		)
-		(property "Description" "Unpolarized capacitor, small symbol"
+		(property "Description" "470nF ±10% 16V Ceramic Capacitor X7R 0402"
 			(at 163.83 121.92 0)
 			(effects
@@
 			)
 		)
-		(property "LCSC Part #" ""
+		(property "LCSC Part #" "C47339"
 			(at 163.83 121.92 0)
 			(effects
@@
 			)
 		)
-		(property "LCSC Part#" "C720477"
+		(property "LCSC Part #" "C720477"
 			(at 96.52 200.66 0)
 			(effects
