File: LaserHAT/usb_uart.kicad_sch (KiCad schematic)
At the start: 6 parts, among them J5 USB_C_Receptacle_USB2.0_16P, U6 CH340N

Commit message: LaserHAT Rev 2: hand-routed HAT, laser + e-stim daughterboards, fab outputs
HAT (LaserHAT/):
- Rev 1 -> Rev 2 schematic migration (tools/rev2_migrate.py): issue #3 fixes,
  OLED bonnet kept, analog stage moved to plug-in daughterboards (J8/J9),
  buffered BNC I/O, USB-C power switch + PFET ideal diode.
- MCU pin map re-optimised for fewest vias: Pi UART on UART1 (PA8/PA9), I2C on
  PA0/PA1 (fail-safe), PWM_A/B on TIMA0 CCP1/CCP3 (PA7/PA12) with FAULT0 on PA6,
  active-low buttons.  Pi header: SWD swapped, NRST <-> MCU_POWER_EN swapped.
- Stable symbol UUIDs so KiCad "Update PCB" never replaces footprints.
- PCB placed and routed by hand; tidied (tools/track_tidy.py), silkscreen
  decluttered (tools/silk_declutter.py).  DRC clean apart from known cosmetic items.
- JLC fab outputs regenerated (fab/LaserHAT).
- CLAUDE.md, REV2_NOTES.md updated; portable Claude memory in claude_memory/.

Daughterboards: LaserDaughter (300 mA laser driver) and EStimDaughter (isolated
e-stim, imported from kbest/estim_module); interface spec in estim_interface/.

Firmware/Pi: `make flash HAT_REV=2` selects the Rev 2 header wiring;
Pi/power_cycle.py takes its power/reset pins from the environment.

Co-Authored-By: Claude Opus 5.5 <noreply@anthropic.com>
Parts:
- removed C5: 100nF, Capacitor_SMD:C_0402_1005Metric, symbol Device:C_Small
- added Q3, Q5: AP30P30Q, Footprints:PDFN3333-8_PMOS_GSD, symbol Transistor_FET:AO3401A
- added Q4: DMMT5401, Package_TO_SOT_SMD:SOT-23-6, symbol Transistor_BJT:DMMT5401
- added R21: 47k, Resistor_SMD:R_0402_1005Metric, symbol Device:R
- added R22: 10k, Resistor_SMD:R_0402_1005Metric, symbol Device:R
- added R26: 100k, Resistor_SMD:R_0402_1005Metric, symbol Device:R
- added SW10: USB PWR, Footprints:SW_SPDT_Shouhan_MSK12C02, symbol Switch:SW_SPDT
Connections:
- net +3V3: now also U6.8 (V3)
- net +5V: now also Q3.2 (S), Q4.5 (E2); no longer J5.A4 (VBUS), J5.A9 (VBUS), J5.B4 (VBUS), J5.B9 (VBUS)
- net GND: now also R21.2, R22.2, SW10.1 (A)
- new net IDEAL_B: Q4.1 (C1), Q4.2 (B1), Q4.3 (B2), R21.1
- new net IDEAL_G: Q3.1 (G), Q4.4 (C2), R22.1
- new net PWR_EN: Q5.1 (G), R26.2, SW10.2 (B)
- new net VBUS: J5.A4 (VBUS), J5.A9 (VBUS), J5.B4 (VBUS), J5.B9 (VBUS), Q5.2 (S), R26.1
- new net VBUS_SW: Q3.3 (D), Q4.6 (E1), Q5.3 (D)
- no-connect marks 0 -> 1
Other:
- note added: "USB power switch: SW10 (right-angle slide, left edge) -> Q5 gate. PWR_EN = GND: Q5 on, USB-C VBUS reaches the ideal diode. Switch OFF: PWR_EN open, R26 pulls it to VBUS, Q5 off. Only cuts HAT USB-C power."
- note added: "USB-C VBUS -> +5V (Pi 5V pins) through a PFET ideal diode: blocks back-feed into the USB host when the Pi has its own supply. A Pi 4 needs a 3 A Type-C source when powered from here."
