File: LaserHAT/usb_uart.kicad_sch (KiCad schematic)
At the start: 12 parts, among them J5 USB_C_Receptacle_USB2.0_16P, Q3 AP30P30Q, Q4 DMMT5401, Q5 AP30P30Q, SW10 USB PWR, U6 CH340N

Commit message: LaserHAT + LaserDaughter: one verified "LCSC Part #" field per part for the Fabrication Toolkit
The schematics carried Rev 1 fields under four spellings ("LCSC Part #", "LCSC Part#",
"LCSC Parth#", "LCSC Part") with stale codes (every 0402 resistor = 47k, TLV2371 = AP2171,
74LVC2G17 = SI3134, zeners = SS14, DMMT5401 = MT3608 ...), which is what the toolkit's BOM showed.

- tools/lcsc_parts.py: every code re-verified against LCSC/JLC (MPN, package, value); LEDs to JLC
  basic KT-0603 (D5 white C2290, D7/D9 red C2286; was extended C5336487), R13 3k -> 2k basic,
  U1 CAT24C32 (out of stock) -> M24C32-WDW6TP C283445 (TSSOP-8, pin-compatible), U5 AP2171
  -> the WG-7 SOT-25 variant C110466 (32k in stock vs 250); VALUES table for the changed parts
- tools/stamp_lcsc.py: writes the table into one "LCSC Part #" field per symbol (text patch of
  the KiCad 9 sheets) and footprint (pcbnew), removes the misspelt variants, sets the Values;
  make_laser_daughter.py stamps its output so the laser sheet stays correct on regeneration
- jlc_fab.py warns when a board field disagrees with the table
- both schematics + boards stamped; ERC/DRC unchanged, path_check 0 mismatches; fab outputs
  regenerated; HAT board backup in stash/LaserDriver_user_2026-09-30_pre-lcsc.kicad_pcb

Co-Authored-By: Claude Fable 5.1 <noreply@anthropic.com>
Claude-Session: https://claude.ai/code/session_018vgLizGzYPynnY93ajvoVA
Parts:
- J5: LCSC Part # C2927038 -> C2988369
- Q3, Q5: LCSC Part # (none) -> C471913
- Q4: LCSC Part # (none) -> C154733
- R21: LCSC Part # (none) -> C25792
- R22: LCSC Part # (none) -> C25744
- R26: LCSC Part # (none) -> C25741
- SW10: LCSC Part # (none) -> C431540
Changed lines of the file:
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@@
+			)
+		)
+		(property "LCSC Part #" "C471913"
+			(at 157.48 40.64 0)
+			(effects
+				(font
+					(size 1.27 1.27)
+				)
+				(hide yes)
 			)
 		)
@@
 			)
 		)
+		(property "LCSC Part #" "C431540"
+			(at 45.72 76.2 0)
+			(effects
+				(font
+					(size 1.27 1.27)
+				)
+				(hide yes)
+			)
+		)
 		(pin "2"
 		)
@@
 			)
 		)
+		(property "LCSC Part #" "C25741"
+			(at 55.88 45.72 0)
+			(effects
+				(font
+					(size 1.27 1.27)
+				)
+				(hide yes)
+			)
+		)
 		(pin "1"
 		)
@@
 					(size 1.27 1.27)
 				)
+			)
+		)
+		(property "LCSC Part #" "C471913"
+			(at 76.2 45.72 0)
+			(effects
+				(font
+					(size 1.27 1.27)
+				)
+				(hide yes)
 			)
 		)
@@
 			)
 		)
-		(property "LCSC Part #" "C2927038"
+		(property "LCSC Part #" "C2988369"
 			(at 107.95 106.68 0)
 			(effects
@@
 			)
 		)
+		(property "LCSC Part #" "C25792"
+			(at 200.66 45.72 0)
+			(effects
+				(font
+					(size 1.27 1.27)
+				)
+				(hide yes)
+			)
+		)
 		(pin "1"
 		)
@@
 					(size 1.27 1.27)
 				)
+			)
+		)
+		(property "LCSC Part #" "C25744"
+			(at 213.36 45.72 0)
+			(effects
+				(font
+					(size 1.27 1.27)
+				)
+				(hide yes)
 			)
 		)
@@
 			)
 		)
+		(property "LCSC Part #" "C154733"
+			(at 175.26 58.42 0)
+			(effects
+				(font
+					(size 1.27 1.27)
+				)
+				(hide yes)
+			)
+		)
 		(pin "3"
 		)
@@
 			)
 		)
+		(property "LCSC Part #" "C154733"
+			(at 139.7 58.42 0)
+			(effects
+				(font
+					(size 1.27 1.27)
+				)
+				(hide yes)
+			)
+		)

Commit message: BOM: descriptions from the LCSC catalog, value verifier and netlist-vs-board check on all three boards
R15 (2k, C4109) still said "200Ω" in its Description: the Rev 1 symbols carried descriptions and
datasheet links of parts long replaced (R13 "1kΩ", D5 "Emerald Green", D7 "Ice Blue", L1 "22uH 6x6",
Rs1 "10Ω", D3 "1N4148", ...). Now:
- tools/lcsc_catalog.json: LCSC MPN, brand, package, description, parameter table (Resistance /
  Capacitance / Inductance ...) and datasheet URL for every code, fetched by tools/lcsc_verify.py
- stamp_lcsc.py writes Description "<MPN> (<brand>, <package>): <LCSC description>" and the LCSC
  datasheet URL into every machine-placed symbol and footprint (HAT + laser)
- tools/lcsc_verify.py: every R/C/L Value must equal LCSC's parameter, other parts' MPN must match
  the Value (label values like "FIRE" are listed, not failed), size codes must match the package;
  covers HAT, laser and the e-stim list (bom_EStimDaughter.csv) and the fields the toolkit reads:
  0 mismatches on all three boards
- tools/sync_check.py: read-only F8 (parts, footprint ids, values, DNP, pad nets, paths vs the
  exported netlist): 0 differences on all three boards after fixing the owl's missing
  "Footprints:" library prefix and the e-stim U5/U8 paths (netlist uses the other unit's uuid;
  backup in stash/EStimDaughter_2026-09-30_pre-unitpath.kicad_pcb)
- values: laser D1/D3 "SS14" -> "DSK14" (the part ordered), HAT J5 -> "GT-USB-7010ASV"
- fab outputs regenerated; ERC/DRC unchanged

Co-Authored-By: Claude Fable 5.1 <noreply@anthropic.com>
Claude-Session: https://claude.ai/code/session_018vgLizGzYPynnY93ajvoVA
Parts:
- J5: value USB_C_Receptacle_USB2.0_16P -> GT-USB-7010ASV
Changed lines of the file:
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@@
 			)
 		)
-		(property "Datasheet" ""
+		(property "Datasheet" "https://datasheet.lcsc.com/datasheet/pdf/741ba14677c88fb4d9f793d97efdadf4.pdf?productCode=C471913"
 			(at 157.48 40.64 0)
 			(effects
@@
 			)
 		)
-		(property "Description" ""
+		(property "Description" "AP30P30Q (ALLPOWER, PDFN3333-8): P-Channel 30V 30A 1.5W Surface Mount PDFN3333-8"
 			(at 157.48 40.64 0)
 			(effects
@@
 			)
 		)
-		(property "Datasheet" "~"
+		(property "Datasheet" "https://datasheet.lcsc.com/datasheet/pdf/02336ea48ea44ca18c72517dd3cb7b47.pdf?productCode=C307331"
 			(at 177.8 87.63 0)
 			(effects
@@
 			)
 		)
-		(property "Description" "100nF ±10% 50V Ceramic Capacitor X7R 0402"
+		(property "Description" "CL05B104KB54PNC (Samsung Electro-Mechanics, 0402): 100nF ±10% 50V Ceramic Capacitor X7R 0402"
 			(at 177.8 87.63 0)
 			(effects
@@
 			)
 		)
-		(property "Datasheet" "~"
+		(property "Datasheet" "https://datasheet.lcsc.com/datasheet/pdf/0a975aaa49b7c97f38a963127be4a823.pdf?productCode=C25905"
 			(at 133.35 99.06 0)
 			(effects
@@
 			)
 		)
-		(property "Description" "5.1kΩ 100mW Thick Film Resistor ±100ppm/℃ ±1% 0402 Chip Resistor - Surface Mount RoHS"
+		(property "Description" "0402WGF5101TCE (UNI-ROYAL, 0402): 5.1kΩ ±1% 62.5mW 0402 Thick Film Resistor"
 			(at 133.35 99.06 0)
 			(effects
@@
 			)
 		)
-		(property "Datasheet" "https://aitendo3.sakura.ne.jp/aitendo_data/product_img/ic/inteface/CH340N/ch340n.pdf"
+		(property "Datasheet" "https://datasheet.lcsc.com/datasheet/pdf/a3b2ca2c7638da2635df3f5b1d90bcc0.pdf?productCode=C2977777"
 			(at 171.45 96.52 0)
 			(effects
@@
 			)
 		)
-		(property "Description" "USB serial converter, 2Mbps, UART, JEITA SOIC-8 (SOP-8)"
+		(property "Description" "CH340N (WCH, SOP-8): 1 USB to serial 2Mbps USB 2.0 SOP-8 Interface Controllers"
 			(at 173.99 101.6 0)
 			(effects
@@
 			)
 		)
-		(property "Datasheet" ""
+		(property "Datasheet" "https://datasheet.lcsc.com/datasheet/pdf/5162155576bfd231c35aa9a893d25c8c.pdf?productCode=C431540"
 			(at 45.72 76.2 0)
 			(effects
@@
 			)
 		)
-		(property "Description" ""
+		(property "Description" "MSK12C02 (SHOU HAN, SMD,8x2.8mm): Slide Switch SPDT 50mA @ 12V Surface Mount, Right Angle 8mm"
 			(at 45.72 76.2 0)
 			(effects
@@
 			)
 		)
-		(property "Datasheet" ""
+		(property "Datasheet" "https://datasheet.lcsc.com/datasheet/pdf/0a975aaa49b7c97f38a963127be4a823.pdf?productCode=C25741"
 			(at 55.88 45.72 0)
 			(effects
@@
 			)
 		)
-		(property "Description" ""
+		(property "Description" "0402WGF1003TCE (UNI-ROYAL, 0402): 100kΩ ±1% 62.5mW 0402 Thick Film Resistor"
 			(at 55.88 45.72 0)
 			(effects
@@
 			)
 		)
-		(property "Datasheet" ""
+		(property "Datasheet" "https://datasheet.lcsc.com/datasheet/pdf/741ba14677c88fb4d9f793d97efdadf4.pdf?productCode=C471913"
 			(at 76.2 45.72 0)
 			(effects
@@
 			)
 		)
-		(property "Description" ""
+		(property "Description" "AP30P30Q (ALLPOWER, PDFN3333-8): P-Channel 30V 30A 1.5W Surface Mount PDFN3333-8"
 			(at 76.2 45.72 0)
 			(effects
@@
 			)
 		)
-		(property "Value" "USB_C_Receptacle_USB2.0_16P"
+		(property "Value" "GT-USB-7010ASV"
 			(at 107.95 86.36 0)
 			(effects
@@
 			)
 		)
-		(property "Datasheet" "https://www.usb.org/sites/default/files/documents/usb_type-c.zip"
+		(property "Datasheet" "https://datasheet.lcsc.com/datasheet/pdf/a1d5a66cf718dd88763ab794dba802b2.pdf?productCode=C2988369"
 			(at 111.76 106.68 0)
 			(effects
@@
 			)
 		)
-		(property "Description" "USB 2.0-only 16P Type-C Receptacle connector"
+		(property "Description" "GT-USB-7010ASV (G-Switch, SMD): USB-C (USB TYPE-C) Receptacle Connector 16 Position Surface Mount, Right Angle"
 			(at 107.95 106.68 0)
 			(effects
@@
 			)
 		)
-		(property "Datasheet" ""
+		(property "Datasheet" "https://datasheet.lcsc.com/datasheet/pdf/0a975aaa49b7c97f38a963127be4a823.pdf?productCode=C25792"
 			(at 200.66 45.72 0)
 			(effects
@@
 			)
 		)
-		(property "Description" ""
+		(property "Description" "0402WGF4702TCE (UNI-ROYAL, 0402): 47kΩ ±1% 62.5mW 0402 Thick Film Resistor"
 			(at 200.66 45.72 0)
 			(effects
@@
 			)
 		)
-		(property "Datasheet" ""
+		(property "Datasheet" "https://datasheet.lcsc.com/datasheet/pdf/0a975aaa49b7c97f38a963127be4a823.pdf?productCode=C25744"
 			(at 213.36 45.72 0)
 			(effects
@@
 			)
 		)
-		(property "Description" ""
+		(property "Description" "0402WGF1002TCE (UNI-ROYAL, 0402): 10kΩ ±1% 62.5mW 0402 Thick Film Resistor"
 			(at 213.36 45.72 0)
 			(effects
@@
 			)
 		)
-		(property "Datasheet" ""
+		(property "Datasheet" "https://datasheet.lcsc.com/datasheet/pdf/05b35e50c47741f69d8631d18fa1a261.pdf?productCode=C154733"
 			(at 175.26 58.42 0)
 			(effects
@@
 			)
 		)
-		(property "Description" ""
+		(property "Description" "DMMT5401-7-F (DIODES, SOT-26(SC74R)): Bipolar (BJT) Transistor PNP 150V 200mA 300MHz 300mW Surface Mount SOT-26(SC74R)"
 			(at 175.26 58.42 0)
 			(effects
@@
 			)
 		)
-		(property "Datasheet" "~"
+		(property "Datasheet" "https://datasheet.lcsc.com/datasheet/pdf/0a975aaa49b7c97f38a963127be4a823.pdf?productCode=C25905"
 			(at 127 96.52 0)
 			(effects
@@
 			)
 		)
-		(property "Description" "5.1kΩ 100mW Thick Film Resistor ±100ppm/℃ ±1% 0402 Chip Resistor - Surface Mount RoHS"
+		(property "Description" "0402WGF5101TCE (UNI-ROYAL, 0402): 5.1kΩ ±1% 62.5mW 0402 Thick Film Resistor"
 			(at 127 96.52 0)
 			(effects
@@
 			)
 		)
-		(property "Datasheet" ""
+		(property "Datasheet" "https://datasheet.lcsc.com/datasheet/pdf/05b35e50c47741f69d8631d18fa1a261.pdf?productCode=C154733"
 			(at 139.7 58.42 0)
 			(effects
@@
 			)
 		)
-		(property "Description" ""
+		(property "Description" "DMMT5401-7-F (DIODES, SOT-26(SC74R)): Bipolar (BJT) Transistor PNP 150V 200mA 300MHz 300mW Surface Mount SOT-26(SC74R)"
 			(at 139.7 58.42 0)
 			(effects

Commit message: LaserHAT: SW8 BACK -> Panasonic EVQP7A01P side-actuated SMD (C79167); Values = part numbers; stamp clears flags
- SW8: schematic footprint Button_Switch_SMD:SW_SPST_EVQP7A; board footprint swapped at the south
  edge (111.55, 98.25), body flush with the edge, button ~0.35 mm proud; BUTTON1 via at the old
  THT pin joins the hand-routed B.Cu run, pad-1 pair bridged; GND pads on the pour. DRC identical
  to before the swap, 0 unconnected; backup stash/LaserDriver_user_2026-09-30_pre-sw8smd.kicad_pcb
- stamp_lcsc.py now also clears DNP / exclude flags on machine-placed parts (SW8 had stayed
  excluded after the previous commit, which wrongly claimed 43 placements)
- Values of LEDs and switches are the part numbers (KT-0603R/W, TS-1088-AR02016, MSK12C02,
  BL-DT, EVQP7A01P, PCM12SMTR) so JLC's BOM matcher sees one part per line; the function names
  remain as silkscreen texts
- verified: lcsc_verify 0 mismatches, sync_check 0 differences (HAT, laser), toolkit BOM/CPL
  consistent in both DNP modes (HAT 29 lines / 43 placements); fab outputs regenerated; docs

Co-Authored-By: Claude Fable 5.1 <noreply@anthropic.com>
Claude-Session: https://claude.ai/code/session_018vgLizGzYPynnY93ajvoVA
Parts:
- SW10: value USB PWR -> MSK12C02
Changed lines of the file:
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@@
 			)
 		)
-		(property "Value" "USB PWR"
+		(property "Value" "MSK12C02"
 			(at 48.26 78.74 0)
 			(effects
