File: LaserHAT/LaserDriver.kicad_pcb (KiCad board)
At the start: 2 copper layers, 65 x 56.9 mm, 58 parts, among them J1 GPIO, J5 USB_C_Receptacle_USB2.0_16P, J6 BNC TRIGGER IN, J7 BNC STIM OUT, J8 DB_POWER_TIMING, J9 DB_ANALOG, Q3 AP30P30Q, Q4 DMMT5401, Q5 AP30P30Q, SW10 USB PWR, SW6 BSL, SW7 BL-DT (LCSC C53223909), SW8 BACK, SW9 FIRE, U1 CAT24C32, U4 MCP1700x-330xxMB, U5 AP2171W, U6 CH340N, U7 MSPM0G3507SRHBR, U8 74LVC2G17

Commit message: LaserHAT: draw the e-stim module outline (26.5 x 33 mm, y 76-109) on User.Drawings
Four 0.1 mm lines matching EStimDaughter's Edge.Cuts in HAT coordinates, plus labels for
the e-stim and laser module rectangles. Notes updated (REV2_NOTES, spec §7, claude_memory).

Co-Authored-By: Claude Fable 5.1 <noreply@anthropic.com>
Claude-Session: https://claude.ai/code/session_018vgLizGzYPynnY93ajvoVA
Other:
- board text added: "E-STIM MODULE 26.5 x 33 mm (overhangs the HAT edge to y 109)"
- board text added: "LASER MODULE 26.5 x 23.5 mm"
Changed lines of the file:
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@@
+		(layer "Dwgs.User")
+	)
+	(gr_line
+		(start 101 109)
+		(end 101 76)
+		(stroke
+			(width 0.1)
+			(type default)
+		)
 		(layer "Dwgs.User")
 	)
@@
 	)
 	(gr_line
+		(start 127.5 76)
+		(end 127.5 109)
+		(stroke
+			(width 0.1)
+			(type default)
+		)
+		(layer "Dwgs.User")
+	)
+	(gr_line
 		(start 127.5 99.5)
 		(end 101 99.5)
+		(stroke
+			(width 0.1)
+			(type default)
+		)
+		(layer "Dwgs.User")
+	)
+	(gr_line
+		(start 127.5 109)
+		(end 101 109)
 		(stroke
 			(width 0.1)
@@
 		)
 	)
+	(gr_text "LASER MODULE 26.5 x 23.5 mm"
+		(at 114.25 98 0)
+		(layer "Dwgs.User")
+		(effects
+			(font
+				(size 0.8 0.8)
+				(thickness 0.12)
+			)
+		)
+	)
+	(gr_text "E-STIM MODULE 26.5 x 33 mm (overhangs the HAT edge to y 109)"
+		(at 114.25 107 0)
+		(layer "Dwgs.User")
+		(effects
+			(font
+				(size 0.8 0.8)
+				(thickness 0.12)
+			)
+		)
+	)
