File: LaserHAT/LaserDriver.kicad_pcb (KiCad board)
At the start: 2 copper layers, 65 x 56.9 mm, 58 parts, among them J1 GPIO, J5 USB_C_Receptacle_USB2.0_16P, J6 BNC TRIGGER IN, J7 BNC STIM OUT, J8 DB_POWER_TIMING, J9 DB_ANALOG, Q3 AP30P30Q, Q4 DMMT5401, Q5 AP30P30Q, SW10 USB PWR, SW6 BSL, SW7 BL-DT (LCSC C53223909), SW8 BACK, SW9 FIRE, U1 CAT24C32, U4 MCP1700x-330xxMB, U5 AP2171W, U6 CH340N, U7 MSPM0G3507SRHBR, U8 74LVC2G17

Commit message: Small shifts on PCB and updated version of schematic
Parts:
- moved C16 1.03 mm to (147.7, 64.4), turned to 0 degrees
Other:
- board text added: "2.0"
- board text added: "GLANCE HAT"
- board text added: "KemereLab.org"
- board text removed: "GLANCE HAT 2.0 Kemere Lab"
Changed lines of the file:
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@@
 		(tags "solder jumper open")
 		(property "Reference" "JP5"
-			(at 0 1.905 0)
+			(at -3.55 -0.05 0)
 			(layer "F.SilkS")
 			(effects
@@
 	(footprint "Capacitor_SMD:C_0402_1005Metric"
 		(layer "F.Cu")
-		(at 146.65 64.3 180)
+		(at 147.68 64.4)
 		(descr "Capacitor SMD 0402 (1005 Metric), square (rectangular) end terminal, IPC-7351 nominal, (Body size source: IPC-SM-782 page 76, https://www.pcb-3d.com/wordpress/wp-content/uploads/ipc-sm-782a_amendment_1_and_2.pdf), generated with kicad-footprint-generator")
 		(tags "capacitor")
@@
 		)
 		(property "LCSC Part #" "C307331"
-			(at 0 0 180)
+			(at 0 0 0)
 			(unlocked yes)
 			(layer "F.Fab")
@@
 		)
 		(property "LCSC Part#" "C77020"
-			(at 0 0 180)
+			(at 0 0 0)
 			(unlocked yes)
 			(layer "F.Fab")
@@
 		(attr smd)
 		(fp_line
-			(start -0.107836 0.36)
-			(end 0.107836 0.36)
+			(start -0.107836 -0.36)
+			(end 0.107836 -0.36)
 			(stroke
 				(width 0.12)
@@
 		)
 		(fp_line
-			(start -0.107836 -0.36)
-			(end 0.107836 -0.36)
+			(start -0.107836 0.36)
+			(end 0.107836 0.36)
 			(stroke
 				(width 0.12)
@@
 		)
 		(pad "1" smd roundrect
-			(at -0.48 0 180)
+			(at -0.48 0)
 			(size 0.56 0.62)
 			(layers "F.Cu" "F.Mask" "F.Paste")
@@
 		)
 		(pad "2" smd roundrect
-			(at 0.48 0 180)
+			(at 0.48 0)
 			(size 0.56 0.62)
 			(layers "F.Cu" "F.Mask" "F.Paste")
@@
 	(footprint "Resistor_SMD:R_0402_1005Metric"
 		(layer "F.Cu")
-		(at 159.6875 81.2 180)
+		(at 159.7 81.2 180)
 		(descr "Resistor SMD 0402 (1005 Metric), square (rectangular) end terminal, IPC-7351 nominal, (Body size source: IPC-SM-782 page 72, https://www.pcb-3d.com/wordpress/wp-content/uploads/ipc-sm-782a_amendment_1_and_2.pdf), generated with kicad-footprint-generator")
 		(tags "resistor")
@@
 	(footprint "Diode_SMD:D_0603_1608Metric"
 		(layer "F.Cu")
-		(at 162.5875 81.2)
+		(at 162.6 81.2)
 		(descr "Diode SMD 0603 (1608 Metric), square (rectangular) end terminal, IPC-7351 nominal, (Body size source: http://www.tortai-tech.com/upload/download/2011102023233369053.pdf), generated with kicad-footprint-generator")
 		(tags "diode")
@@
 			)
 		)
-		(property "Description" ""
+		(property "Description" "Owl logo with laser eyes (graphic only, no pins); keeps the board logo through F8"
 			(at 0 0 0)
 			(layer "F.Fab")
@@
 		(tags "solder jumper open")
 		(property "Reference" "JP1"
-			(at -3 0 0)
+			(at 3.7 -0.6 0)
 			(layer "F.SilkS")
 			(effects
@@
 		(sheetname "/")
 		(sheetfile "LaserDriver.kicad_sch")
-		(attr smd)
+		(attr smd dnp)
 		(fp_line
 			(start -3.92 1.38)
@@
 		(layer "Edge.Cuts")
 	)
-	(gr_text "~{R}"
-		(at 120.5 45 0)
+	(gr_text "USB RST"
+		(at 123.775 69.075 0)
 		(layer "F.SilkS")
 		(effects
 			(font
-				(size 1 1)
+				(size 0.8 0.8)
 				(thickness 0.15)
 			)
-			(justify left bottom)
 		)
 	)
-	(gr_text "SK"
-		(at 127.75 45 0)
+	(gr_text "EEPROM WP"
+		(at 142.5 59.074999 0)
 		(layer "F.SilkS")
 		(effects
 			(font
-				(size 1 1)
+				(size 0.8 0.8)
 				(thickness 0.15)
 			)
-			(justify left bottom)
 		)
 	)
-	(gr_text "SD"
-		(at 132.75 45 0)
+	(gr_text "STANDALONE"
+		(at 124.8 51.2 0)
 		(layer "F.SilkS")
 		(effects
 			(font
-				(size 1 1)
+				(size 0.8 0.8)
 				(thickness 0.15)
+				(bold yes)
 			)
-			(justify left bottom)
 		)
 	)
-	(gr_text "(c)2026.9"
-		(at 148.25 51.5 0)
+	(gr_text "~{R}"
+		(at 120.5 45 0)
 		(layer "F.SilkS")
 		(effects
@@
 		)
 	)
-	(gr_text "OUTPUT MODULE"
-		(at 116 88 0)
+	(gr_text "SK"
+		(at 127.75 45 0)
 		(layer "F.SilkS")
 		(effects
@@
 				(thickness 0.15)
 			)
+			(justify left bottom)
 		)
 	)
-	(gr_text "USB RST"
-		(at 123.775 69.075 0)
+	(gr_text "SD"
+		(at 132.75 45 0)
 		(layer "F.SilkS")
 		(effects
@@
 				(thickness 0.15)
 			)
+			(justify left bottom)
 		)
 	)
-	(gr_text "EEPROM WP"
-		(at 142.5 59.074999 0)
+	(gr_text "(c)2026.9"
+		(at 150.6 54.8 0)
 		(layer "F.SilkS")
 		(effects
@@
 				(thickness 0.15)
 			)
+			(justify left bottom)
 		)
 	)
-	(gr_text "PWR"
-		(at 107 74.75 0)
+	(gr_text "OUTPUT MODULE"
+		(at 116 88 0)
 		(layer "F.SilkS")
 		(effects
@@
 				(thickness 0.15)
 			)
-			(justify right)
 		)
 	)
@@
 		)
 	)
-	(gr_text "GLANCE HAT\n2.0\nKemere Lab"
-		(at 152.25 57.75 0)
+	(gr_text "KemereLab.org"
+		(at 152.2 56.6 0)
 		(layer "F.SilkS")
 		(effects
 			(font
 				(size 1.1 1.1)
-				(thickness 0.275)
+				(thickness 0.2)
 				(bold yes)
 			)
@@
 		)
 	)
-	(gr_text "TRIG IN"
-		(at 135.3 77.5 0)
-		(layer "F.SilkS")
-		(effects
-			(font
-				(size 1.25 1.25)
-				(thickness 0.175)
-			)
-		)
-	)
 	(gr_text "BSL"
-		(at 145.25 74.75 90)
+		(at 134.4 75.6 0)
 		(layer "F.SilkS")
 		(effects
@@
 		)
 	)
-	(gr_text "STANDALONE"
-		(at 123 50.75 0)
+	(gr_text "PWR"
+		(at 108.8 74.8 0)
 		(layer "F.SilkS")
 		(effects
@@
 				(thickness 0.21)
 			)
+			(justify right)
 		)
 	)
-	(gr_text "STIM OUT"
-		(at 150.6 77.5 0)
+	(gr_text "MCU"
+		(at 163.5 74.8 0)
 		(layer "F.SilkS")
 		(effects
@@
 				(thickness 0.21)
 			)
+			(justify right)
 		)
 	)
-	(gr_text "MCU"
-		(at 163.5 75 0)
+	(gr_text "STIM"
+		(at 163.75 79.5 0)
 		(layer "F.SilkS")
 		(effects
@@
 		)
 	)
-	(gr_text "STIM"
-		(at 163.75 79.5 0)
+	(gr_text "FIRE"
+		(at 159.6 89 90)
 		(layer "F.SilkS")
 		(effects
@@
 				(thickness 0.21)
 			)
-			(justify right)
 		)
 	)
-	(gr_text "FIRE"
-		(at 159.6 89 90)
+	(gr_text "TRIG IN"
+		(at 135.3 78 0)
 		(layer "F.SilkS")
 		(effects
 			(font
 				(size 1.5 1.5)
-				(thickness 0.21)
+				(thickness 0.25)
+				(bold yes)
+			)
+		)
+	)
+	(gr_text "TRIG IN"
+		(at 135.3 97.6 0)
+		(layer "F.SilkS")
+		(effects
+			(font
+				(size 1.5 1.5)
+				(thickness 0.25)
+				(bold yes)
+			)
+		)
+	)
+	(gr_text "STIM OUT"
+		(at 150.6 78 0)
+		(layer "F.SilkS")
+		(effects
+			(font
+				(size 1.5 1.5)
+				(thickness 0.25)
+				(bold yes)
+			)
+		)
+	)
+	(gr_text "STIM OUT"
+		(at 150.6 97.6 0)
+		(layer "F.SilkS")
+		(effects
+			(font
+				(size 1.5 1.5)
+				(thickness 0.25)
+				(bold yes)
 			)
 		)
 	)
+	(gr_text "GLANCE\nHAT\n"
+		(at 142.8 64.6 0)
+		(layer "F.SilkS")
+		(effects
+			(font
+				(size 1.5 1.5)
+				(thickness 0.275)
+				(bold yes)
+			)
+			(justify left bottom)
+		)
+	)
+	(gr_text "2.0"
+		(at 152 72.4 0)
+		(layer "F.SilkS")
+		(effects
+			(font
+				(size 1.5 1.5)
+				(thickness 0.275)
+				(bold yes)
+			)
+			(justify left bottom)
+		)
+	)
 	(gr_text "CK SDG"
 		(at 150.75 98 0)
@@
 	)
 	(segment
-		(start 160.1975 81.2)
-		(end 161.75 81.25)
+		(start 160.21 81.2)
+		(end 161.8125 81.2)
 		(width 0.15)
 		(layer "F.Cu")
