File: LaserHAT/LaserDriver.kicad_pcb (KiCad board)
At the start: 2 copper layers, 65 x 56.9 mm, 58 parts, among them J1 GPIO, J5 USB_C_Receptacle_USB2.0_16P, J6 BNC TRIGGER IN, J7 BNC STIM OUT, J8 DB_POWER_TIMING, J9 DB_ANALOG, Q3 AP30P30Q, Q4 DMMT5401, Q5 AP30P30Q, SW10 USB PWR, SW6 BSL, SW7 BL-DT (LCSC C53223909), SW8 BACK, SW9 FIRE, U1 M24C32-WDW6TP, U4 MCP1700x-330xxMB, U5 AP2171W, U6 CH340N, U7 MSPM0G3507SRHBR, U8 74LVC2G17

Commit message: BOM clean-up: one line per part, non-parts excluded, SW10 shield pads unnumbered
- Values unified where the same LCSC part had two spellings (HAT R3 "47k 1%" -> "47k";
  laser R1-R5 drop the " 1%"), so the Fabrication Toolkit merges them into one BOM line
- lcsc_parts.NON_PARTS (solder jumpers, mounting holes, logo, laser J4/TP1): symbol
  "exclude from BOM" + footprint exclude-from-BOM/-position-files, so they no longer show up
  as BOM lines without a part number
- SW10 (MSK12C02) footprint: the four "SH" shield pads are unnumbered now (library + board),
  which removes the F8 warning "no pin SH in symbol"
- verified by running the Fabrication Toolkit's ProcessManager headlessly on both boards:
  HAT 36 BOM lines / 42 CPL rows, laser 24 / 23; ERC, DRC and path_check unchanged

Co-Authored-By: Claude Fable 5.1 <noreply@anthropic.com>
Claude-Session: https://claude.ai/code/session_018vgLizGzYPynnY93ajvoVA
Parts:
- R3: value 47k 1% -> 47k
Changed lines of the file:
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@@
 		(sheetfile "LaserDriver.kicad_sch")
 		(zone_connect 1)
-		(attr exclude_from_pos_files allow_soldermask_bridges)
+		(attr exclude_from_pos_files exclude_from_bom allow_soldermask_bridges)
 		(fp_rect
 			(start -0.15 -0.75)
@@
 			)
 		)
+		(pad "" smd roundrect
+			(at -3.675 -1.1 270)
+			(size 1.05 0.7)
+			(layers "F.Cu" "F.Mask" "F.Paste")
+			(roundrect_rratio 0.25)
+		)
+		(pad "" smd roundrect
+			(at -3.675 1.1 270)
+			(size 1.05 0.7)
+			(layers "F.Cu" "F.Mask" "F.Paste")
+			(roundrect_rratio 0.25)
+		)
 		(pad "" np_thru_hole circle
 			(at -1.5 0 270)
@@
 			(layers "*.Mask")
 		)
+		(pad "" smd roundrect
+			(at 3.675 -1.1 270)
+			(size 1.05 0.7)
+			(layers "F.Cu" "F.Mask" "F.Paste")
+			(roundrect_rratio 0.25)
+		)
+		(pad "" smd roundrect
+			(at 3.675 1.1 270)
+			(size 1.05 0.7)
+			(layers "F.Cu" "F.Mask" "F.Paste")
+			(roundrect_rratio 0.25)
+		)
 		(pad "1" smd roundrect
 			(at -2.25 -1.95 270)
@@
 			(pintype "passive+no_connect")
 		)
-		(pad "SH" smd roundrect
-			(at -3.675 -1.1 270)
-			(size 1.05 0.7)
-			(layers "F.Cu" "F.Mask" "F.Paste")
-			(roundrect_rratio 0.25)
-		)
-		(pad "SH" smd roundrect
-			(at -3.675 1.1 270)
-			(size 1.05 0.7)
-			(layers "F.Cu" "F.Mask" "F.Paste")
-			(roundrect_rratio 0.25)
-		)
-		(pad "SH" smd roundrect
-			(at 3.675 -1.1 270)
-			(size 1.05 0.7)
-			(layers "F.Cu" "F.Mask" "F.Paste")
-			(roundrect_rratio 0.25)
-		)
-		(pad "SH" smd roundrect
-			(at 3.675 1.1 270)
-			(size 1.05 0.7)
-			(layers "F.Cu" "F.Mask" "F.Paste")
-			(roundrect_rratio 0.25)
-		)
 		(embedded_fonts no)
 		(model "${KIPRJMOD}/Footprints.3dshapes/SW_SPDT_Shouhan_MSK12C02.step"
@@
 		(sheetfile "LaserDriver.kicad_sch")
 		(zone_connect 1)
-		(attr exclude_from_pos_files allow_soldermask_bridges)
+		(attr exclude_from_pos_files exclude_from_bom allow_soldermask_bridges)
 		(fp_rect
 			(start -1.225 -0.75)
@@
 			)
 		)
-		(property "Value" "47k 1%"
+		(property "Value" "47k"
 			(at 0 1.17 90)
 			(layer "F.Fab")
@@
 		(sheetfile "LaserDriver.kicad_sch")
 		(zone_connect 1)
-		(attr exclude_from_pos_files allow_soldermask_bridges)
+		(attr exclude_from_pos_files exclude_from_bom allow_soldermask_bridges)
 		(fp_rect
 			(start -0.15 -0.75)

Commit message: BOM: descriptions from the LCSC catalog, value verifier and netlist-vs-board check on all three boards
R15 (2k, C4109) still said "200Ω" in its Description: the Rev 1 symbols carried descriptions and
datasheet links of parts long replaced (R13 "1kΩ", D5 "Emerald Green", D7 "Ice Blue", L1 "22uH 6x6",
Rs1 "10Ω", D3 "1N4148", ...). Now:
- tools/lcsc_catalog.json: LCSC MPN, brand, package, description, parameter table (Resistance /
  Capacitance / Inductance ...) and datasheet URL for every code, fetched by tools/lcsc_verify.py
- stamp_lcsc.py writes Description "<MPN> (<brand>, <package>): <LCSC description>" and the LCSC
  datasheet URL into every machine-placed symbol and footprint (HAT + laser)
- tools/lcsc_verify.py: every R/C/L Value must equal LCSC's parameter, other parts' MPN must match
  the Value (label values like "FIRE" are listed, not failed), size codes must match the package;
  covers HAT, laser and the e-stim list (bom_EStimDaughter.csv) and the fields the toolkit reads:
  0 mismatches on all three boards
- tools/sync_check.py: read-only F8 (parts, footprint ids, values, DNP, pad nets, paths vs the
  exported netlist): 0 differences on all three boards after fixing the owl's missing
  "Footprints:" library prefix and the e-stim U5/U8 paths (netlist uses the other unit's uuid;
  backup in stash/EStimDaughter_2026-09-30_pre-unitpath.kicad_pcb)
- values: laser D1/D3 "SS14" -> "DSK14" (the part ordered), HAT J5 -> "GT-USB-7010ASV"
- fab outputs regenerated; ERC/DRC unchanged

Co-Authored-By: Claude Fable 5.1 <noreply@anthropic.com>
Claude-Session: https://claude.ai/code/session_018vgLizGzYPynnY93ajvoVA
Parts:
- G1: footprint OwlLogo_Laser_14mm -> Footprints:OwlLogo_Laser_14mm
- J5: value USB_C_Receptacle_USB2.0_16P -> GT-USB-7010ASV
