File: LaserHAT/LaserDaughter/LaserDaughter.kicad_sch (KiCad schematic)
At the start: 20 parts, among them J2 Conn_02x02_Counter_Clockwise, J4 Jumper for 4-terminal diode c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, Q1 SI3134KDWA-TP, Q2 DMN2056U, SW5 SW_SPDT, U2 MT3608, U3 TLV2371DBV

Commit message: LaserHAT Rev 2: hand-routed HAT, laser + e-stim daughterboards, fab outputs
HAT (LaserHAT/):
- Rev 1 -> Rev 2 schematic migration (tools/rev2_migrate.py): issue #3 fixes,
  OLED bonnet kept, analog stage moved to plug-in daughterboards (J8/J9),
  buffered BNC I/O, USB-C power switch + PFET ideal diode.
- MCU pin map re-optimised for fewest vias: Pi UART on UART1 (PA8/PA9), I2C on
  PA0/PA1 (fail-safe), PWM_A/B on TIMA0 CCP1/CCP3 (PA7/PA12) with FAULT0 on PA6,
  active-low buttons.  Pi header: SWD swapped, NRST <-> MCU_POWER_EN swapped.
- Stable symbol UUIDs so KiCad "Update PCB" never replaces footprints.
- PCB placed and routed by hand; tidied (tools/track_tidy.py), silkscreen
  decluttered (tools/silk_declutter.py).  DRC clean apart from known cosmetic items.
- JLC fab outputs regenerated (fab/LaserHAT).
- CLAUDE.md, REV2_NOTES.md updated; portable Claude memory in claude_memory/.

Daughterboards: LaserDaughter (300 mA laser driver) and EStimDaughter (isolated
e-stim, imported from kbest/estim_module); interface spec in estim_interface/.

Firmware/Pi: `make flash HAT_REV=2` selects the Rev 2 header wiring;
Pi/power_cycle.py takes its power/reset pins from the environment.

Co-Authored-By: Claude Opus 5.5 <noreply@anthropic.com>
Parts:
- removed D2: Zener 4.7V, 1.5W, Diode_SMD:D_SMA, symbol Diode:1N4148W
- removed Q2: DMN2056U, Package_TO_SOT_SMD:SOT-23, symbol Transistor_FET:DMG2302U
- added C12: 100nF, Capacitor_SMD:C_0402_1005Metric, symbol Device:C
- added D2: 2.4V 1W (KDZVTR2.4B), Diode_SMD:D_SOD-123F, symbol Device:D_Zener
- added D4: 2.7V 1W (KDZVTR2.7B), Diode_SMD:D_SOD-123F, symbol Device:D_Zener
- added J1: HAT_J8, Connector_PinHeader_2.54mm:PinHeader_1x05_P2.54mm_Vertical, symbol Connector_Generic:Conn_01x05
- added J3: HAT_J9, Connector_PinHeader_2.54mm:PinHeader_1x05_P2.54mm_Vertical, symbol Connector_Generic:Conn_01x05
- added J5: RED_SHUNT, Connector_PinHeader_2.00mm:PinHeader_1x02_P2.00mm_Vertical, symbol Connector_Generic:Conn_01x02
- added Q2: NDT3055L, Package_TO_SOT_SMD:SOT-223-3_TabPin2, symbol Transistor_FET:NDT3055L
- added R1: 100k 1%, Resistor_SMD:R_0402_1005Metric, symbol Device:R
- added R2: 33k 1%, Resistor_SMD:R_0402_1005Metric, symbol Device:R
- added R3: 39k 1%, Resistor_SMD:R_0402_1005Metric, symbol Device:R
- added R4: 10k 1%, Resistor_SMD:R_0402_1005Metric, symbol Device:R
- D3: value 1N4148W -> SS14; footprint Footprints:D_SOD-323F -> Diode_SMD:D_SOD-123F
- J4: value Jumper for 4-terminal diode configuration -> PD_K-LASER_V (solder jumper); footprint Connector_PinHeader_2.54mm:PinHeader_1x02_P2.54mm_Vertical -> Jumper:SolderJumper-2_P1.3mm_Open_RoundedPad1.0x1.5mm
- L1: value 22uH -> 10uH Isat>=1.5A (SRN4018-100M); footprint Inductor_SMD:L_APV_ANR6045 -> Inductor_SMD:L_Bourns-SRN4018
- Rs1: value 10Ω 1% -> 2R 1% 0.5W (ESR18EZPF2R00)
Connections:
- net GND: now also C12.2, J1.1 (Pin_1), J3.1 (Pin_1), R2.2, R4.2
- net IDrive: now also Q2.3 (S)
- net LASER_V: now also R1.1; no longer U3.5 (V+)
- net LaserDrive: now also Q2.2 (D)
- net DUMMY_BOT: now reaches Q1.6 (D)
- net DUMMY_BOT: now also D4.2 (A), J5.2 (Pin_2)
- net DUMMY_TOP: now reaches D3.1 (K)
- net DUMMY_TOP: now also D2.1 (K)
- net at U3.1: now also Q2.1 (G)
- net DIODE_ADC renamed DB_ADC_A
- net DB_ADC_A: now also J3.4 (Pin_4)
- net LASER_VREF renamed IREF
- net IREF: now also R3.2, R4.1
- net PWM_DUMMY renamed DB_PWM_B
- net DB_PWM_B: now also J1.4 (Pin_4)
- net PWM_LASER renamed DB_PWM_A
- net DB_PWM_A: now also J1.3 (Pin_3)
- net V_LASER_BOOST_IN renamed +5V
- net +5V: now also U3.5 (V+), C12.1, J1.2 (Pin_2)
- new net DB_ADC_B: J3.5 (Pin_5), R1.2, R2.1
- new net DB_DAC: J3.3 (Pin_3), R3.1
- new net DUMMY_MID: D2.2 (A), D4.1 (K), J5.1 (Pin_1)
- no-connect marks 0 -> 2
Other:
- note added: "Compliance monitor: V(ADC_B) = LASER_V x 33/133 (12 V -> 2.98 V, 5 V -> 1.24 V). Firmware reports 5 V / 12 V to the OLED + web GUI."
- note added: "Current setpoint: I_LD = V(IREF) / Rs1 = DAC x (10k / 49k) / 2R (full scale ~335 mA) Dummy load: D3 + D2 (+ D4 unless J5 shunted). J5 ON = red LD (~2.8 V), OFF = blue LD (~5.5 V). Q2 dissipation: red on 5 V ~0.5 W, blue on 12 V ~0.8 W -> SOT-223 on copper. Use the 5 V setting for a single red LD (12 V would put ~2.5 W into Q2)."
- note added: "HAT interface (two 1x5, 2.54 mm) J1 (HAT J8): 1 GND 2 +5V 3 PWM_A = laser 4 PWM_B = dummy 5 GPIO (n/c) J3 (HAT J9): 1 GND 2 +3V3 (n/c) 3 DAC = current setpoint 4 ADC_A = PD 5 ADC_B = compliance"
- note removed: "At Vref=0.5V, Rsense=10Ω → I_LD=50mA"
- note removed: "Dummy load tries to ~match LD Vf for switching 4.7V Zener + 1N4148W matches 2 red (series) LDs (or 1 blue) User a 1.8V Zener for a single red LD"
- note removed: "Rsense sets I_LD = Vref / Rsense"
