File: LaserHAT/LaserDaughter/LaserDaughter.kicad_sch (KiCad schematic)
At the start: 29 parts, among them J1 HAT_J8, J2 Conn_02x02_Counter_Clockwise, J3 HAT_J9, J4 PD_K-LASER_V (solder jumper), J5 RED_SHUNT, Q1 SI3134KDWA-TP, Q2 NDT3055L, SW5 SW_SPDT, U2 MT3608, U3 TLV2371DBV

Commit message: LaserHAT + LaserDaughter: one verified "LCSC Part #" field per part for the Fabrication Toolkit
The schematics carried Rev 1 fields under four spellings ("LCSC Part #", "LCSC Part#",
"LCSC Parth#", "LCSC Part") with stale codes (every 0402 resistor = 47k, TLV2371 = AP2171,
74LVC2G17 = SI3134, zeners = SS14, DMMT5401 = MT3608 ...), which is what the toolkit's BOM showed.

- tools/lcsc_parts.py: every code re-verified against LCSC/JLC (MPN, package, value); LEDs to JLC
  basic KT-0603 (D5 white C2290, D7/D9 red C2286; was extended C5336487), R13 3k -> 2k basic,
  U1 CAT24C32 (out of stock) -> M24C32-WDW6TP C283445 (TSSOP-8, pin-compatible), U5 AP2171
  -> the WG-7 SOT-25 variant C110466 (32k in stock vs 250); VALUES table for the changed parts
- tools/stamp_lcsc.py: writes the table into one "LCSC Part #" field per symbol (text patch of
  the KiCad 9 sheets) and footprint (pcbnew), removes the misspelt variants, sets the Values;
  make_laser_daughter.py stamps its output so the laser sheet stays correct on regeneration
- jlc_fab.py warns when a board field disagrees with the table
- both schematics + boards stamped; ERC/DRC unchanged, path_check 0 mismatches; fab outputs
  regenerated; HAT board backup in stash/LaserDriver_user_2026-09-30_pre-lcsc.kicad_pcb

Co-Authored-By: Claude Fable 5.1 <noreply@anthropic.com>
Claude-Session: https://claude.ai/code/session_018vgLizGzYPynnY93ajvoVA
Parts:
- C12: LCSC Part # (none) -> C307331
- D1: LCSC Part # C894423 -> C37049
- D2: LCSC Part # (none) -> C209582
- D3: LCSC Part # C119617 -> C37049
- D4: LCSC Part # (none) -> C209583
- L1: LCSC Part # C7427158 -> C503307
- Q2: LCSC Part # (none) -> C274612
- R1: LCSC Part # (none) -> C25741
- R11: LCSC Part # C843869 -> C852624
- R2: LCSC Part # (none) -> C25779
- R3: LCSC Part # (none) -> C25783
- R4: LCSC Part # (none) -> C25744
- R5: LCSC Part # C844101 -> C25761
- Rs1: LCSC Part # C42460620 -> C2105197
Changed lines of the file:
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@@
 			)
 		)
-		(property "LCSC Part #" "C7427158"
+		(property "LCSC Part #" "C503307"
 			(at 130.81 44.45 90)
 			(effects
@@
 			)
 		)
-		(property "LCSC Part #" "C844101"
+		(property "LCSC Part #" "C25761"
 			(at 157.48 62.23 0)
 			(effects
@@
 			)
 		)
-		(property "LCSC Part #" "C42460620"
+		(property "LCSC Part #" "C2105197"
 			(at 146.05 226.06 0)
 			(effects
@@
 			)
 		)
-		(property "LCSC Part #" "C843869"
+		(property "LCSC Part #" "C852624"
 			(at 200.66 148.59 0)
 			(effects
@@
 			)
 		)
-		(property "LCSC Part #" "C119617"
+		(property "LCSC Part #" "C37049"
 			(at 127 138.43 90)
 			(effects
@@
 			)
 		)
-		(property "LCSC Part #" "C894423"
+		(property "LCSC Part #" "C37049"
 			(at 149.86 55.88 0)
 			(effects
@@
       (effects (font (size 1.27 1.27)) hide)
     )
+		(property "LCSC Part #" "C25783"
+			(at 88.9 185.42 0)
+			(effects
+				(font
+					(size 1.27 1.27)
+				)
+				(hide yes)
+			)
+		)
     (pin "1")
     (pin "2")
@@
       (effects (font (size 1.27 1.27)) hide)
     )
+		(property "LCSC Part #" "C25744"
+			(at 99.06 185.42 0)
+			(effects
+				(font
+					(size 1.27 1.27)
+				)
+				(hide yes)
+			)
+		)
     (pin "1")
     (pin "2")
@@
       (effects (font (size 1.27 1.27)) hide)
     )
+		(property "LCSC Part #" "C274612"
+			(at 143.51 199.39 0)
+			(effects
+				(font
+					(size 1.27 1.27)
+				)
+				(hide yes)
+			)
+		)
     (pin "1")
     (pin "2")
@@
       (effects (font (size 1.27 1.27)) hide)
     )
+		(property "LCSC Part #" "C307331"
+			(at 109.22 185.42 0)
+			(effects
+				(font
+					(size 1.27 1.27)
+				)
+				(hide yes)
+			)
+		)
     (pin "1")
     (pin "2")
@@
       (effects (font (size 1.27 1.27)) hide)
     )
+		(property "LCSC Part #" "C209582"
+			(at 139.7 110.49 0)
+			(effects
+				(font
+					(size 1.27 1.27)
+				)
+				(hide yes)
+			)
+		)
     (pin "1")
     (pin "2")
@@
       (effects (font (size 1.27 1.27)) hide)
     )
+		(property "LCSC Part #" "C209583"
+			(at 154.94 110.49 0)
+			(effects
+				(font
+					(size 1.27 1.27)
+				)
+				(hide yes)
+			)
+		)
     (pin "1")
     (pin "2")
@@
       (effects (font (size 1.27 1.27)) hide)
     )
+		(property "LCSC Part #" "C25741"
+			(at 254.0 71.12 0)
+			(effects
+				(font
+					(size 1.27 1.27)
+				)
+				(hide yes)
+			)
+		)
     (pin "1")
     (pin "2")
@@
       (effects (font (size 1.27 1.27)) hide)
     )
+		(property "LCSC Part #" "C25779"
+			(at 254.0 91.44 0)
+			(effects
+				(font
+					(size 1.27 1.27)
+				)
+				(hide yes)
+			)
+		)
     (pin "1")
     (pin "2")

Commit message: Fab flags: DNP = not populated, hand-fitted = no part number + exclude from position files
The schematic DNP attribute had been doing double duty ("JLC doesn't place it" for the Pi header,
BNCs and the laser-diode socket, and "not fitted"). KiCad has a flag for each:
- lcsc_parts.NOT_FITTED -> symbol DNP (schematic, carried to the board): HAT R1/R2, the ID_SD/ID_SC
  pull-ups the Pi already provides
- lcsc_parts.HAND_FIT -> DNP cleared, no "LCSC Part #", footprint attribute "exclude from position
  files" (board-only): HAT J1/J6/J7/J8/J9/SW8, laser J1/J2/J3/J5, e-stim J1/J8/J9. They stay in the
  Fabrication Toolkit BOM with an empty number, which JLC's upload shows as "do not place".
stamp_lcsc.py applies both (e-stim board: flags only, its own "LCSC" fields untouched);
jlc_fab.py lists "Hand-fitted" and "Not fitted (DNP)" separately and accepts the toolkit's field
names. HAT now 42 placements / 28 unique. ERC/DRC/path_check unchanged; fab outputs regenerated.

Co-Authored-By: Claude Fable 5.1 <noreply@anthropic.com>
Claude-Session: https://claude.ai/code/session_018vgLizGzYPynnY93ajvoVA
Parts:
- J2: now fitted
Changed lines of the file:
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@@
 		(in_bom yes)
 		(on_board yes)
-		(dnp yes)
+		(dnp no)
 		(property "Reference" "J2"
 			(at 173.99 147.066 0)

Commit message: BOM clean-up: one line per part, non-parts excluded, SW10 shield pads unnumbered
- Values unified where the same LCSC part had two spellings (HAT R3 "47k 1%" -> "47k";
  laser R1-R5 drop the " 1%"), so the Fabrication Toolkit merges them into one BOM line
- lcsc_parts.NON_PARTS (solder jumpers, mounting holes, logo, laser J4/TP1): symbol
  "exclude from BOM" + footprint exclude-from-BOM/-position-files, so they no longer show up
  as BOM lines without a part number
- SW10 (MSK12C02) footprint: the four "SH" shield pads are unnumbered now (library + board),
  which removes the F8 warning "no pin SH in symbol"
- verified by running the Fabrication Toolkit's ProcessManager headlessly on both boards:
  HAT 36 BOM lines / 42 CPL rows, laser 24 / 23; ERC, DRC and path_check unchanged

Co-Authored-By: Claude Fable 5.1 <noreply@anthropic.com>
Claude-Session: https://claude.ai/code/session_018vgLizGzYPynnY93ajvoVA
Parts:
- J4, TP1: now left out of the parts list
- R1: value 100k 1% -> 100k
- R2: value 33k 1% -> 33k
- R3: value 39k 1% -> 39k
- R4: value 10k 1% -> 10k
- R5: value 187k 1% -> 187k
Changed lines of the file:
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@@
 		(unit 1)
 		(exclude_from_sim no)
-		(in_bom yes)
+		(in_bom no)
 		(on_board yes)
 		(dnp yes)
@@
 			)
 		)
-		(property "Value" "187k 1%"
+		(property "Value" "187k"
 			(at 160.02 63.4999 0)
 			(effects
@@
 		(unit 1)
 		(exclude_from_sim no)
-		(in_bom yes)
+		(in_bom no)
 		(on_board yes)
 		(dnp no)
@@
       (effects (font (size 1.27 1.27)))
     )
-    (property "Value" "39k 1%" (id 1) (at 91.44 187.96 0)
+    (property "Value" "39k" (id 1) (at 91.44 187.96 0)
       (effects (font (size 1.27 1.27)))
     )
@@
       (effects (font (size 1.27 1.27)))
     )
-    (property "Value" "10k 1%" (id 1) (at 101.6 187.96 0)
+    (property "Value" "10k" (id 1) (at 101.6 187.96 0)
       (effects (font (size 1.27 1.27)))
     )
@@
       (effects (font (size 1.27 1.27)))
     )
-    (property "Value" "100k 1%" (id 1) (at 256.54 73.66 0)
+    (property "Value" "100k" (id 1) (at 256.54 73.66 0)
       (effects (font (size 1.27 1.27)))
     )
@@
       (effects (font (size 1.27 1.27)))
     )
-    (property "Value" "33k 1%" (id 1) (at 256.54 93.98 0)
-      (effects (font (size 1.27 1.27)))
-    )
+    (property "Value" "33k" (id 1) (at 256.54 93.98 0)
+      (effects (font (size 1.27 1.27)))
+    )

Commit message: BOM: descriptions from the LCSC catalog, value verifier and netlist-vs-board check on all three boards
R15 (2k, C4109) still said "200Ω" in its Description: the Rev 1 symbols carried descriptions and
datasheet links of parts long replaced (R13 "1kΩ", D5 "Emerald Green", D7 "Ice Blue", L1 "22uH 6x6",
Rs1 "10Ω", D3 "1N4148", ...). Now:
- tools/lcsc_catalog.json: LCSC MPN, brand, package, description, parameter table (Resistance /
  Capacitance / Inductance ...) and datasheet URL for every code, fetched by tools/lcsc_verify.py
- stamp_lcsc.py writes Description "<MPN> (<brand>, <package>): <LCSC description>" and the LCSC
  datasheet URL into every machine-placed symbol and footprint (HAT + laser)
- tools/lcsc_verify.py: every R/C/L Value must equal LCSC's parameter, other parts' MPN must match
  the Value (label values like "FIRE" are listed, not failed), size codes must match the package;
  covers HAT, laser and the e-stim list (bom_EStimDaughter.csv) and the fields the toolkit reads:
  0 mismatches on all three boards
- tools/sync_check.py: read-only F8 (parts, footprint ids, values, DNP, pad nets, paths vs the
  exported netlist): 0 differences on all three boards after fixing the owl's missing
  "Footprints:" library prefix and the e-stim U5/U8 paths (netlist uses the other unit's uuid;
  backup in stash/EStimDaughter_2026-09-30_pre-unitpath.kicad_pcb)
- values: laser D1/D3 "SS14" -> "DSK14" (the part ordered), HAT J5 -> "GT-USB-7010ASV"
- fab outputs regenerated; ERC/DRC unchanged

Co-Authored-By: Claude Fable 5.1 <noreply@anthropic.com>
Claude-Session: https://claude.ai/code/session_018vgLizGzYPynnY93ajvoVA
Parts:
- D1, D3: value SS14 -> DSK14

Commit message: Fab: nothing JLC does not place may be in its BOM (hand-fitted and DNP parts excluded from BOM too)
JLC's upload rejects "R2,SW8,J1,J6,J7,J8,R1,J9 designators don't exist in the CPL file": a BOM
line without a placement is an error, not a "do not place". So HAND_FIT parts now carry symbol
"exclude from BOM" + footprint exclude-from-BOM and -position-files, NOT_FITTED parts DNP +
exclude-from-BOM (independent of the toolkit's "Exclude DNP" checkbox), e-stim PS1 likewise on
its board. jlc_fab.py classifies from lcsc_parts.HAND_FIT and warns on any flag drift.
Verified with the toolkit's own ProcessManager in both checkbox states: every BOM designator is
in the CPL on all three boards (HAT 30 lines / 42, laser 20 / 23, e-stim 23 / 42).

Co-Authored-By: Claude Fable 5.1 <noreply@anthropic.com>
Claude-Session: https://claude.ai/code/session_018vgLizGzYPynnY93ajvoVA
Parts:
- J1, J2, J3, J5: now left out of the parts list
Changed lines of the file:
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@@
 		(unit 1)
 		(exclude_from_sim no)
-		(in_bom yes)
+		(in_bom no)
 		(on_board yes)
 		(dnp no)
@@
   )
   (symbol (lib_id "Connector_Generic:Conn_01x02") (at 170.18 110.49 0) (unit 1)
-    (in_bom yes) (on_board yes) (fields_autoplaced)
+    (in_bom no) (on_board yes) (fields_autoplaced)
     (property "Reference" "J5" (id 0) (at 172.72 107.95 0)
       (effects (font (size 1.27 1.27)))
@@
   )
   (symbol (lib_id "Connector_Generic:Conn_01x05") (at 330.2 116.84 0) (unit 1)
-    (in_bom yes) (on_board yes) (fields_autoplaced)
+    (in_bom no) (on_board yes) (fields_autoplaced)
     (property "Reference" "J1" (id 0) (at 332.74 114.3 0)
       (effects (font (size 1.27 1.27)))
@@
   )
   (symbol (lib_id "Connector_Generic:Conn_01x05") (at 330.2 147.32 0) (unit 1)
-    (in_bom yes) (on_board yes) (fields_autoplaced)
+    (in_bom no) (on_board yes) (fields_autoplaced)
     (property "Reference" "J3" (id 0) (at 332.74 144.78 0)
       (effects (font (size 1.27 1.27)))

Commit message: LaserHAT: SW8 BACK -> Panasonic EVQP7A01P side-actuated SMD (C79167); Values = part numbers; stamp clears flags
- SW8: schematic footprint Button_Switch_SMD:SW_SPST_EVQP7A; board footprint swapped at the south
  edge (111.55, 98.25), body flush with the edge, button ~0.35 mm proud; BUTTON1 via at the old
  THT pin joins the hand-routed B.Cu run, pad-1 pair bridged; GND pads on the pour. DRC identical
  to before the swap, 0 unconnected; backup stash/LaserDriver_user_2026-09-30_pre-sw8smd.kicad_pcb
- stamp_lcsc.py now also clears DNP / exclude flags on machine-placed parts (SW8 had stayed
  excluded after the previous commit, which wrongly claimed 43 placements)
- Values of LEDs and switches are the part numbers (KT-0603R/W, TS-1088-AR02016, MSK12C02,
  BL-DT, EVQP7A01P, PCM12SMTR) so JLC's BOM matcher sees one part per line; the function names
  remain as silkscreen texts
- verified: lcsc_verify 0 mismatches, sync_check 0 differences (HAT, laser), toolkit BOM/CPL
  consistent in both DNP modes (HAT 29 lines / 43 placements); fab outputs regenerated; docs

Co-Authored-By: Claude Fable 5.1 <noreply@anthropic.com>
Claude-Session: https://claude.ai/code/session_018vgLizGzYPynnY93ajvoVA
Parts:
- SW5: value SW_SPDT -> PCM12SMTR
Changed lines of the file:
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@@
 			)
 		)
-		(property "Value" "SW_SPDT"
+		(property "Value" "PCM12SMTR"
 			(at 190.5 46.99 0)
 			(effects
