File: LaserHAT/LaserDaughter/LaserDaughter.kicad_sch (KiCad schematic)
At the start: 29 parts, among them J1 HAT_J8, J2 Conn_02x02_Counter_Clockwise, J3 HAT_J9, J4 PD_K-LASER_V (solder jumper), J5 RED_SHUNT, Q1 SI3134KDWA-TP, Q2 NDT3055L, SW5 PCM12SMTR, U2 MT3608, U3 TLV2371DBV

Commit message: Updated layout of laser daughter PCB
Parts:
- removed TP1: TestPoint, TestPoint:TestPoint_Pad_D1.5mm, symbol Connector:TestPoint
