File: LaserHAT/LaserDaughter/LaserDaughter.kicad_sch (KiCad schematic)
At the start: 28 parts, among them J1 HAT_J8, J2 Conn_02x02_Counter_Clockwise, J3 HAT_J9, J4 PD_K-LASER_V (solder jumper), J5 RED_SHUNT, Q1 SI3134KDWA-TP, Q2 NDT3055L, SW5 PCM12SMTR, U2 MT3608, U3 TLV2371DBV

Commit message: Updated laser daughter PCB design with higher current PWM switch
Parts:
- D2: value 2.4V 1W (KDZVTR2.4B) -> 2.7V 1W (KDZVTR2.7B); LCSC Part # C209582 -> C209583
- D4: value 2.7V 1W (KDZVTR2.7B) -> 2.4V 1W (KDZVTR2.4B); LCSC Part # C209583 -> C209582
- Q1: value SI3134KDWA-TP -> AO9926B; footprint Package_TO_SOT_SMD:SOT-363_SC-70-6 -> Package_SO:SOIC-8_3.9x4.9mm_P1.27mm; symbol Transistor_FET:Q_Dual_NMOS_S1G1D2S2G2D1 -> Transistor_FET:FDS9926A; LCSC Part # C3290118 -> C428343
Connections:
- net +12V: now also SW5.1 (A); no longer SW5.3 (C)
- net +5V: now also SW5.3 (C); no longer SW5.1 (A)
- net DB_PWM_A: now also Q1.2 (G1); no longer Q1.5 (G)
- net DB_PWM_B: now also Q1.4 (G2); no longer Q1.2 (G)
- net DUMMY_BOT: now also Q1.5 (D2), Q1.6 (D2); no longer J5.2 (Pin_2), Q1.6 (D)
- net DUMMY_MID: now also J5.2 (Pin_2); no longer J5.1 (Pin_1)
- net DUMMY_TOP: now also J5.1 (Pin_1)
- net LaserDrive: now also Q1.3 (S2); no longer Q1.4 (S)
- net at J2.2 (LD_Cathode): now also Q1.7 (D1), Q1.8 (D1); no longer Q1.3 (D)
Other:
- note added: "Current setpoint: I_LD = V(IREF) / Rs1 = DAC x (10k / 49k) / 2R (full scale ~335 mA) Dummy load: D3 + D4 2.4 V (+ D2 2.7 V unless J5 shunts it). J5 ON = red LD (~2.8 V), OFF = blue LD (~5.5 V). Q1 is a cascode (gates at 3.3 V): it takes LASER_V - V_LD - ~2.3 V, Q2 <= 0.5 W. 100 ms pulses, DAC to 0 between pulses. Use the 5 V setting for a single red LD (12 V would put ~1.9 W into Q1)."
- note removed: "Current setpoint: I_LD = V(IREF) / Rs1 = DAC x (10k / 49k) / 2R (full scale ~335 mA) Dummy load: D3 + D2 (+ D4 unless J5 shunted). J5 ON = red LD (~2.8 V), OFF = blue LD (~5.5 V). Q2 dissipation: red on 5 V ~0.5 W, blue on 12 V ~0.8 W -> SOT-223 on copper. Use the 5 V setting for a single red LD (12 V would put ~2.5 W into Q2)."
- moved on the sheet: C12, D2, D3, D4, J5, R4, SW5
