File: LaserHAT/LaserDaughter/LaserDaughter.kicad_pcb (KiCad board)
At the start: 2 copper layers, 26.5 x 23.5 mm, 29 parts, among them J1 HAT_J8, J2 Conn_02x02_Counter_Clockwise, J3 HAT_J9, J4 PD_K-LASER_V (solder jumper), J5 RED_SHUNT, Q1 SI3134KDWA-TP, Q2 NDT3055L, SW5 SW_SPDT, U2 MT3608, U3 TLV2371DBV

Commit message: BOM clean-up: one line per part, non-parts excluded, SW10 shield pads unnumbered
- Values unified where the same LCSC part had two spellings (HAT R3 "47k 1%" -> "47k";
  laser R1-R5 drop the " 1%"), so the Fabrication Toolkit merges them into one BOM line
- lcsc_parts.NON_PARTS (solder jumpers, mounting holes, logo, laser J4/TP1): symbol
  "exclude from BOM" + footprint exclude-from-BOM/-position-files, so they no longer show up
  as BOM lines without a part number
- SW10 (MSK12C02) footprint: the four "SH" shield pads are unnumbered now (library + board),
  which removes the F8 warning "no pin SH in symbol"
- verified by running the Fabrication Toolkit's ProcessManager headlessly on both boards:
  HAT 36 BOM lines / 42 CPL rows, laser 24 / 23; ERC, DRC and path_check unchanged

Co-Authored-By: Claude Fable 5.1 <noreply@anthropic.com>
Claude-Session: https://claude.ai/code/session_018vgLizGzYPynnY93ajvoVA
Parts:
- R1: value 100k 1% -> 100k
- R2: value 33k 1% -> 33k
- R3: value 39k 1% -> 39k
- R4: value 10k 1% -> 10k
- R5: value 187k 1% -> 187k
Changed lines of the file:
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@@
 			)
 		)
-		(property "Value" "100k 1%"
+		(property "Value" "100k"
 			(at 0 1.17 0)
 			(layer "F.Fab")
@@
 			)
 		)
-		(property "Value" "33k 1%"
+		(property "Value" "33k"
 			(at 0 1.17 0)
 			(layer "F.Fab")
@@
 			)
 		)
-		(property "Value" "39k 1%"
+		(property "Value" "39k"
 			(at 0 1.17 270)
 			(layer "F.Fab")
@@
 			)
 		)
-		(property "Value" "10k 1%"
+		(property "Value" "10k"
 			(at 0 1.17 90)
 			(layer "F.Fab")
@@
 			)
 		)
-		(property "Value" "187k 1%"
+		(property "Value" "187k"
 			(at 0 1.17 180)
 			(layer "F.Fab")
@@
 		)
 		(zone_connect 1)
-		(attr exclude_from_pos_files dnp allow_soldermask_bridges)
+		(attr exclude_from_pos_files exclude_from_bom dnp allow_soldermask_bridges)
 		(fp_rect
 			(start -0.15 -0.75)
@@
 			)
 		)
-		(attr exclude_from_pos_files)
+		(attr exclude_from_pos_files exclude_from_bom)
 		(fp_circle
 			(center 0 0)

Commit message: BOM: descriptions from the LCSC catalog, value verifier and netlist-vs-board check on all three boards
R15 (2k, C4109) still said "200Ω" in its Description: the Rev 1 symbols carried descriptions and
datasheet links of parts long replaced (R13 "1kΩ", D5 "Emerald Green", D7 "Ice Blue", L1 "22uH 6x6",
Rs1 "10Ω", D3 "1N4148", ...). Now:
- tools/lcsc_catalog.json: LCSC MPN, brand, package, description, parameter table (Resistance /
  Capacitance / Inductance ...) and datasheet URL for every code, fetched by tools/lcsc_verify.py
- stamp_lcsc.py writes Description "<MPN> (<brand>, <package>): <LCSC description>" and the LCSC
  datasheet URL into every machine-placed symbol and footprint (HAT + laser)
- tools/lcsc_verify.py: every R/C/L Value must equal LCSC's parameter, other parts' MPN must match
  the Value (label values like "FIRE" are listed, not failed), size codes must match the package;
  covers HAT, laser and the e-stim list (bom_EStimDaughter.csv) and the fields the toolkit reads:
  0 mismatches on all three boards
- tools/sync_check.py: read-only F8 (parts, footprint ids, values, DNP, pad nets, paths vs the
  exported netlist): 0 differences on all three boards after fixing the owl's missing
  "Footprints:" library prefix and the e-stim U5/U8 paths (netlist uses the other unit's uuid;
  backup in stash/EStimDaughter_2026-09-30_pre-unitpath.kicad_pcb)
- values: laser D1/D3 "SS14" -> "DSK14" (the part ordered), HAT J5 -> "GT-USB-7010ASV"
- fab outputs regenerated; ERC/DRC unchanged

Co-Authored-By: Claude Fable 5.1 <noreply@anthropic.com>
Claude-Session: https://claude.ai/code/session_018vgLizGzYPynnY93ajvoVA
Parts:
- D1, D3: value SS14 -> DSK14

Commit message: LaserHAT: SW8 BACK -> Panasonic EVQP7A01P side-actuated SMD (C79167); Values = part numbers; stamp clears flags
- SW8: schematic footprint Button_Switch_SMD:SW_SPST_EVQP7A; board footprint swapped at the south
  edge (111.55, 98.25), body flush with the edge, button ~0.35 mm proud; BUTTON1 via at the old
  THT pin joins the hand-routed B.Cu run, pad-1 pair bridged; GND pads on the pour. DRC identical
  to before the swap, 0 unconnected; backup stash/LaserDriver_user_2026-09-30_pre-sw8smd.kicad_pcb
- stamp_lcsc.py now also clears DNP / exclude flags on machine-placed parts (SW8 had stayed
  excluded after the previous commit, which wrongly claimed 43 placements)
- Values of LEDs and switches are the part numbers (KT-0603R/W, TS-1088-AR02016, MSK12C02,
  BL-DT, EVQP7A01P, PCM12SMTR) so JLC's BOM matcher sees one part per line; the function names
  remain as silkscreen texts
- verified: lcsc_verify 0 mismatches, sync_check 0 differences (HAT, laser), toolkit BOM/CPL
  consistent in both DNP modes (HAT 29 lines / 43 placements); fab outputs regenerated; docs

Co-Authored-By: Claude Fable 5.1 <noreply@anthropic.com>
Claude-Session: https://claude.ai/code/session_018vgLizGzYPynnY93ajvoVA
Parts:
- SW5: value SW_SPDT -> PCM12SMTR
Changed lines of the file:
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@@
 			)
 		)
-		(property "Value" "SW_SPDT"
+		(property "Value" "PCM12SMTR"
 			(at 0 4.25 270)
 			(layer "F.Fab")
