File: LaserHAT/LaserDaughter/LaserDaughter.kicad_pcb (KiCad board)
At the start: 4 copper layers, 26.5 x 23.5 mm, 28 parts, among them J1 HAT_J8, J2 Conn_02x02_Counter_Clockwise, J3 HAT_J9, J4 PD_K-LASER_V (solder jumper), J5 RED_SHUNT, Q1 SI3134KDWA-TP, Q2 NDT3055L, SW5 PCM12SMTR, U2 MT3608, U3 TLV2371DBV

Commit message: LaserDaughter: LASER_V closure routed west under the LD pads, clear of J2 pin 2 (DRC clearance clean)
Co-Authored-By: Claude Fable 5.1 <noreply@anthropic.com>
Claude-Session: https://claude.ai/code/session_018vgLizGzYPynnY93ajvoVA
Routing:
- net LASER_V: track 38.2 -> 39.7 mm
Changed lines of the file:
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@@
+	)
+	(segment
+		(start 113.697 92.975)
+		(end 112.2 92.975)
+		(width 0.5)
+		(layer "B.Cu")
+		(net 16)
 	)
 	(segment
@@
 	)
 	(segment
-		(start 113.697 92.975)
-		(end 111.812 94.86)
+		(start 112.2 92.975)
+		(end 110.315 94.86)
 		(width 0.5)
 		(layer "B.Cu")
