File: LaserHAT/stash/EStimDaughter_M1_2026-09-28_pre-fault.kicad_sch (KiCad schematic)
At the start: 60 parts, among them J1 ELECTRODE E1/E2, J8 J8 power/timing (underside), J9 J9 analog/SPI (underside), U1 ISO7761FDBQR, U2 TLV76050DBZR, U3 TL431 (2.5V), U4 MCP4921-E/MS, U5 OPA2192IDGKR, U6 74HC4053BQ, U7 DG419BDQ, U8 LM393DGKR

Commit message: EStimDaughter rev M3: fault detector restored, 26.5 x 36.5 mm single-sided board, DHVQFN 4053 + MSOP DG419B
- LM393 compliance / open-electrode window (U8, R20-R28, C18, C19) back exactly as in rev E;
  sim/fault.py + monitor() in sim/spice.py (LM2903B TI model): trips at |E1| > 0.915 V,
  7-12 us before the current collapses, open electrode in 3.8 us, no false trips.
- 74HC4053PW -> 74HC4053BQ (DHVQFN-16), DG419DY -> DG419BDQ (MSOP-8; 15 ohm, 38 pC, 12 pF).
- Module outline extended 12.5 mm south over the Pi's port edge (y 76-112.5, HAT NOTICE 12),
  all SMD on the top; HAT column ends at y 100 so the SE corner is isolated.
- tools: route_pcb/build_pcb/netcheck take FREEROUTING / KICAD_CLI / KICAD_FOOTPRINTS from
  the environment (Ubuntu); U8 anchored, single-sided placement; Freerouting seed 0 + fix-ups:
  DRC clean, 0 unconnected, netcheck OK.
- Docs: README, DESIGN_NOTES (M2/M3 sections), spec MCU pins (PA7/PA12/PA6/PA22) and outline,
  NOTICE 11 (fault detector) and 12 (outline), REV2_NOTES, BOM (57 lines), fab outputs.
- stash/: M1 and M2 boards for reference. EStimDaughter/route/ is git-ignored.

Co-Authored-By: Claude Fable 5.1 <noreply@anthropic.com>
Claude-Session: https://claude.ai/code/session_018vgLizGzYPynnY93ajvoVA
Parts:
- U6: value 74HC4053BQ -> 74HC4053PW; footprint Package_DFN_QFN:DHVQFN-16-1EP_2.5x3.5mm_P0.5mm_EP1x2mm -> Package_SO:TSSOP-16_4.4x5mm_P0.65mm; LCSC C547007 -> C5648
- U7: value DG419BDQ -> DG419DY; footprint Package_SO:MSOP-8_3x3mm_P0.65mm -> Package_SO:SOIC-8_3.9x4.9mm_P1.27mm; LCSC C2673354 -> C6581
