File: LaserHAT/stash/EStimDaughter_M4_layout_2026-09-29_pre-tlv1702.kicad_pcb (KiCad board)
At the start: 4 copper layers, 26.5 x 36.5 mm, 53 parts, among them J1 ELECTRODE E1/E2, J8 J8 power/timing (underside), J9 J9 I2C/release (underside), U1 ISO7741FDBQR, U2 TLV76050DBZR, U4 DAC60501ZDGSR, U5 OPA2192IDGKR, U6 74HC4053BQ, U7 DG419BDQ, U8 TLV1702AIDGKR, U9 ISO1640BDR

Commit message: EStimDaughter M4b: fault detector simplified to a TLV1702 window on the +/-V rails
- U8 LM393 (0/5 V, nine resistors) -> TLV1702AIDGKR on +V/-V (rail-to-rail inputs, same
  VSSOP-8 footprint): E1 compared directly with the taps of one 10k / 215k / 10k string
  (R23-R25); outputs through R26 10k with D2 BAT54WS clamping FAULT_n; C19 -> 100n 50V
  across the rails.  Removed R20-R22, C18, R27, R28.  Thresholds +/-0.915 V for equal packs,
  the average margin for unequal packs, fault held with a pack missing.
- sims: behavioural comparator (COMPOC) + level shift; full run: lead 8-13 us, open electrode
  ~1 us, no false trips.  Schematic regenerated (netcheck OK, ERC 0), BOM 50 lines.
- Board (the layout session's file, tracks kept): removed parts deleted, U8/R23-R26/R19
  re-netted and revalued, C19 swapped to 0603, D2 parked east of the outline.
  tools/pcb_sync.py loads footprints through PCB_IO_KICAD_SEXPR (9.0.8 quirk).
- Docs: README, DESIGN_NOTES (M4b), LAYOUT_HANDOFF (open question 1 answered: J9.4 = SDA,
  J9.5 = SCL accepted), spec section 7, REV2_NOTES firmware pins, sim/models README.

Co-Authored-By: Claude Fable 5.1 <noreply@anthropic.com>
Claude-Session: https://claude.ai/code/session_018vgLizGzYPynnY93ajvoVA
Parts:
- removed D2: BAT54WS, Diode_SMD:D_SOD-323
- added C18: 100p, C_0402_1005Metric, F.Cu at (132.9, 104.8)
- added R20: 100k, R_0402_1005Metric, F.Cu at (131.5, 103.2)
- added R21: 12k, R_0402_1005Metric, F.Cu at (134.5, 105.2)
- added R22: 27k, R_0402_1005Metric, F.Cu at (134.4, 104.0)
- added R27: 12k, R_0402_1005Metric, F.Cu at (126.2, 100.5)
- added R28: 27k, R_0402_1005Metric, F.Cu at (140.3, 106.3)
- C19: footprint Capacitor_SMD:C_0603_1608Metric -> C_0402_1005Metric
- R23, R26: value 10k -> 110k
- R24: value 215k -> 12k
- R25: value 10k -> 27k
- U8: value TLV1702AIDGKR -> LM393DGKR
- moved C19 3.13 mm to (91.3, 106.6)
Connections:
- C19 pad 1: +V_STIM -> +5V_ISO
- C19 pad 2: -V_STIM -> GND_ISO
- R24 pad 2: Net-(U8B--) -> GND_ISO
- R25 pad 1: Net-(U8B--) -> +5V_ISO
- R25 pad 2: -V_STIM -> Net-(U8A-+)
- R26 pad 1: /FAULT_OC -> Net-(U8B--)
- R26 pad 2: FAULT_n -> -V_STIM
- U8 pad 1: /FAULT_OC -> FAULT_n
- U8 pad 2: E1 -> Net-(U8A--)
- U8 pad 4: -V_STIM -> GND_ISO
- U8 pad 5: E1 -> Net-(U8A--)
- U8 pad 7: /FAULT_OC -> FAULT_n
- U8 pad 8: +V_STIM -> +5V_ISO
