File: LaserHAT/stash/LaserDaughter_2026-09-29_pre-j8swap.kicad_pcb (KiCad board)
At the start: 2 copper layers, 26.5 x 23.5 mm, 29 parts, among them J1 HAT_J8, J2 Conn_02x02_Counter_Clockwise, J3 HAT_J9, J4 PD_K-LASER_V (solder jumper), J5 RED_SHUNT, Q1 SI3134KDWA-TP, Q2 NDT3055L, SW5 SW_SPDT, U2 MT3608, U3 TLV2371DBV

Commit message: LaserHAT: J8.3 = FAULT_n (PA6), J8.5 = EN/PWM_A (PA7) on the HAT and the laser module
Follows the e-stim module's connector standard (spec §3/§7, LAYOUT_HANDOFF Q2):
- bnc_daughter_io.kicad_sch: DB_GPIO on J8.3, DB_PWM_A on J8.5 (rev2_migrate.py matches)
- LaserDriver.kicad_pcb: J8 pads re-netted, PA6/PA7 traces re-routed along the old
  corridors (same vias at U7); DRC unchanged, 0 unconnected; backup in stash/
- LaserDaughter: J1.5 = DB_PWM_A, J1.3 n/c; schematic regenerated, board re-routed
- REV2_NOTES/CLAUDE.md: PA17/PA22 rows now say I2C SDA/SCL; note on why hardware I2C1
  cannot use them and the re-map that would (J9.4 -> PA16, J9.5 -> PA17, BUTTON3 -> PA22)
- LAYOUT_HANDOFF Q1/Q2 answered, spec §7 marked applied, fab outputs regenerated
- tools/schlib.py: symbol dir from env / Linux default

Co-Authored-By: Claude Fable 5.1 <noreply@anthropic.com>
Claude-Session: https://claude.ai/code/session_018vgLizGzYPynnY93ajvoVA
Connections:
- J1 pad 3: (no net) -> DB_PWM_A
- J1 pad 5: DB_PWM_A -> unconnected-(J1-Pin_5-Pad5)
Routing:
- net DB_PWM_A: track 15.5 -> 20.8 mm
Changed lines of the file:
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@@
 	(net 20 "Net-(Q2-G)")
 	(net 21 "Net-(U2-FB)")
-	(net 22 "unconnected-(J3-Pin_2-Pad2)")
-	(net 23 "unconnected-(U2-NC-Pad6)")
+	(net 22 "unconnected-(J1-Pin_5-Pad5)")
+	(net 23 "unconnected-(J3-Pin_2-Pad2)")
+	(net 24 "unconnected-(U2-NC-Pad6)")
 	(footprint "Package_TO_SOT_SMD:SOT-363_SC-70-6"
 		(layer "F.Cu")
@@
 			(layers "F.Cu" "F.Mask" "F.Paste")
 			(roundrect_rratio 0.25)
-			(net 23 "unconnected-(U2-NC-Pad6)")
+			(net 24 "unconnected-(U2-NC-Pad6)")
 			(pinfunction "NC")
 			(pintype "no_connect")
@@
 			(layers "*.Cu" "*.Mask")
 			(remove_unused_layers no)
+			(net 13 "DB_PWM_A")
 		)
 		(pad "4" thru_hole circle
@@
 			(layers "*.Cu" "*.Mask")
 			(remove_unused_layers no)
-			(net 13 "DB_PWM_A")
+			(net 22 "unconnected-(J1-Pin_5-Pad5)")
 		)
 		(embedded_fonts no)
@@
 			(layers "*.Cu" "*.Mask")
 			(remove_unused_layers no)
-			(net 22 "unconnected-(J3-Pin_2-Pad2)")
+			(net 23 "unconnected-(J3-Pin_2-Pad2)")
 		)
 		(pad "3" thru_hole circle
@@
 	)
 	(segment
+		(start 114.975 77.575)
+		(end 115.275 77.275)
+		(width 0.25)
+		(locked yes)
+		(layer "F.Cu")
+		(net 13)
+	)
+	(segment
 		(start 118.275 92.175)
 		(end 117.875 92.575)
@@
 	)
 	(segment
-		(start 119.16 80)
+		(start 117.875 77.375)
+		(end 117.875 80.475)
+		(width 0.25)
+		(locked yes)
+		(layer "F.Cu")
+		(net 13)
+	)
+	(segment
+		(start 117.875 80.475)
 		(end 118.275 80.875)
 		(width 0.25)
+		(locked yes)
 		(layer "F.Cu")
 		(net 13)
@@
 	)
 	(segment
-		(start 119.16 78.5)
-		(end 119.16 80)
+		(start 117.875 92.575)
+		(end 117.575 92.575)
+		(width 0.25)
+		(locked yes)
+		(layer "F.Cu")
+		(net 13)
+	)
+	(segment
+		(start 115.275 77.275)
+		(end 117.775 77.275)
+		(width 0.25)
+		(locked yes)
+		(layer "F.Cu")
+		(net 13)
+	)
+	(segment
+		(start 117.775 77.275)
+		(end 117.875 77.375)
 		(width 0.25)
+		(locked yes)
 		(layer "F.Cu")
 		(net 13)
 	)
 	(segment
-		(start 117.875 92.575)
-		(end 117.575 92.575)
+		(start 114.08 78.5)
+		(end 114.975 77.575)
 		(width 0.25)
 		(locked yes)
