File: LaserHAT/stash/LaserDriver_user_2026-09-30_pre-owlgnd.kicad_pcb (KiCad board)
At the start: 2 copper layers, 65 x 56.9 mm, 58 parts, among them J1 GPIO, J5 USB_C_Receptacle_USB2.0_16P, J6 BNC TRIGGER IN, J7 BNC STIM OUT, J8 DB_POWER_TIMING, J9 DB_ANALOG, Q3 AP30P30Q, Q4 DMMT5401, Q5 AP30P30Q, SW10 USB PWR, SW6 BSL, SW7 BL-DT (LCSC C53223909), SW8 BACK, SW9 FIRE, U1 CAT24C32, U4 MCP1700x-330xxMB, U5 AP2171W, U6 CH340N, U7 MSPM0G3507SRHBR, U8 74LVC2G17

Commit message: LaserHAT: owl logo's laser eyes and beams are pads on GND
- Footprints.pretty/OwlLogo_Laser_14mm: the two eye polygons and two beam lines on F.Cu/F.Mask
  become four custom pads numbered 1 (solid zone connection), so the exposed copper is on a net
- LaserHAT.kicad_sym + root sheet lib copy: OwlLogo gets pin 1 "GND" (passive, below the body);
  G1 moved onto the 1.27 mm grid and a GND power symbol placed on its pin
- LaserDriver.kicad_pcb: G1 swapped for the new footprint (same position/path), pads on GND,
  zones refilled; DRC unchanged, 0 unconnected; backup stash/LaserDriver_user_2026-09-30_pre-owlgnd
- tools/jlc_fab.py: footprints excluded from both BOM and position files count as non-parts
  (the logo was being listed as hand-fit); HAT fab outputs regenerated

Co-Authored-By: Claude Fable 5.1 <noreply@anthropic.com>
Claude-Session: https://claude.ai/code/session_018vgLizGzYPynnY93ajvoVA
Parts:
- G1: footprint OwlLogo_Laser_14mm -> Footprints:OwlLogo_Laser_14mm
