File: LaserHAT/stash/LaserDaughter_2026-09-30_pre-relink.kicad_pcb (KiCad board)
At the start: 2 copper layers, 26.5 x 23.5 mm, 29 parts, among them J1 HAT_J8, J2 Conn_02x02_Counter_Clockwise, J3 HAT_J9, J4 PD_K-LASER_V (solder jumper), J5 RED_SHUNT, Q1 SI3134KDWA-TP, Q2 NDT3055L, SW5 SW_SPDT, U2 MT3608, U3 TLV2371DBV

Commit message: LaserDaughter: relink the board to the schematic UUIDs so F8 keeps the placement
11 footprints (C12 D2 D4 J1 J3 J5 Q2 R1-R4: the parts make_laser_daughter.py adds) still
carried the random uuid4 paths from the first generation while the schematic now uses uuid5,
so "Update PCB from Schematic" deleted and re-added them.

- schlib.uid() is deterministic (uuid5 counter) and add_symbol's pin uuids are keyed on
  ref/pin, so make_laser_daughter.py re-runs are byte-identical
- make_laser_daughter.py --sync-pcb: netlist export + pcb_sync.py --keep-tracks + zone fill
  (headless F8; refuses while pcbnew holds the board)
- tools/path_check.py: verifies every footprint path against the schematic hierarchy
  (root "/<sym>", sub-sheet "/<sheet>/<sym>", any unit); HAT, laser and e-stim all report 0
- LaserDaughter.kicad_pcb relinked (paths only; DRC unchanged, 0 unconnected); backup in
  stash/LaserDaughter_2026-09-30_pre-relink.kicad_pcb
- CLAUDE.md: rev2_migrate.py is stale since the HAT sheets were re-saved in KiCad (9a940e9)

Co-Authored-By: Claude Fable 5.1 <noreply@anthropic.com>
Claude-Session: https://claude.ai/code/session_018vgLizGzYPynnY93ajvoVA
Connections:
- J1 pad 3: unconnected-(J1-Pin_3-Pad3) -> (no net)
Changed lines of the file:
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@@
 	(net 22 "unconnected-(J3-Pin_2-Pad2)")
 	(net 23 "unconnected-(U2-NC-Pad6)")
-	(net 24 "unconnected-(J1-Pin_3-Pad3)")
 	(footprint "Package_TO_SOT_SMD:SOT-363_SC-70-6"
 		(layer "F.Cu")
@@
 			(layers "*.Cu" "*.Mask")
 			(remove_unused_layers no)
-			(net 24 "unconnected-(J1-Pin_3-Pad3)")
 		)
 		(pad "4" thru_hole circle
