File: LaserHAT/stash/LaserDriver_user_2026-09-30_pre-lcsc.kicad_pcb (KiCad board)
At the start: 2 copper layers, 65 x 56.9 mm, 58 parts, among them J1 GPIO, J5 USB_C_Receptacle_USB2.0_16P, J6 BNC TRIGGER IN, J7 BNC STIM OUT, J8 DB_POWER_TIMING, J9 DB_ANALOG, Q3 AP30P30Q, Q4 DMMT5401, Q5 AP30P30Q, SW10 USB PWR, SW6 BSL, SW7 BL-DT (LCSC C53223909), SW8 BACK, SW9 FIRE, U1 M24C32-WDW6TP, U4 MCP1700x-330xxMB, U5 AP2171W, U6 CH340N, U7 MSPM0G3507SRHBR, U8 74LVC2G17

Commit message: LaserHAT + LaserDaughter: one verified "LCSC Part #" field per part for the Fabrication Toolkit
The schematics carried Rev 1 fields under four spellings ("LCSC Part #", "LCSC Part#",
"LCSC Parth#", "LCSC Part") with stale codes (every 0402 resistor = 47k, TLV2371 = AP2171,
74LVC2G17 = SI3134, zeners = SS14, DMMT5401 = MT3608 ...), which is what the toolkit's BOM showed.

- tools/lcsc_parts.py: every code re-verified against LCSC/JLC (MPN, package, value); LEDs to JLC
  basic KT-0603 (D5 white C2290, D7/D9 red C2286; was extended C5336487), R13 3k -> 2k basic,
  U1 CAT24C32 (out of stock) -> M24C32-WDW6TP C283445 (TSSOP-8, pin-compatible), U5 AP2171
  -> the WG-7 SOT-25 variant C110466 (32k in stock vs 250); VALUES table for the changed parts
- tools/stamp_lcsc.py: writes the table into one "LCSC Part #" field per symbol (text patch of
  the KiCad 9 sheets) and footprint (pcbnew), removes the misspelt variants, sets the Values;
  make_laser_daughter.py stamps its output so the laser sheet stays correct on regeneration
- jlc_fab.py warns when a board field disagrees with the table
- both schematics + boards stamped; ERC/DRC unchanged, path_check 0 mismatches; fab outputs
  regenerated; HAT board backup in stash/LaserDriver_user_2026-09-30_pre-lcsc.kicad_pcb

Co-Authored-By: Claude Fable 5.1 <noreply@anthropic.com>
Claude-Session: https://claude.ai/code/session_018vgLizGzYPynnY93ajvoVA
Parts:
- R13: value 2k -> 3k
- U1: value M24C32-WDW6TP -> CAT24C32
