File: LaserHAT/stash/LaserDriver_user_2026-09-30_pre-sw8smd.kicad_pcb (KiCad board)
At the start: 2 copper layers, 65 x 56.9 mm, 58 parts, among them J1 GPIO, J5 GT-USB-7010ASV, J6 BNC TRIGGER IN, J7 BNC STIM OUT, J8 DB_POWER_TIMING, J9 DB_ANALOG, Q3 AP30P30Q, Q4 DMMT5401, Q5 AP30P30Q, SW10 MSK12C02, SW6 TS-1088-AR02016, SW7 BL-DT, SW8 EVQP7A01P, SW9 TS-1088-AR02016, U1 M24C32-WDW6TP, U4 MCP1700x-330xxMB, U5 AP2171W, U6 CH340N, U7 MSPM0G3507SRHBR, U8 74LVC2G17

Commit message: LaserHAT: SW8 BACK -> Panasonic EVQP7A01P side-actuated SMD (C79167); Values = part numbers; stamp clears flags
- SW8: schematic footprint Button_Switch_SMD:SW_SPST_EVQP7A; board footprint swapped at the south
  edge (111.55, 98.25), body flush with the edge, button ~0.35 mm proud; BUTTON1 via at the old
  THT pin joins the hand-routed B.Cu run, pad-1 pair bridged; GND pads on the pour. DRC identical
  to before the swap, 0 unconnected; backup stash/LaserDriver_user_2026-09-30_pre-sw8smd.kicad_pcb
- stamp_lcsc.py now also clears DNP / exclude flags on machine-placed parts (SW8 had stayed
  excluded after the previous commit, which wrongly claimed 43 placements)
- Values of LEDs and switches are the part numbers (KT-0603R/W, TS-1088-AR02016, MSK12C02,
  BL-DT, EVQP7A01P, PCM12SMTR) so JLC's BOM matcher sees one part per line; the function names
  remain as silkscreen texts
- verified: lcsc_verify 0 mismatches, sync_check 0 differences (HAT, laser), toolkit BOM/CPL
  consistent in both DNP modes (HAT 29 lines / 43 placements); fab outputs regenerated; docs

Co-Authored-By: Claude Fable 5.1 <noreply@anthropic.com>
Claude-Session: https://claude.ai/code/session_018vgLizGzYPynnY93ajvoVA
Parts:
- D5: value KT-0603W -> 5V
- D7: value KT-0603R -> MCU
- D9: value KT-0603R -> STIM
- SW10: value MSK12C02 -> USB PWR
- SW6: value TS-1088-AR02016 -> BSL
- SW7: value BL-DT -> BL-DT (LCSC C53223909)
- SW8: value EVQP7A01P -> BACK; footprint Button_Switch_SMD:SW_SPST_EVQP7A -> Button_Switch_THT:SW_Tactile_SPST_Angled_PTS645Vx39-2LFS
- SW9: value TS-1088-AR02016 -> FIRE
- moved SW8 2.40 mm to (113.8, 97.4), turned to 180 degrees
Routing:
- net /MSPM0 Controller/BUTTON1: track 45.4 -> 41.3 mm, vias 2 -> 1
