File: LaserHAT/EStimDaughter/EStimDaughter.kicad_pcb (KiCad board)
At the start: 4 copper layers, 26.5 x 33 mm, 48 parts, among them J1 ELECTRODE E1/E2, J8 J8 power/timing (underside), J9 J9 I2C/release (underside), U1 ISO7741FDBQR, U2 TLV76050DBZR, U4 DAC60501ZDGSR, U5 OPA2192IDGKR, U6 ADG1436YCPZ, U7 DG419BDQ, U8 TLV1702AIDGKR, U9 ISO1640BDR

Commit message: Edited silk screen in EStim daughterboard
Routing:
- net GND_ISO: vias 21 -> 23
Other:
- board text added: "ESTIM 1.0"
- board text added: "ISENSE"
- board text added: "KemereLab.org (c) 2026.10"
- board text added: "sdg"
Changed lines of the file:
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@@
 			(at 0 -0.0525 90)
 			(layer "F.SilkS")
+			(hide yes)
 			(effects
 				(font
@@
 		(tags "capacitor")
 		(property "Reference" "C16"
-			(at -3.136905 0 90)
+			(at 0.6 1.5 90)
 			(layer "F.SilkS")
 			(effects
@@
 			(at 0 -1.43 0)
 			(layer "F.SilkS")
+			(hide yes)
 			(effects
 				(font
@@
 		)
 		(fp_text user "${REFERENCE}"
-			(at 26.6125 -8.825 270)
+			(at 0.025 0 270)
 			(layer "F.Fab")
 			(effects
@@
 			(at -2.3336 0 0)
 			(layer "F.SilkS")
+			(hide yes)
 			(effects
 				(font
@@
 			(at 0 -1.5836 0)
 			(layer "F.SilkS")
+			(hide yes)
 			(effects
 				(font
@@
 			(at 15.1 -2.7 90)
 			(layer "F.SilkS")
+			(hide yes)
 			(effects
 				(font
@@
 			(at 0 0 90)
 			(layer "F.SilkS")
+			(hide yes)
 			(effects
 				(font
@@
 			(at 0 1.5836 0)
 			(layer "F.SilkS")
+			(hide yes)
 			(effects
 				(font
@@
 			(at 3.95 0 0)
 			(layer "F.SilkS")
+			(hide yes)
 			(effects
 				(font
@@
 		)
 		(fp_text user "${REFERENCE}"
-			(at -1.85 38.75 90)
+			(at -0.45 0.3 90)
 			(layer "F.Fab")
 			(effects
@@
 		)
 		(fp_text user "${REFERENCE}"
-			(at -8.825 -26.6125 90)
+			(at -0.01 -0.05 90)
 			(layer "F.Fab")
 			(effects
@@
 			(at 1.2 1.8 180)
 			(layer "F.SilkS")
+			(hide yes)
 			(effects
 				(font
@@
 			(at 0 -0.0525 180)
 			(layer "F.SilkS")
+			(hide yes)
 			(effects
 				(font
@@
 			(at 0 -1.85 90)
 			(layer "F.SilkS")
+			(hide yes)
 			(effects
 				(font
@@
 		)
 	)
+	(gr_text "ESTIM 1.0"
+		(at 110.3 77.5 0)
+		(layer "F.SilkS")
+		(effects
+			(font
+				(size 1 1)
+				(thickness 0.15)
+			)
+			(justify left bottom)
+		)
+	)
+	(gr_text "ISENSE"
+		(at 117.7 108.5 0)
+		(layer "F.SilkS")
+		(effects
+			(font
+				(size 1 1)
+				(thickness 0.15)
+			)
+			(justify left bottom)
+		)
+	)
+	(gr_text "sdg"
+		(at 126.6 77.7 0)
+		(layer "B.SilkS")
+		(effects
+			(font
+				(size 0.8 0.8)
+				(thickness 0.15)
+				(bold yes)
+			)
+			(justify left bottom mirror)
+		)
+	)
+	(gr_text "KemereLab.org\n(c) 2026.10"
+		(at 107.7 84.7 90)
+		(layer "B.SilkS")
+		(effects
+			(font
+				(size 1.25 1.25)
+				(thickness 0.18)
+			)
+			(justify left bottom mirror)
+		)
+	)
 	(segment
 		(start 122.75 86.27)
@@
 	)
 	(via
+		(at 108.1 96.4)
+		(size 0.5)
+		(drill 0.3)
+		(layers "F.Cu" "B.Cu")
+		(free yes)
+		(net 4)
+	)
+	(via
 		(at 121 100.25)
 		(size 0.5)
@@
 		(net 4)
 	)
+	(via
+		(at 103 100.2)
+		(size 0.5)
+		(drill 0.3)
+		(layers "F.Cu" "B.Cu")
+		(free yes)
+		(net 4)
+	)
