File: LaserHAT/BatteryPack/BatteryPack.kicad_sch (KiCad schematic)
At the start: 101 parts, among them J1 USB-C PD 20V in, J3 OUT +V/0V/-V + link, J4 LINK from lower pack, Q1 AO3401A, Q10 AO3400A, Q2 AO3401A, Q3 AO3400A, Q4 AO3401A, Q5 AO3400A, Q6 AO3401A, Q7 AO3400A, Q8 AO3400A, Q9 AO3400A, SW1 MTS-203 RUN/OFF/CHG, U1 LM393DR2G, U2 LM393DR2G, U3 CJ431, U4 CH224A, U5 CN3704, U6 HY2213-BB3A, U7 HY2213-BB3A, U8 HY2213-BB3A, U9 HY2213-BB3A

Commit message: BatteryPack: LCSC codes on the board footprints, JLC model strings as values
A BOM made from the PCB with the Fabrication Toolkit had no part numbers,
because the footprints carried none; JLC then matched by Comment and failed on
the parts with descriptive values (C5, F1, J1, J3, J4, SW1).

- sch_engine.py writes the code into every symbol as "LCSC Part #" (the field
  the Fabrication Toolkit reads) instead of "LCSC"; mounting holes are out of
  the BOM
- new tools/stamp_fields.py stamps the same field (hidden, F.Fab) into every
  footprint, syncs the Values and excludes H1-H4 from BOM and position files
- values of the toggle, PTC, LEDs, USB-C, PH-4 headers, inductor and NTC are
  now JLC's model strings so the Comment matches; J3/J4 roles noted as text
- schematic regenerated (netcheck OK, ERC 0), path/sync checks 0, DRC 0/0,
  fab outputs and PDF regenerated; all codes verified against JLC (toggle
  stock 192)

Co-Authored-By: Claude Fable 5.1 <noreply@anthropic.com>
Claude-Session: https://claude.ai/code/session_018vgLizGzYPynnY93ajvoVA
Parts:
- BC1, BC2, BC3, BC4, BC5, BC6, BC7, BC8: LCSC C2979183 -> (none); LCSC Part # (none) -> C2979183
- C1, C11, C12, C13, C14, C15, C2, C4: LCSC C14663 -> (none); LCSC Part # (none) -> C14663
- C10: LCSC C21120 -> (none); LCSC Part # (none) -> C21120
- C3, C6: LCSC C15849 -> (none); LCSC Part # (none) -> C15849
- C5: LCSC C2836438 -> (none); LCSC Part # (none) -> C2836438
- C7, C8: LCSC C15850 -> (none); LCSC Part # (none) -> C15850
- C9: LCSC C1620 -> (none); LCSC Part # (none) -> C1620
- D1: value red ON -> KT-0603R; LCSC C2286 -> (none); LCSC Part # (none) -> C2286
- D10: value green DONE -> KT-0805G; LCSC C2297 -> (none); LCSC Part # (none) -> C2297
- D2: value yellow >20% -> KT-0805Y; LCSC C2296 -> (none); LCSC Part # (none) -> C2296
- D3: value green >50% -> KT-0805G; LCSC C2297 -> (none); LCSC Part # (none) -> C2297
- D4: value green >80% -> KT-0805G; LCSC C2297 -> (none); LCSC Part # (none) -> C2297
- D5, D6: LCSC C2480 -> (none); LCSC Part # (none) -> C2480
- D7, D8: LCSC C8678 -> (none); LCSC Part # (none) -> C8678
- D9: value red CHRG -> KT-0603R; LCSC C2286 -> (none); LCSC Part # (none) -> C2286
- F1: value 100mA PTC -> MF-MSMF010-2; LCSC C12430 -> (none); LCSC Part # (none) -> C12430
- H1, H2, H3, H4: now left out of the parts list
- J1: value USB-C PD 20V in -> TYPE-C-31-M-12; LCSC C165948 -> (none); LCSC Part # (none) -> C165948
- J3: value OUT +V/0V/-V + link -> B4B-PH-K-S(LF)(SN); LCSC C131334 -> (none); LCSC Part # (none) -> C131334
- J4: value LINK from lower pack -> B4B-PH-K-S(LF)(SN); LCSC C131334 -> (none); LCSC Part # (none) -> C131334
- L1: value 22uH 3A -> MWSA0603S-220MT; LCSC C408453 -> (none); LCSC Part # (none) -> C408453
- Q1, Q2, Q4, Q6: LCSC C15127 -> (none); LCSC Part # (none) -> C15127
- Q10, Q3, Q5, Q7, Q8, Q9: LCSC C20917 -> (none); LCSC Part # (none) -> C20917
- R1, R16, R17, R18, R2, R20, R21, R22, R23: LCSC C25803 -> (none); LCSC Part # (none) -> C25803
- R10: LCSC C25804 -> (none); LCSC Part # (none) -> C25804
- R11, R30: LCSC C22935 -> (none); LCSC Part # (none) -> C22935
- R12, R13: LCSC C22797 -> (none); LCSC Part # (none) -> C22797
- R14, R15: LCSC C22790 -> (none); LCSC Part # (none) -> C22790
- R19: LCSC C4216 -> (none); LCSC Part # (none) -> C4216
- R24: LCSC C25808 -> (none); LCSC Part # (none) -> C25808
- R25, R26: LCSC C25334 -> (none); LCSC Part # (none) -> C25334
- R27: LCSC C22787 -> (none); LCSC Part # (none) -> C22787
- R28, R29: LCSC C22809 -> (none); LCSC Part # (none) -> C22809
- R3, R4: LCSC C23212 -> (none); LCSC Part # (none) -> C23212
- R31, R32, R33, R34: LCSC C22775 -> (none); LCSC Part # (none) -> C22775
- R35, R36, R37, R38: LCSC C17901 -> (none); LCSC Part # (none) -> C17901
- R5, R6: LCSC C22975 -> (none); LCSC Part # (none) -> C22975
- R7: LCSC C4260 -> (none); LCSC Part # (none) -> C4260
- R8: LCSC C22984 -> (none); LCSC Part # (none) -> C22984
- R9: LCSC C23231 -> (none); LCSC Part # (none) -> C23231
- RT1: value NTC 10k -> NCP18XH103F03RB; LCSC C13564 -> (none); LCSC Part # (none) -> C13564
- SW1: value MTS-203 RUN/OFF/CHG -> CAX-MTS203M-YB-10.6JL; LCSC C55160018 -> (none); LCSC Part # (none) -> C55160018
- U1, U2: LCSC C7955 -> (none); LCSC Part # (none) -> C7955
- U3: LCSC C3113 -> (none); LCSC Part # (none) -> C3113
- U4: LCSC C42459160 -> (none); LCSC Part # (none) -> C42459160
- U5: LCSC C51659 -> (none); LCSC Part # (none) -> C51659
- U6, U7, U8, U9: LCSC C113632 -> (none); LCSC Part # (none) -> C113632
Other:
- note added: "LINK IN from the lower board's J3 (lower +OUT -> GND here)"
- note added: "OUT: +V / 0V / -V / STACK_IN (to the module, or to the upper board's J4)"

Commit message: BatteryPack rev C: two hobby 4S packs on one 100 x 100 board, one charger, one toggle
Pack sockets J5/J6 (JST-XH right-angle) replace the 18650 clips; packs strap under the board.
Pole 1 of the toggle puts the packs in series (RUN) or joins their negatives (CHARGE); pole 2
runs pack B's output chain or joins the positives through a 1.1 A PTC so one CN3704 charges
both in parallel.  N-FET cutoff in pack A's negative, second gauge, VBUS switch so the charger
only sees the brick in CHARGE.  No stack cable or slave enable.  autoroute.py runs each board
edit in its own process; place.py adds keep-outs round the slots.  DRC 0/0/0, checks clean.

Co-Authored-By: Claude Fable 5.1 <noreply@anthropic.com>
Claude-Session: https://claude.ai/code/session_018vgLizGzYPynnY93ajvoVA
Parts:
- removed BC1, BC2, BC3, BC4, BC5, BC6, BC7, BC8: MY-18650-01, battpack:Clip_MY-18650-01, symbol battpack:Clip18650
- removed J4: B4B-PH-K-S(LF)(SN), Connector_JST:JST_PH_B4B-PH-K_1x04_P2.00mm_Vertical, symbol battpack:Conn_01x04
- removed Q2, Q4: AO3401A, Package_TO_SOT_SMD:SOT-23, symbol battpack:Q_PMOS_GSD
- removed Q3, Q5: AO3400A, Package_TO_SOT_SMD:SOT-23, symbol battpack:Q_NMOS_GSD
- removed R16, R17, R18, R20, R21, R22, R23: 100k, Resistor_SMD:R_0603_1608Metric, symbol battpack:R
- removed R19: 33k, Resistor_SMD:R_0603_1608Metric, symbol battpack:R
- added C16, C17, C18, C19, C20, C21: 100n, Capacitor_SMD:C_0603_1608Metric, symbol battpack:C
- added D11: KT-0603R, LED_SMD:LED_0603_1608Metric, symbol battpack:LED
- added D12: KT-0805Y, LED_SMD:LED_0805_2012Metric, symbol battpack:LED
- added D13, D14: KT-0805G, LED_SMD:LED_0805_2012Metric, symbol battpack:LED
- added D15, D16: SS14, Diode_SMD:D_SMA, symbol battpack:D_Schottky
- added F2: MF-MSMF010-2, Fuse:Fuse_1812_4532Metric, symbol battpack:Polyfuse
- added F3: MF-MSMF110/24X-2, Fuse:Fuse_1812_4532Metric, symbol battpack:Polyfuse
- added J5, J6: S5B-XH-A-1(LF)(SN), Connector_JST:JST_XH_S5B-XH-A-1_1x05_P2.50mm_Horizontal, symbol battpack:Conn_01x05
- added Q11, Q12, Q14, Q15, Q16, Q17, Q18: AO3400A, Package_TO_SOT_SMD:SOT-23, symbol battpack:Q_NMOS_GSD
- added Q13: AO3401A, Package_TO_SOT_SMD:SOT-23, symbol battpack:Q_PMOS_GSD
- added R39, R40, R41, R42, R43, R44: 100k, Resistor_SMD:R_0603_1608Metric, symbol battpack:R
- added R45, R46: 6.8k, Resistor_SMD:R_0603_1608Metric, symbol battpack:R
- added R47, R48: 2k, Resistor_SMD:R_0603_1608Metric, symbol battpack:R
- added R49: 6.2k, Resistor_SMD:R_0603_1608Metric, symbol battpack:R
- added R50: 30k, Resistor_SMD:R_0603_1608Metric, symbol battpack:R
- added R51: 68k, Resistor_SMD:R_0603_1608Metric, symbol battpack:R
- added R52: 10k, Resistor_SMD:R_0603_1608Metric, symbol battpack:R
- added R53: 1M, Resistor_SMD:R_0603_1608Metric, symbol battpack:R
- added R54, R55: 13k, Resistor_SMD:R_0603_1608Metric, symbol battpack:R
- added R56, R57: 12k, Resistor_SMD:R_0603_1608Metric, symbol battpack:R
- added R58, R59, R60, R61: 100, Resistor_SMD:R_0603_1608Metric, symbol battpack:R
- added R62, R63, R64, R65: 100, Resistor_SMD:R_1206_3216Metric, symbol battpack:R
- added U10, U11, U12, U13: HY2213-BB3A, Package_TO_SOT_SMD:SOT-23-6, symbol battpack:HY2213
- added U14, U15: LM393DR2G, Package_SO:SOIC-8_3.9x4.9mm_P1.27mm, symbol battpack:LM393
- added U16: CJ431, Package_TO_SOT_SMD:SOT-23, symbol battpack:TL431_SOT23
- R11: value 1M -> 470k; LCSC Part # C22935 -> C23178
Connections:
- net +BAT: now also SW1.1 (A1), F3.2, J5.5 (Pin_5); no longer SW1.2 (C1)
- net +G: now also R12.1, D15.1 (K), D16.1 (K); no longer D5.1 (K), D6.1 (K)
- net +OUT: now also R53.1, R54.1; no longer R11.1, R12.1
- net +RUN: now also SW1.4 (A2); no longer SW1.1 (A1)
- net C1: now also J5.2 (Pin_2)
- net C2: now also J5.3 (Pin_3)
- net C3: now also J5.4 (Pin_4)
- net GND: now also C10.2, C11.2, C3.2, C5.2 (-), C6.2, C7.2, C8.2, C9.2, D8.2 (A), J1.A1 (GND), J1.A12 (GND), J1.B1 (GND), J1.B12 (GND), J1.S1 (SH), R24.2, RT1.2, SW1.3 (B1), U4.11 (GND), U5.10 (test), U5.2 (PGND), U5.3 (GND), U5.7 (EOC), F2.1, J5.1 (Pin_1), Q12.2 (S), Q14.2 (S), R40.2, R42.2; no longer D1.1 (K), SW1.5 (C2)
- net THCUT: now also U2.6 (-); no longer U2.5 (+)
- net VBUS: now also Q13.2 (S), R43.1; no longer C4.2, C5.1 (+), C6.1, Q6.2 (S), R28.1, R29.1, U5.15 (VCC)
- net VS: now also U2.5 (+); no longer U2.6 (-)
- net +CHG renamed +CHGB
- net +CHGB: now also SW1.6 (B2), D16.2 (A), F3.1, R41.1; no longer SW1.3 (B1)
- removed net CGND: C10.2, C11.2, C3.2, C5.2 (-), C6.2, C7.2, C8.2, C9.2, D8.2 (A), J1.A1 (GND), J1.A12 (GND), J1.B1 (GND), J1.B12 (GND), J1.S1 (SH), R24.2, R30.1, RT1.2, SW1.6 (B2), U4.11 (GND), U5.10 (test), U5.2 (PGND), U5.3 (GND), U5.7 (EOC)
- net CUT_OC renamed CUT_OCB
- net CUT_OCB: now also U15.7; no longer U2.7
- net LINK_N renamed -V
- net -V: now also Q11.3 (D)
- net OUT_GND renamed 0V
- net 0V: now also R30.1, SW1.2 (C1), C16.2, C20.2, C21.2, D11.1 (K), D15.2 (A), J6.1 (Pin_1), Q15.2 (S), R39.1, R50.2, R52.2, U10.3 (VSS), U14.4 (V-), U15.4 (V-), U16.3 (A); no longer SW1.4 (A2)
- net STACK_IN: no longer names the net of J3.4 (Pin_4)
- new net: C18.1, R60.2, U12.2 (VDD)
- new net: C16.1, R58.2, U10.2 (VDD)
- new net: C19.1, R61.2, U13.2 (VDD)
- new net: Q18.1 (G), U13.6 (OUT)
- new net: D11.2 (A), R54.2
- new net: D14.1 (K), U14.1
- new net: D14.2 (A), R57.2
- new net: Q17.1 (G), U12.6 (OUT)
- new net: D12.1 (K), U15.1
- new net: D12.2 (A), R55.2
- new net: C17.1, R59.2, U11.2 (VDD)
- new net: Q16.1 (G), U11.6 (OUT)
- new net: Q18.3 (D), R65.2
- new net: D13.1 (K), U14.7
- new net: D13.2 (A), R56.2
- new net: Q15.1 (G), U10.6 (OUT)
- new net: Q15.3 (D), R62.2
- new net: Q16.3 (D), R63.2
- new net: Q17.3 (D), R64.2
- new net +BATB: J6.5 (Pin_5), R61.1, R65.1, SW1.5 (C2)
- new net +GB: C20.1, C21.1, D5.1 (K), D6.1 (K), R45.1, R51.1, R55.1, R56.1, R57.1, U14.8 (V+), U15.8 (V+)
- new net B1: C17.2, J6.2 (Pin_2), Q16.2 (S), R58.1, R62.1, U11.3 (VSS)
- new net B2: C18.2, J6.3 (Pin_3), Q17.2 (S), R59.1, R63.1, U12.3 (VSS)
- new net B3: C19.2, J6.4 (Pin_4), Q18.2 (S), R60.1, R64.1, U13.3 (VSS)
- new net D1_K: D1.1 (K), Q14.3 (D)
- new net GNDF: F2.2, Q11.2 (S)
- new net Q11_G: Q11.1 (G), Q14.1 (G), R11.1, R39.2, R40.1, U2.7
- new net Q12_G: Q12.1 (G), R41.2, R42.1
- new net Q13_G: Q13.1 (G), R43.2, R44.1
- new net Q13_GD: Q12.3 (D), R44.2
- new net TH20B: R48.2, R49.1, U15.3 (+)
- new net TH50B: R47.2, R48.1, U14.5 (+)
- new net TH80B: R46.2, R47.1, U14.3 (+)
- new net THCUTB: R49.2, R50.1, U15.5 (+)
- new net VCHG: C4.2, C5.1 (+), C6.1, Q13.3 (D), Q6.2 (S), R28.1, R29.1, U5.15 (VCC)
- new net VREFB: R45.2, R46.1, U16.1 (REF), U16.2 (K)
- new net VSB: R51.2, R52.1, R53.2, U14.2 (-), U14.6 (-), U15.2 (-), U15.6 (-)
- no-connect marks 19 -> 31
Other:
- note added: "+GB = +SW or +CHGB (D5/D6), +G = 0V or +CHGB (D15/D16): both gauges run in RUN and CHARGE and are dead in OFF."
- note added: "1. TWO 4S PACKS ON JST-XH BALANCE LEADS (pin 1 = black = pack negative) AND PER-CELL BALANCERS (HY2213-BB3A, 42 mA above 4.20 V)"
- note added: "2. RUN / OFF / CHARGE TOGGLE, OUTPUT CHAINS (+V: Q1, -V: Q11), PARALLEL LINK FOR CHARGING"
- note added: "3A. PACK A: 2.495 V REFERENCE, LADDER, SAMPLE (on +G)"
- note added: "3B. PACK B: THE SAME ON +GB, REFERENCED TO 0V"
- note added: "4A. PACK A GAUGE: THREE COMPARATORS, FOUR LEDs"
- note added: "4B. PACK B GAUGE (on +GB / 0V)"
- note added: "5. OUTPUT AND MOUNTING HOLES"
- note added: "6. USB-C PD 20 V INPUT (CH224A), VBUS SWITCH (CHARGE ONLY), 4S BUCK CHARGER (CN3704, 1 A)"
- note added: "9 % (92 mA), trickle at 150 mA below 11.2 V, re-charge below 16.0 V, over-voltage cut at 18.1 V. RT1 10k NTC (board temperature; a 10k"
- note added: "Any 4S LiPo / Li-ion hobby pack with a JST-XH 2.5 mm 5-pin balance plug (XT60 lead unused). Balancer per cell: HY2213 OUT drives an AO3400A that bleeds the cell"
- note added: "C1 / C2 at pin 8 of U1 / U2. Bars read the open-circuit voltage (the module draws ~10 mA)."
- note added: "CHARGE); a brick plugged in while RUN or OFF does nothing. U5: buck at 300 kHz, Q6 switch, D7 blocks the packs from the input, D8 freewheels,"
- note added: "D14 / D13 / D12 as pack A; D11 (ON) from +OUT = +V live. C20 / C21 at pin 8 of U14 / U15."
- note added: "D4 >= 16.0 V (80 %), D3 >= 15.2 V (50 %), D2 >= 14.4 V (20 %) from +G; D1 (ON) lit by Q14 while Q11 conducts (-V live)."
- note added: "J1 / U4: the CH224A asks a PD brick for 20 V (R24 120k on CFG1). Q13 passes VBUS to the charger only while Q12 sees +CHGB (toggle in"
- note added: "L1 22 uH, R25 + R26 = 0.2 R -> 1 A constant current shared by the two packs in parallel (F3), 16.8 V +-1 % constant voltage, termination at"
- note added: "Ladder (107 uA): TH80 2.137 V, TH50 2.029 V, TH20 1.920 V, THCUT 1.595 V. VS = rail x 0.1357 with the output live, x 0.1271 cut off; rail = pack - 0.25 V (SS14)."
- note added: "OUT: +V / 0V / -V / nc (JST-PH 4, to the module)"
- note added: "PACK A (-V side): GND .. +BAT"
- note added: "PACK B (+V side): 0V .. +BATB"
- note added: "Packs strapped under the board (two 20 mm straps through the slots), leads to J5 / J6 at the front edge."
- note added: "R30 holds 0V at GND. Q1: U15B pulls the gate low (R1/R2) while VSB > THCUTB. Q11 (N, on pack A's negative): R39 from 0V and R40 give Vgs = +BAT/2 in RUN;"
- note added: "RUN -> +RUN -> F1 -> +SW -> Q1 -> +OUT (+V); CHARGE -> +CHGB -> F3 (1.1 A PTC) -> +BAT (positives joined: both packs on the one charger). OFF opens both,"
- note added: "SW1 pole 1 (common 0V = pack B negative): RUN -> +BAT (packs in series, 0V = output 0 V); CHARGE -> GND (negatives joined). Pole 2 (common +BATB):"
- note added: "Standing draw in OFF about 40 uA (balancers, charger output stage)."
- note added: "Thresholds 16.0 / 15.2 / 14.4 V (pack) for the 80 / 50 / 20 % LEDs, cutoff 12.0 V, re-enable 12.8 V (pack B, R53 from +OUT) / 12.9 V (pack A, R11 from Q11's gate)."
- note added: "Toggle RUN powers the module; OFF; CHARGE joins the packs in parallel on the charger and opens"
- note added: "U2B pulls the gate low below 12.0 V (R11 470k from the gate: back on at 12.9 V); in OFF and CHARGE 0V is at GND, so Q11 is off and -V floats. Gauge rails:"
- note added: "both outputs. -V floats whenever pack A is off (OFF, CHARGE, under-voltage), +V whenever pack B"
- note added: "cell 1"
- note added: "cell 2"
- note added: "cell 3"
- note added: "cell 4"
- note added: "is: the module's fault comparator reports a missing rail."
- note added: "resistor disables it). D9 CHRG (red), D10 DONE (green). All of it on GND = pack A negative = the USB-C shell."
- note added: "through 100 R (42 mA, 0.18 W) above 4.200 V, off at 4.19 V; 2.5 uA standing. With the charger's 16.8 V this is the balance. Pack B's negative is the 0 V output node."
- note removed: "(= 0 V), lower OUT_GND -> LINK_N -> upper J3.3 (= -V), upper +RUN -> lower STACK_IN (slave enable). Upper J3 = +V / 0 V / -V / (+RUN) to the"
- note removed: "(R1/R2: Vgs = -(+SW)/2) while VS > THCUT: +OUT off below 12.0 V, back on above 12.8 V (R11). Slave: with the upper board in RUN its +RUN"
- note removed: "+"
- note removed: "+G = +BAT - 0.25 V (SS14). Thresholds 16.0 / 15.2 / 14.4 V (pack) for D4 / D3 / D2, cutoff 12.0 V, re-enable 12.8 V. R3: >= 1.3 mA in U3 at 12 V."
- note removed: "-"
- note removed: "1. CELLS (4S 18650 in MY-18650-01 clips) AND PER-CELL BALANCERS (HY2213-BB3A, 42 mA above 4.20 V)"
- note removed: "16.8 V +-1 % constant voltage, termination at 9 % (92 mA), trickle at 150 mA below 11.2 V, re-charge below 16.0 V, over-voltage cut at 18.1 V."
- note removed: "18650 #1"
- note removed: "18650 #2"
- note removed: "18650 #3"
- note removed: "18650 #4"
- note removed: "2. RUN / OFF / CHARGE TOGGLE, 100 mA PTC, UNDER-VOLTAGE CUTOFF, STACK SLAVE ENABLE"
- note removed: "3. 2.495 V REFERENCE, THRESHOLD LADDER, PACK SAMPLE (on +G)"
- note removed: "300 kHz, Q6 switch, D7 blocks the pack from the input through Q6's body diode, D8 freewheels, L1 22 uH, R25 + R26 = 0.2 R -> 1 A constant current,"
- note removed: "4. GAUGE: THREE COMPARATORS, FOUR LEDs (about 1 mA each)"
- note removed: "5. OUTPUT, STACK LINK, MOUNTING HOLES"
- note removed: "6. USB-C PD 20 V INPUT (CH224A) AND 4S BUCK CHARGER (CN3704, 1 A), ALL ON CGND"
- note removed: "CHARGE -> CGND (USB-C ground, charger return). OFF opens both. Gauge rail +G = +SW or +CHG through D5 / D6. U2B pulls Q1's gate low"
- note removed: "Charging: either or both toggles in CHARGE, plug USB-C PD bricks in; a charging board has both output lines open, so grounds never loop."
- note removed: "Each cell: two clips 48.0 mm apart (pin rows), contact plates 65 mm apart. Balancer per cell: HY2213 OUT drives an AO3400A that bleeds the"
- note removed: "J1 / U4: the CH224A asks a PD brick for 20 V (R24 120k on CFG1); below 20 V the CN3704 cannot reach 16.8 V and nothing charges. U5: buck at"
- note removed: "LINK IN from the lower board's J3 (lower +OUT -> GND here)"
- note removed: "Ladder (107 uA): TH80 2.137 V, TH50 2.029 V, TH20 1.920 V, THCUT 1.595 V. VS = +G x 0.1357 with +OUT live (R9 || R11 against R10), x 0.1271 cut off;"
- note removed: "OUT: +V / 0V / -V / STACK_IN (to the module, or to the upper board's J4)"
- note removed: "Open collectors sink the LED cathodes: D4 >= 16.0 V (80 %), D3 >= 15.2 V (50 %), D2 >= 14.4 V (20 %) from +G, so the bar also shows while"
- note removed: "RT1 10k NTC between the cells stops charging hot / cold (10k fixed resistor disables it). D9 CHRG (red), D10 DONE (green). CGND meets GND only"
- note removed: "SW1 pole 1 (common +BAT): RUN -> +RUN -> F1 (100 mA hold, 300 mA trip) -> +SW -> Q1 -> +OUT; CHARGE -> +CHG. Pole 2 (common GND): RUN -> OUT_GND (J3.2);"
- note removed: "Two identical boards stacked on 25 mm M3 standoffs; lower J3 -> upper J4 with a straight 4-wire JST-PH cable: lower +OUT -> upper GND"
- note removed: "arrives on J3.4 (STACK_IN), Q2 (gate on +OUT = upper GND) sources into Q3's gate, Q3 pulls Q4's gate down, Q4 feeds +RUN. Q5 blocks it in CHARGE."
- note removed: "cell through 100 R (42 mA, 0.18 W) above 4.200 V, off at 4.19 V; 2.5 uA standing. Together with the charger's 16.8 V this is the balance."
- note removed: "charging; D1 (from +OUT) = output live. Bar reads the open-circuit voltage (the e-stim module draws ~10 mA). C1 / C2 at pin 8 of U1 / U2."
- note removed: "e-stim module. Lower toggle: OFF normally (its output follows the upper toggle), CHARGE to charge; RUN only for a board on its own."
- note removed: "in the CHARGE position (SW1 pole 2); R30 1M keeps it defined otherwise, so a brick plugged in while running does nothing. 20 uA from the pack idle."
- title: 4S 18650 battery pack for the LaserHAT e-stim module -> Battery board for the LaserHAT e-stim module: two 4S hobby packs, one charger
- moved on the sheet: C1, C10, C11, C12, C13, C14, C2, C3, C4, C5, C6, C7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

Commit message: BatteryPack rev C: XT60 sockets for the packs' discharge leads, pack B ON LED in its column
J7 / J8 (Amass XT60PW-M, C98732) at the front edge inboard of the XH sockets carry the run and charge
current; the balance leads keep the cell taps (XH pins 1 / 5 parallel the XT60).  Toggle and output
header sit between the XT60s, chain B moved right of its gauge, F3 / R30 above J7.  R54 on +OUT beside
Q1, thin net to D11 at the bottom of pack B's LED column.  Re-routed (Freerouting), stubs pruned,
DRC 0 / 0 / 0, ERC 0, path / sync 0, fab 136 placements / 44 BOM lines.

Co-Authored-By: Claude Fable 5.1 <noreply@anthropic.com>
Claude-Session: https://claude.ai/code/session_018vgLizGzYPynnY93ajvoVA
Parts:
- added J7, J8: XT60PW-M, Connector_AMASS:AMASS_XT60PW-M_1x02_P7.20mm_Horizontal, symbol battpack:Conn_01x02
Connections:
- net +BAT: now also J7.2 (Pin_2)
- net +BATB: now also J8.2 (Pin_2)
- net 0V: now also J8.1 (Pin_1)
- net GND: now also J7.1 (Pin_1)
Other:
- note added: "1. TWO 4S PACKS: XT60 DISCHARGE PLUGS (J7 / J8, run + charge current) AND JST-XH BALANCE LEADS (pin 1 = black = pack negative), PER-CELL BALANCERS (HY2213-BB3A, 42 mA above 4.20 V)"
- note added: "Any 4S LiPo / Li-ion hobby pack with a JST-XH 2.5 mm 5-pin balance plug and an XT60 discharge plug. Balancer per cell: HY2213 OUT drives an AO3400A that bleeds the cell"
- note added: "Packs strapped under the board (two 20 mm straps through the slots), XT60 plugs to J7 / J8 and balance leads to J5 / J6 at the front edge."
- note removed: "1. TWO 4S PACKS ON JST-XH BALANCE LEADS (pin 1 = black = pack negative) AND PER-CELL BALANCERS (HY2213-BB3A, 42 mA above 4.20 V)"
- note removed: "Any 4S LiPo / Li-ion hobby pack with a JST-XH 2.5 mm 5-pin balance plug (XT60 lead unused). Balancer per cell: HY2213 OUT drives an AO3400A that bleeds the cell"
- note removed: "Packs strapped under the board (two 20 mm straps through the slots), leads to J5 / J6 at the front edge."

Commit message: BatteryPack: 3D model for the XT60PW-M sockets
KiCad 9 ships no model for the horizontal XT60, so battpack.pretty/XT60PW-M.kicad_mod is KiCad's AMASS footprint
pointed at battpack.3dshapes/XT60PW-M.step, built by tools/make_xt60_model.py (CadQuery) from the vertical XT60-M
nose plus the PW body, bent pins and legs after Amass drawing XT60PW-M30.  Board swapped in place (copper kept),
DRC 0 / 0 / 0, path / sync 0; renders show the sockets.

Co-Authored-By: Claude Fable 5.1 <noreply@anthropic.com>
Claude-Session: https://claude.ai/code/session_018vgLizGzYPynnY93ajvoVA
Parts:
- J7, J8: footprint Connector_AMASS:AMASS_XT60PW-M_1x02_P7.20mm_Horizontal -> battpack:XT60PW-M
Changed lines of the file:
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@@
     (property "Reference" "J7" (at 30.48 100.33  0) (effects (font (size 1.27 1.27)) ))
     (property "Value" "XT60PW-M" (at 30.48 97.79  0) (effects (font (size 1.27 1.27)) ))
-    (property "Footprint" "Connector_AMASS:AMASS_XT60PW-M_1x02_P7.20mm_Horizontal" (at 30.48 104.14 0) (effects (font (size 1.27 1.27)) (hide yes)))
+    (property "Footprint" "battpack:XT60PW-M" (at 30.48 104.14 0) (effects (font (size 1.27 1.27)) (hide yes)))
     (property "Datasheet" "" (at 30.48 104.14 0) (effects (font (size 1.27 1.27)) (hide yes)))
     (property "LCSC Part #" "C98732" (at 30.48 104.14 0) (effects (font (size 1.27 1.27)) (hide yes)))
@@
     (property "Reference" "J8" (at 289.56 100.33  0) (effects (font (size 1.27 1.27)) ))
     (property "Value" "XT60PW-M" (at 289.56 97.79  0) (effects (font (size 1.27 1.27)) ))
-    (property "Footprint" "Connector_AMASS:AMASS_XT60PW-M_1x02_P7.20mm_Horizontal" (at 289.56 104.14 0) (effects (font (size 1.27 1.27)) (hide yes)))
+    (property "Footprint" "battpack:XT60PW-M" (at 289.56 104.14 0) (effects (font (size 1.27 1.27)) (hide yes)))
     (property "Datasheet" "" (at 289.56 104.14 0) (effects (font (size 1.27 1.27)) (hide yes)))
     (property "LCSC Part #" "C98732" (at 289.56 104.14 0) (effects (font (size 1.27 1.27)) (hide yes)))
