File: LaserHAT/StimHAT/StimHAT.kicad_sch (KiCad schematic)
At the start: 123 parts, among them J1 GPIO, J10 OLED 0.91 (GND VCC SCL SDA), J101 ELECTRODE E1/E2, J102 B4B-PH-K-S(LF)(SN), J5 GT-USB-7010ASV, J6 BNC TRIGGER IN, J7 BNC STIM OUT, Q101 MMBT3904, Q102 MMBT3906, Q3 AP30P30Q, Q4 DMMT5401, Q5 AP30P30Q, SW10 MSK12C02, SW6 TS-1088-AR02016, SW7 SKRHADE010, SW9 TS-1088-AR02016, U1 M24C32-WDW6TP, U101 ISO7741FDBQR, U104 TLV76050DBZR, U105 DAC60501ZDGSR, U106 OPA2192IDGKR, U107 CD74HC4053PWR, U108 DG418DY-T1-E3, U109 ISO1640BDR, U110 TLV1702AIDGKR, U4 MCP1700T-3302E/MB, U5 AP2171W, U6 CH340N, U7 MSPM0G3507SRHBR, U8 74LVC2G17GW

Commit message: StimHAT: third layout review - 15.5 mm tab, vertical electrode header below the DC-DC pins, barrier margin above U109, NYLON marker, Pi 4 AV-jack note
Co-Authored-By: Claude Fable 5.1 <noreply@anthropic.com>
Claude-Session: https://claude.ai/code/session_015kiXLxnPpBaXdXJu2EMvn7
Parts:
- J101: footprint Connector_PinHeader_2.54mm:PinHeader_1x02_P2.54mm_Horizontal -> Connector_PinHeader_2.54mm:PinHeader_1x02_P2.54mm_Vertical
Changed lines of the file:
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@@
     (property "Reference" "J101" (at 336.55 327.66  0) (effects (font (size 1.27 1.27)) ))
     (property "Value" "ELECTRODE E1/E2" (at 336.55 335.28  0) (effects (font (size 1.27 1.27)) ))
-    (property "Footprint" "Connector_PinHeader_2.54mm:PinHeader_1x02_P2.54mm_Horizontal" (at 336.55 331.47 0) (effects (font (size 1.27 1.27)) (hide yes)))
+    (property "Footprint" "Connector_PinHeader_2.54mm:PinHeader_1x02_P2.54mm_Vertical" (at 336.55 331.47 0) (effects (font (size 1.27 1.27)) (hide yes)))
     (property "Datasheet" "" (at 336.55 331.47 0) (effects (font (size 1.27 1.27)) (hide yes)))
     (pin "1")

Commit message: StimHAT: PS1 moves to the band north of the right-angle BNCs (vertical BNC option dropped), 7.5 mm tab with J101 beside J102, nothing below the HAT; DRC 0/0
Co-Authored-By: Claude Fable 5.1 <noreply@anthropic.com>
Claude-Session: https://claude.ai/code/session_015kiXLxnPpBaXdXJu2EMvn7
Parts:
- J6, J7: footprint Footprints:BNC_Amphenol_031-5540_031-5539_Dual -> stimhat:BNC_Amphenol_031-5540_RA
Changed lines of the file:
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@@
     (property "Reference" "J6" (at 533.4 36.83  0) (effects (font (size 1.27 1.27)) ))
     (property "Value" "BNC TRIGGER IN" (at 533.4 44.45  0) (effects (font (size 1.27 1.27)) ))
-    (property "Footprint" "Footprints:BNC_Amphenol_031-5540_031-5539_Dual" (at 533.4 40.64 0) (effects (font (size 1.27 1.27)) (hide yes)))
+    (property "Footprint" "stimhat:BNC_Amphenol_031-5540_RA" (at 533.4 40.64 0) (effects (font (size 1.27 1.27)) (hide yes)))
     (property "Datasheet" "" (at 533.4 40.64 0) (effects (font (size 1.27 1.27)) (hide yes)))
     (pin "1")
@@
     (property "Reference" "J7" (at 624.84 77.47  0) (effects (font (size 1.27 1.27)) ))
     (property "Value" "BNC STIM OUT" (at 624.84 85.09  0) (effects (font (size 1.27 1.27)) ))
-    (property "Footprint" "Footprints:BNC_Amphenol_031-5540_031-5539_Dual" (at 624.84 81.28 0) (effects (font (size 1.27 1.27)) (hide yes)))
+    (property "Footprint" "stimhat:BNC_Amphenol_031-5540_RA" (at 624.84 81.28 0) (effects (font (size 1.27 1.27)) (hide yes)))
     (property "Datasheet" "" (at 624.84 81.28 0) (effects (font (size 1.27 1.27)) (hide yes)))
     (pin "1")

Commit message: StimHAT: round 6 placement - J102 beside PS1 (one fitted), J101 alone on a 10 mm tab, J10 vertical OLED socket at the strip's west end, PS1 silk + 3D model, MH4 keep-out 3.25; invalidated copper ripped, 23 open connections left for hand routing
Co-Authored-By: Claude Fable 5.1 <noreply@anthropic.com>
Claude-Session: https://claude.ai/code/session_015kiXLxnPpBaXdXJu2EMvn7
Parts:
- J10: footprint Connector_PinSocket_2.54mm:PinSocket_1x04_P2.54mm_Horizontal -> Connector_PinSocket_2.54mm:PinSocket_1x04_P2.54mm_Vertical
- J102: footprint Connector_JST:JST_PH_B4B-PH-K_1x04_P2.00mm_Vertical -> stimhat:JST_PH_B4B-PH-K_NoCrtYd
Changed lines of the file:
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@@
     (property "Reference" "J10" (at 467.36 128.27  0) (effects (font (size 1.27 1.27)) ))
     (property "Value" "OLED 0.91 (GND VCC SCL SDA)" (at 467.36 146.05  0) (effects (font (size 1.27 1.27)) ))
-    (property "Footprint" "Connector_PinSocket_2.54mm:PinSocket_1x04_P2.54mm_Horizontal" (at 467.36 137.16 0) (effects (font (size 1.27 1.27)) (hide yes)))
+    (property "Footprint" "Connector_PinSocket_2.54mm:PinSocket_1x04_P2.54mm_Vertical" (at 467.36 137.16 0) (effects (font (size 1.27 1.27)) (hide yes)))
     (property "Datasheet" "" (at 467.36 137.16 0) (effects (font (size 1.27 1.27)) (hide yes)))
     (pin "1")
@@
     (property "Reference" "J102" (at 187.96 227.33  0) (effects (font (size 1.27 1.27)) ))
     (property "Value" "B4B-PH-K-S(LF)(SN)" (at 187.96 240.03  0) (effects (font (size 1.27 1.27)) ))
-    (property "Footprint" "Connector_JST:JST_PH_B4B-PH-K_1x04_P2.00mm_Vertical" (at 187.96 233.68 0) (effects (font (size 1.27 1.27)) (hide yes)))
+    (property "Footprint" "stimhat:JST_PH_B4B-PH-K_NoCrtYd" (at 187.96 233.68 0) (effects (font (size 1.27 1.27)) (hide yes)))
     (property "Datasheet" "" (at 187.96 233.68 0) (effects (font (size 1.27 1.27)) (hide yes)))
     (pin "1")
