File: LaserHAT/StimHAT/StimHAT.kicad_sch (KiCad schematic)
At the start: 112 parts, among them J1 GPIO, J10 OLED 0.91 (GND VCC SCL SDA), J101 ELECTRODE E1/E2, J102 B4B-PH-K-S(LF)(SN), J103 5V TO DC-DC POD, J5 GT-USB-7010ASV, J6 BNC TRIGGER IN, J7 BNC STIM OUT, Q3 AP30P30Q, Q4 DMMT5401, Q5 AP30P30Q, SW10 MSK12C02, SW6 TS-1088-AR02016, SW7 SKRHADE010, SW9 TS-1088-AR02016, U1 M24C32-WDW6TP, U101 ISO7741FDBQR, U104 TLV76050DBZR, U105 DAC60501ZDGSR, U106 OPA2192IDGKR, U107 CD74HC4053PWR, U108 DG418DY-T1-E3, U109 ISO1640BDR, U110 TLV1702AIDGKR, U4 MCP1700T-3302E/MB, U5 AP2171W, U6 CH340N, U7 MSPM0G1507SRHBR, U8 74LVC2G17GW

Commit message: Semi-final main routing
Connections:
- net LED_MCU: now also U7.9 (PA5); no longer U7.10 (PA6)
