File: LaserHAT/StimHAT/StimHAT.kicad_pcb (KiCad board)
At the start: 4 copper layers, 65 x 57 mm, 112 parts, among them J1 GPIO, J10 OLED 0.91 (GND VCC SCL SDA), J101 ELECTRODE E1/E2, J102 B4B-PH-K-S(LF)(SN), J103 5V TO DC-DC POD, J5 GT-USB-7010ASV, J6 BNC TRIGGER IN, J7 BNC STIM OUT, Q3 AP30P30Q, Q4 DMMT5401, Q5 AP30P30Q, SW10 MSK12C02, SW6 TS-1088-AR02016, SW7 SKRHADE010, SW9 TS-1088-AR02016, U1 M24C32-WDW6TP, U101 ISO7741FDBQR, U104 TLV76050DBZR, U105 DAC60501ZDGSR, U106 OPA2192IDGKR, U107 CD74HC4053PWR, U108 DG418DY-T1-E3, U109 ISO1640BDR, U110 TLV1702AIDGKR, U4 MCP1700T-3302E/MB, U5 AP2171W, U6 CH340N, U7 MSPM0G1507SRHBR, U8 74LVC2G17GW

Commit message: Updated routing for isolated portion and correctly rotated screen connector
Parts:
- moved J10 14.6 mm to (11.8, 19.5), turned to 180 degrees
- moved TP101 1.38 mm to (62.2, 45.0)
Routing:
- net SHORT_IN: track 0.00 -> 16.6 mm, vias 0 -> 2
- net E1: track 32.9 -> 37.3 mm, vias 0 -> 2
- net +V_STIM: track 62.5 -> 58.5 mm, vias 10 -> 9
- net ISENSE: track 34.1 -> 36.7 mm
- net -V_STIM: track 46.9 -> 48.0 mm
