File: LaserHAT/StimHAT/StimHAT.kicad_pcb (KiCad board)
At the start: 4 copper layers, 65 x 57 mm, 112 parts, among them J1 GPIO, J10 OLED 0.91 (GND VCC SCL SDA), J101 ELECTRODE E1/E2, J102 B4B-PH-K-S(LF)(SN), J103 5V TO DC-DC POD, J5 GT-USB-7010ASV, J6 BNC TRIGGER IN, J7 BNC STIM OUT, Q3 AP30P30Q, Q4 DMMT5401, Q5 AP30P30Q, SW10 MSK12C02, SW6 TS-1088-AR02016, SW7 SKRHADE010, SW9 TS-1088-AR02016, U1 M24C32-WDW6TP, U101 ISO7741FDBQR, U104 TLV76050DBZR, U105 DAC60501ZDGSR, U106 OPA2192IDGKR, U107 CD74HC4053PWR, U108 DG418DY-T1-E3, U109 ISO1640BDR, U110 TLV1702AIDGKR, U4 MCP1700T-3302E/MB, U5 AP2171W, U6 CH340N, U7 MSPM0G1507SRHBR, U8 74LVC2G17GW

Commit message: Updated main routing
Parts:
- moved R3 15.6 mm to (22.3, 19.2), turned to 180 degrees
- moved C3 14.8 mm to (20.3, 19.2), turned to 180 degrees
- moved U1 13.0 mm to (53.4, 12.2), turned to 180 degrees
- moved R2 11.8 mm to (46.7, 12.2), turned to 0 degrees
- moved C18 7.99 mm to (50.5, 15.0), turned to -90 degrees
- moved JP4 7.12 mm to (12.2, 30.5), turned to 180 degrees
- moved U6 6.83 mm to (14.5, 25.9), turned to 0 degrees
- moved JP1 6.43 mm to (53.1, 15.6)
- moved R101 4.82 mm to (29.5, 26.8), turned to 180 degrees
- moved U7 3.25 mm to (23.2, 26.0)
- moved R103 3.12 mm to (31.0, 25.6)
- moved R102 2.83 mm to (29.4, 27.8), turned to 180 degrees
- moved R1 2.80 mm to (48.3, 11.2), turned to 0 degrees
- moved C4 2.38 mm to (27.0, 23.4)
- moved C101 2.01 mm to (31.0, 22.0)
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Routing:
- net ID_SCL: track 0.00 -> 17.4 mm, vias 0 -> 1
- net ID_SDA: track 0.00 -> 11.7 mm, vias 0 -> 1
- net +3V3_PI: track 0.00 -> 10.4 mm, vias 0 -> 2
- net USB_DM: track 17.9 -> 8.55 mm, vias 0 -> 2
- net USB_DP: track 17.8 -> 9.75 mm, vias 2 -> 0
- net I2C_SDA: track 0.00 -> 5.85 mm
- net I2C_SCL: track 0.00 -> 5.40 mm
- net PI_TXD: track 0.00 -> 5.23 mm
- net JP1_A: track 0.00 -> 4.58 mm
- net PI_RXD: track 0.00 -> 4.49 mm
- net SDA_H: track 0.00 -> 4.31 mm
- net MCU_UART_TX: track 0.00 -> 4.26 mm
- net MCU_UART_RX: track 0.00 -> 3.94 mm
- net SWCLK: track 0.00 -> 1.88 mm
- net ROSC: track 0.00 -> 1.88 mm
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