File: LaserHAT/StimHAT/StimHAT.kicad_pcb (KiCad board)
At the start: 4 copper layers, 65 x 57 mm, 112 parts, among them J1 GPIO, J10 OLED 0.91 (GND VCC SCL SDA), J101 ELECTRODE E1/E2, J102 B4B-PH-K-S(LF)(SN), J103 5V TO DC-DC POD, J5 GT-USB-7010ASV, J6 BNC TRIGGER IN, J7 BNC STIM OUT, Q3 AP30P30Q, Q4 DMMT5401, Q5 AP30P30Q, SW10 MSK12C02, SW6 TS-1088-AR02016, SW7 SKRHADE010, SW9 TS-1088-AR02016, U1 M24C32-WDW6TP, U101 ISO7741FDBQR, U104 TLV76050DBZR, U105 DAC60501ZDGSR, U106 OPA2192IDGKR, U107 CD74HC4053PWR, U108 DG418DY-T1-E3, U109 ISO1640BDR, U110 TLV1702AIDGKR, U4 MCP1700T-3302E/MB, U5 AP2171W, U6 CH340N, U7 MSPM0G1507SRHBR, U8 74LVC2G17GW

Commit message: StimHAT: PI_TRIGGER moved to Pi GPIO10 (J1.19) / U7 pin 8, RELEASE_H to pin 31
At the user's request (routing): the trigger line now comes straight down from the header's west
half into PA4 (pin 8) instead of crossing the board from J1.37 to PA27; RELEASE_H takes pin 31
(PA27) so it leaves U7 on the isolator side; pin 19 (PA15, DAC0_OUT) and pin 7 (PA3) are spare.
GPIO10 rather than 4 / 17 / 22 / 27 (bonnet buttons) or 7 / 8 (pull up at boot).

Schematic regenerated (netcheck OK, ERC 0), nets pushed into the board with the tracks kept
(path / sync checks 0), placement table synced from the user's board (21 parts).  README pin map
updated.  The Pi software still defaults to GPIO 26: StimHAT needs LASERHAT_TRIGGER_PIN=10 and
`laserhat-brokerd --gpio-pin 10`.

Co-Authored-By: Claude Fable 5.1 <noreply@anthropic.com>
Claude-Session: https://claude.ai/code/session_015kiXLxnPpBaXdXJu2EMvn7
Connections:
- J1 pad 19: unconnected-(J1-GPIO10-Pad19) -> PI_TRIGGER
- J1 pad 37: PI_TRIGGER -> unconnected-(J1-GPIO26-Pad37)
- U7 pad 19: RELEASE_H -> unconnected-(U7-PA15/DAC-Pad19)
- U7 pad 31: PI_TRIGGER -> RELEASE_H
- U7 pad 8: unconnected-(U7-PA4-Pad8) -> PI_TRIGGER
