File: LaserHAT/StimHAT/StimHAT.kicad_pcb (KiCad board)
At the start: 4 copper layers, 65 x 57 mm, 112 parts, among them J1 GPIO, J10 OLED 0.91 (GND VCC SCL SDA), J101 ELECTRODE E1/E2, J102 B4B-PH-K-S(LF)(SN), J103 5V TO DC-DC POD, J5 GT-USB-7010ASV, J6 BNC TRIGGER IN, J7 BNC STIM OUT, Q3 AP30P30Q, Q4 DMMT5401, Q5 AP30P30Q, SW10 MSK12C02, SW6 TS-1088-AR02016, SW7 SKRHADE010, SW9 TS-1088-AR02016, U1 M24C32-WDW6TP, U101 ISO7741FDBQR, U104 TLV76050DBZR, U105 DAC60501ZDGSR, U106 OPA2192IDGKR, U107 CD74HC4053PWR, U108 DG418DY-T1-E3, U109 ISO1640BDR, U110 TLV1702AIDGKR, U4 MCP1700T-3302E/MB, U5 AP2171W, U6 CH340N, U7 MSPM0G1507SRHBR, U8 74LVC2G17GW

Commit message: Updated main routing
Parts:
- moved SW6 25.0 mm to (22.5, 33.9), turned to -90 degrees
- moved JP5 20.4 mm to (27.2, 10.6)
- moved R107 15.3 mm to (42.6, 14.3), turned to -90 degrees
- moved R108 12.1 mm to (41.4, 14.3), turned to -90 degrees
- moved C17 11.7 mm to (21.1, 20.7), turned to 180 degrees
- moved C13 7.43 mm to (23.1, 10.4), turned to 180 degrees
- moved C6 3.52 mm to (23.1, 11.5)
- moved C2 1.74 mm to (32.5, 15.6)
- moved U5 1.43 mm to (28.9, 15.4), turned to 180 degrees
- moved R7 1.00 mm to (27.3, 12.9), turned to 0 degrees
- moved R103 0.90 mm to (30.1, 25.6), turned to 180 degrees
- moved C3 0.89 mm to (21.2, 19.2), turned to 90 degrees
- moved U8 0.88 mm to (27.4, 32.6), turned to 0 degrees
- moved R102 0.70 mm to (30.1, 27.8)
- moved R101 0.61 mm to (30.1, 26.7)
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Routing:
- net BUTTON6: track 1.40 -> 27.9 mm
- net BUTTON4: track 1.51 -> 28.0 mm
- net LED_MCU: track 1.61 -> 26.6 mm
- net Net-(J7-In): track 0.00 -> 18.2 mm
- net BUTTON1: track 0.00 -> 13.3 mm
- net +3V3: track 0.00 -> 12.8 mm
- net BUTTON2: track 0.00 -> 12.6 mm
- net Net-(J6-In): track 0.00 -> 9.99 mm
- net MCU_STIM_IN: track 0.00 -> 8.06 mm
- net MCU_STIM_OUT: track 0.00 -> 8.02 mm, vias 0 -> 2
- net BUTTON5: track 0.00 -> 6.34 mm
- net NRST: track 0.00 -> 6.13 mm
- net Net-(U8-1A): track 0.00 -> 5.48 mm
- net BUTTON3: track 0.00 -> 5.27 mm
- net Net-(D9-A): track 0.00 -> 4.24 mm
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