File: LaserHAT/StimHAT/StimHAT.kicad_pcb (KiCad board)
At the start: 4 copper layers, 65 x 57 mm, 112 parts, among them J1 GPIO, J10 OLED 0.91 (GND VCC SCL SDA), J101 ELECTRODE E1/E2, J102 B4B-PH-K-S(LF)(SN), J103 5V TO DC-DC POD, J5 GT-USB-7010ASV, J6 BNC TRIGGER IN, J7 BNC STIM OUT, Q3 AP30P30Q, Q4 DMMT5401, Q5 AP30P30Q, SW10 MSK12C02, SW6 TS-1088-AR02016, SW7 SKRHADE010, SW9 TS-1088-AR02016, U1 M24C32-WDW6TP, U101 ISO7741FDBQR, U104 TLV76050DBZR, U105 DAC60501ZDGSR, U106 OPA2192IDGKR, U107 CD74HC4053PWR, U108 DG418DY-T1-E3, U109 ISO1640BDR, U110 TLV1702AIDGKR, U4 MCP1700T-3302E/MB, U5 AP2171W, U6 CH340N, U7 MSPM0G1507SRHBR, U8 74LVC2G17GW

Commit message: StimHAT: U7's east column re-ordered to match the isolator's pin order
At the user's request (routing): top to bottom SCL_H / SDA_H (PA27 / PA26, ADC0 ch 0 / 1) toward
U109, then RELEASE_H, EN_H, CATH_H, FAULT_H (PA25, PA24, PA23, PA22) in U101's HAT-side pin order,
STIM_IN (PA21) at the bottom toward U8.  FAULT_H is now a plain GPIO IRQ pin (the firmware's
fault path already is one; TIMA0's hardware fault inputs are only on PA26 / PA27); for a laser
variant PWM_A on PA24 would be TIMA0_CCP3N or TIMA1_CCP1 against PWM_B on PA23 = TIMA0_CCP3.

Schematic regenerated (netcheck OK, ERC 0), nets pushed into the board with the tracks kept
(path / sync checks 0); the user's SDA_H stub on the old pin 28 was removed.  README pin map
updated.

Co-Authored-By: Claude Fable 5.1 <noreply@anthropic.com>
Claude-Session: https://claude.ai/code/session_015kiXLxnPpBaXdXJu2EMvn7
Connections:
- U7 pad 26: CATH_H -> FAULT_H
- U7 pad 27: EN_H -> CATH_H
- U7 pad 28: SDA_H -> EN_H
- U7 pad 29: SCL_H -> RELEASE_H
- U7 pad 30: FAULT_H -> SDA_H
- U7 pad 31: RELEASE_H -> SCL_H
Routing:
- net SDA_H: track 0.85 -> 0.00 mm
Changed lines of the file:
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@@
 			(size 0.254 0.8128)
 			(layers "F.Cu" "F.Mask" "F.Paste")
-			(net 25 "CATH_H")
+			(net 30 "FAULT_H")
 			(pinfunction "PA22")
 			(pintype "bidirectional")
@@
 			(size 0.254 0.8128)
 			(layers "F.Cu" "F.Mask" "F.Paste")
-			(net 29 "EN_H")
+			(net 25 "CATH_H")
 			(pinfunction "PA23")
 			(pintype "bidirectional")
@@
 			(size 0.254 0.8128)
 			(layers "F.Cu" "F.Mask" "F.Paste")
-			(net 67 "SDA_H")
+			(net 29 "EN_H")
 			(pinfunction "PA24")
 			(pintype "bidirectional")
@@
 			(size 0.254 0.8128)
 			(layers "F.Cu" "F.Mask" "F.Paste")
-			(net 65 "SCL_H")
+			(net 62 "RELEASE_H")
 			(pinfunction "PA25")
 			(pintype "bidirectional")
@@
 			(size 0.254 0.8128)
 			(layers "F.Cu" "F.Mask" "F.Paste")
-			(net 30 "FAULT_H")
+			(net 67 "SDA_H")
 			(pinfunction "PA26")
 			(pintype "bidirectional")
@@
 			(size 0.254 0.8128)
 			(layers "F.Cu" "F.Mask" "F.Paste")
-			(net 62 "RELEASE_H")
+			(net 65 "SCL_H")
 			(pinfunction "PA27")
 			(pintype "bidirectional")
@@
 	)
 	(segment
-		(start 25.7011 26.250063)
-		(end 26.549937 26.250063)
-		(width 0.2)
-		(layer "F.Cu")
-		(net 67)
-	)
-	(segment
