File: LaserHAT/StimHAT/StimHAT.kicad_pcb (KiCad board)
At the start: 4 copper layers, 65 x 57 mm, 112 parts, among them J1 GPIO, J10 OLED 0.91 (GND VCC SCL SDA), J101 ELECTRODE E1/E2, J102 B4B-PH-K-S(LF)(SN), J103 5V TO DC-DC POD, J5 GT-USB-7010ASV, J6 BNC TRIGGER IN, J7 BNC STIM OUT, Q3 AP30P30Q, Q4 DMMT5401, Q5 AP30P30Q, SW10 MSK12C02, SW6 TS-1088-AR02016, SW7 SKRHADE010, SW9 TS-1088-AR02016, U1 M24C32-WDW6TP, U101 ISO7741FDBQR, U104 TLV76050DBZR, U105 DAC60501ZDGSR, U106 OPA2192IDGKR, U107 CD74HC4053PWR, U108 DG418DY-T1-E3, U109 ISO1640BDR, U110 TLV1702AIDGKR, U4 MCP1700T-3302E/MB, U5 AP2171W, U6 CH340N, U7 MSPM0G1507SRHBR, U8 74LVC2G17GW

Commit message: Updated main routing again
Parts:
- moved R20 6.93 mm to (8.80, 14.4)
- moved R19 3.84 mm to (8.90, 11.9)
- moved U5 3.59 mm to (31.2, 12.7)
- moved C2 3.59 mm to (34.8, 12.8)
- moved C15 2.83 mm to (7.92, 10.2), turned to 180 degrees
- moved R103 0.81 mm to (30.2, 24.8), turned to 90 degrees
- moved R102 0.60 mm to (30.1, 28.4)
- moved R101 0.30 mm to (30.1, 27.0)
- turned SW7 to 135 degrees
Routing:
- net SWDIO: track 1.87 -> 37.2 mm
- net Net-(D9-A): track 4.24 -> 38.1 mm, vias 0 -> 2
- net SWCLK: track 1.46 -> 35.2 mm
- net SDA_H: track 0.00 -> 27.1 mm, vias 0 -> 2
- net BUTTON5: track 6.34 -> 31.3 mm
- net SCL_H: track 0.00 -> 23.7 mm
- net PI_RXD: track 4.49 -> 24.5 mm
- net PI_TXD: track 5.23 -> 24.2 mm
- net BUTTON6: track 27.9 -> 14.7 mm, vias 1 -> 2
- net BUTTON4: track 28.0 -> 15.6 mm, vias 1 -> 2
- net +3V3_PI: track 14.0 -> 24.9 mm
- net I2C_SCL: track 5.40 -> 15.6 mm
- net FAULT_H: track 0.00 -> 8.67 mm
- net CATH_H: track 0.00 -> 8.20 mm
- net EN_H: track 0.00 -> 7.88 mm
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