File: LaserHAT/StimHAT/StimHAT.kicad_pcb (KiCad board)
At the start: 4 copper layers, 65 x 57 mm, 113 parts, among them J1 GPIO, J10 OLED 0.91 (GND VCC SCL SDA), J101 ELECTRODE E1/E2, J102 B4B-PH-K-S(LF)(SN), J103 5V TO DC-DC POD, J5 GT-USB-7010ASV, J6 BNC TRIGGER IN, J7 BNC STIM OUT, Q3 AP30P30Q, Q4 DMMT5401, Q5 AP30P30Q, SW10 MSK12C02, SW6 TS-1088-AR02016, SW7 SKRHADE010, SW9 TS-1088-AR02016, U1 M24C32-WDW6TP, U101 ISO7741FDBQR, U104 TLV76050DBZR, U105 DAC60501ZDGSR, U106 OPA2192IDGKR, U107 CD74HC4053PWR, U108 DG418DY-T1-E3, U109 ISO1640BDR, U110 TLV1702AIDGKR, U4 MCP1700T-3302E/MB, U5 AP2171W, U6 CH340N, U7 MSPM0G1507SRHBR, U8 74LVC2G17GW

Commit message: StimHAT: full-size owl with copper eyes for hand placement
tools/owl_logo.py now derives stimhat:OwlLogo_Eyes_14mm at 100 % (eyes as GND pads, beams as
silk, no courtyard) and keeps G1 wherever it is on the board; the 10 mm variant is removed.
G1 stays at the user's (33.5, 18.05).  As committed DRC has 4 errors (the left eye on the
+3V3 track at x 32.23) and the right eye lies in the barrier strip, which the keep-outs do not
flag for pads: the user is moving the owl by hand, both eyes must end west of x 33.7.

Co-Authored-By: Claude Fable 5.1 <noreply@anthropic.com>
Claude-Session: https://claude.ai/code/session_015kiXLxnPpBaXdXJu2EMvn7
Parts:
- G1: value OwlLogo_Eyes_10mm -> OwlLogo_Eyes_14mm; footprint stimhat:OwlLogo_Eyes_10mm -> stimhat:OwlLogo_Eyes_14mm
