File: LaserHAT/StimHAT/StimHAT.kicad_pcb (KiCad board)
At the start: 4 copper layers, 65 x 57 mm, 113 parts, among them J1 GPIO, J10 OLED 0.91 (GND VCC SCL SDA), J101 ELECTRODE E1/E2, J102 B4B-PH-K-S(LF)(SN), J103 5V TO DC-DC POD, J5 GT-USB-7010ASV, J6 BNC TRIGGER IN, J7 BNC STIM OUT, Q3 AP30P30Q, Q4 DMMT5401, Q5 AP30P30Q, SW10 MSK12C02, SW6 TS-1088-AR02016, SW7 SKRHADE010, SW9 TS-1088-AR02016, U1 M24C32-WDW6TP, U101 ISO7741FDBQR, U104 TLV76050DBZR, U105 DAC60501ZDGSR, U106 OPA2192IDGKR, U107 CD74HC4053PWR, U108 DG418DY-T1-E3, U109 ISO1640BDR, U110 TLV1702AIDGKR, U4 MCP1700T-3302E/MB, U5 AP2171W, U6 CH340N, U7 MSPM0G1507SRHBR, U8 74LVC2G17GW

Commit message: Moved owl
Parts:
- JP5: moved to B.Cu
- moved C2 9.52 mm to (28.5, 15.0), turned to 0 degrees
- moved G1 9.38 mm to (34.8, 8.75)
- moved U5 5.34 mm to (28.3, 11.6), turned to 90 degrees
- moved R7 3.96 mm to (28.0, 9.00)
- moved JP5 0.38 mm to (26.9, 10.8)
Routing:
- net +3V3: track 18.0 -> 12.6 mm, vias 0 -> 1
- net MCU_PWR_EN: track 8.68 -> 6.12 mm
- net +3V3_PI: track 76.4 -> 74.8 mm
- net MSPM0_3V3: track 89.6 -> 91.1 mm, vias 8 -> 9
- net GND: track 7.70 -> 7.88 mm, vias 31 -> 30
