File: LaserHAT/DCDCPod/DCDCPod.kicad_sch (KiCad schematic)
At the start: 17 parts, among them J1 5V IN (HAT J103), J2 +/-V OUT (HAT J102), Q101 MMBT3904, Q102 MMBT3906

Commit message: DCDCPod: converter footprint for the fitted RECOM RB-0515D/HP
New dcdcpod:DCDC_SIP6_RB0515D generated from the RECOM RB drawing (pins 1.27 mm behind / 4.73 mm
in front of the marked face, pin 1 2.0 mm from the end, 19.6 x 6.0 x 10.2 body on 0.5 mm standoffs
in the model; same 1-2-4-5-6 holes) replaces the copy of the Mornsun footprint; PS1's value is
RB-0515D/HP and it moved 0.4 mm down the pod so the body stays 0.43 mm inside the top edge (z
16.57-22.57, 0.97 mm over the BNC tops).  Body side confirmed from both datasheets; the README's
open point is closed.  DRC 0/0/0, isolation OK, fab outputs and renders regenerated.

Co-Authored-By: Claude Fable 5.1 <noreply@anthropic.com>
Claude-Session: https://claude.ai/code/session_015kiXLxnPpBaXdXJu2EMvn7
Parts:
- PS1: value A0515S-1WR3 -> RB-0515D/HP; footprint dcdcpod:DCDC_SIP6_A0515S_BodyN -> dcdcpod:DCDC_SIP6_RB0515D
Changed lines of the file:
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@@
   (symbol (lib_id "dcdcpod:A0515S") (at 83.82 50.8 0) (unit 1) (exclude_from_sim no) (in_bom no) (on_board yes) (dnp no)
     (property "Reference" "PS1" (at 83.82 41.91  0) (effects (font (size 1.27 1.27)) ))
-    (property "Value" "A0515S-1WR3" (at 83.82 59.69  0) (effects (font (size 1.27 1.27)) ))
-    (property "Footprint" "dcdcpod:DCDC_SIP6_A0515S_BodyN" (at 83.82 50.8 0) (effects (font (size 1.27 1.27)) (hide yes)))
+    (property "Value" "RB-0515D/HP" (at 83.82 59.69  0) (effects (font (size 1.27 1.27)) ))
+    (property "Footprint" "dcdcpod:DCDC_SIP6_RB0515D" (at 83.82 50.8 0) (effects (font (size 1.27 1.27)) (hide yes)))
     (property "Datasheet" "" (at 83.82 50.8 0) (effects (font (size 1.27 1.27)) (hide yes)))
     (pin "1")
